Commit message: Almost working-ish

File: pybullet_data/robot_backup.urdf (robot description, URDF)
Before this commit: robot robot, 6 links, 5 joints
Links:
- link left_hand_link: geometry collision box size=0.1 0.1 0.5; visual box size=0.1 0.1 0.5
- link right_hand_link: geometry collision box size=0.1 0.1 0.5; visual box size=0.1 0.1 0.5
Joints:
- joint body_left_arm_joint: axis 0 0 1 -> 0 1 0; origin xyz=.5 .5 0 rpy=0 0 0 -> xyz=0.5 0 0 rpy=0 0 0
- joint body_right_arm_joint: axis 0 0 1 -> 0 1 0; origin xyz=.5 -.5 0 rpy=0 0 0 -> xyz=0.5 0 0 rpy=0 0 0
- joint left_arm_left_hand_joint: axis 0 0 1 -> 1 0 0; origin xyz=1 0 0 rpy=0 0 0 -> xyz=1 .5 0 rpy=0 0 0
- joint right_arm_right_hand_joint: axis 0 0 1 -> 1 0 0; origin xyz=1 0 0 rpy=0 0 0 -> xyz=1 -.5 0 rpy=0 0 0
