Commit message: working ish

File: pybullet_data/plane.urdf (robot description, URDF)
Before this commit: robot plane, 1 links, 0 joints
Links:
- link planeLink: geometry collision box size=100 100 1; visual box size=100 100 1

File: pybullet_data/robot.urdf (robot description, URDF)
Before this commit: robot robot, 8 links, 7 joints
Links:
- link arm: geometry collision box size=3 .1 .6; visual box size=3 .1 .6
- link arm_sensor: geometry collision box size=3.01 .11 .61; visual box size=3.01 .11 .61
- link hand: geometry collision box size=.1 3 .6; visual box size=.1 3 .6
- link hand_sensor: geometry collision box size=.11 3.01 .61; visual box size=.11 3.01 .61
- link shoulder: geometry collision box size=.1 .1 .6; visual box size=.1 .1 .6
Joints:
- joint body_shoulder_joint: origin xyz=0 .5 0 rpy=0 0 0 -> xyz=0 .55 0 rpy=0 0 0
- joint shoulder_arm_joint: origin xyz=1.5 0 0 rpy=0 0 0 -> xyz=1.45 .1 0 rpy=0 0 0
