Commit message: functioning

File: pybullet_data/robot.urdf (robot description, URDF)
Before this commit: robot robot, 6 links, 5 joints
Links:
- link left_arm_link: geometry collision box size=.5 0.1 0.1; visual box size=.5 0.1 0.1
- link left_hand_link: geometry collision box size=.5 .1 .1; visual box size=.5 .1 .1
- link right_arm_link: geometry collision box size=.5 0.1 0.1; visual box size=.5 0.1 0.1
- link right_hand_link: geometry collision box size=.5 .1 .1; visual box size=.5 .1 .1
Joints:
- joint left_arm_left_hand_joint: origin xyz=1 0 0 rpy=0 0 0 -> xyz=.5 0 0 rpy=0 0 0
- joint right_arm_right_hand_joint: origin xyz=1 0 0 rpy=0 0 0 -> xyz=.5 0 0 rpy=0 0 0

Commit message: so far so okay

File: pybullet_data/robot.urdf (robot description, URDF)
Before this commit: robot robot, 6 links, 5 joints
Links:
- added link left_shoulder_link, mass 1; collision box size=.1 0.1 0.1; visual box size=.1 0.1 0.1
- added link right_shoulder_link, mass 1; collision box size=.1 0.1 0.1; visual box size=.1 0.1 0.1
Joints:
- removed joint body_left_arm_joint
- removed joint body_right_arm_joint
- added joint body_left_shoulder_joint: type continuous, parent body_link, child left_shoulder_link, origin xyz=.5 .5 0 rpy=0 0 0, axis 0 1 0
- added joint body_right_shoulder_joint: type continuous, parent body_link, child right_shoulder_link, origin xyz=.5 -.5 0 rpy=0 0 0, axis 0 1 0
- added joint left_shoulder_left_arm_joint: type continuous, parent left_shoulder_link, child left_arm_link, origin xyz=0 0 0 rpy=0 0 0, axis 0 0 1
- added joint right_shoulder_right_arm_joint: type continuous, parent right_shoulder_link, child right_arm_link, origin xyz=0 0 0 rpy=0 0 0, axis 0 0 1

File: pybullet_data/shapes/1_pole.urdf (robot description, URDF)
Before this commit: robot 1_pole, 21 links, 20 joints
Links:
- removed link 10_link
- removed link 11_link
- removed link 12_link
- removed link 13_link
- removed link 14_link
- removed link 15_link
- removed link 16_link
- removed link 17_link
- removed link 18_link
- removed link 19_link
- removed link 1_link
- removed link 2_link
- removed link 3_link
- removed link 4_link
- removed link 5_link
- removed link 6_link
- removed link 7_link
- removed link 8_link
- removed link 9_link
- link 0_link: geometry collision cylinder length=1 radius=0.2; visual cylinder length=1 radius=0.2
- link base_link: geometry collision cylinder length=1 radius=0.6; visual cylinder length=1 radius=0.6
Joints:
- removed joint 0_1_joint
- removed joint 10_11_joint
- removed joint 11_12_joint
- removed joint 12_13_joint
- removed joint 13_14_joint
- removed joint 14_15_joint
- removed joint 15_16_joint
- removed joint 16_17_joint
- removed joint 17_18_joint
- removed joint 18_19_joint
- removed joint 1_2_joint
- removed joint 2_3_joint
- removed joint 3_4_joint
- removed joint 4_5_joint
- removed joint 5_6_joint
- removed joint 6_7_joint
- removed joint 7_8_joint
- removed joint 8_9_joint
- removed joint 9_10_joint
- joint base_0_joint: origin xyz=0 0 0.05 rpy=0 0 0 -> xyz=0 0 0.5 rpy=0 0 0

File: pybullet_data/shapes/2_top.urdf (robot description, URDF)
Before this commit: robot 2_top, 21 links, 20 joints
Links:
- removed link 10_link
- removed link 11_link
- removed link 12_link
- removed link 13_link
- removed link 14_link
- removed link 15_link
- removed link 16_link
- removed link 17_link
- removed link 18_link
- removed link 19_link
- removed link 2_link
- removed link 3_link
- removed link 4_link
- removed link 5_link
- removed link 6_link
- removed link 7_link
- removed link 8_link
- removed link 9_link
- link 0_link: geometry collision cylinder length=0.9 radius=0.2; visual cylinder length=0.9 radius=0.2
- link 1_link: geometry collision cylinder length=0.1 radius=0.6; visual cylinder length=0.1 radius=0.6
- link base_link: geometry collision cylinder length=1 radius=0.6; visual cylinder length=1 radius=0.6
Joints:
- removed joint 10_11_joint
- removed joint 11_12_joint
- removed joint 12_13_joint
- removed joint 13_14_joint
- removed joint 14_15_joint
- removed joint 15_16_joint
- removed joint 16_17_joint
- removed joint 17_18_joint
- removed joint 18_19_joint
- removed joint 1_2_joint
- removed joint 2_3_joint
- removed joint 3_4_joint
- removed joint 4_5_joint
- removed joint 5_6_joint
- removed joint 6_7_joint
- removed joint 7_8_joint
- removed joint 8_9_joint
- removed joint 9_10_joint
- joint 0_1_joint: origin xyz=0 0 0.05 rpy=0 0 0 -> xyz=0 0 0.5 rpy=0 0 0
- joint base_0_joint: origin xyz=0 0 0.05 rpy=0 0 0 -> xyz=0 0 0.45 rpy=0 0 0

File: pybullet_data/shapes/3_bottom.urdf (robot description, URDF)
Before this commit: robot 3_bottom, 21 links, 20 joints
Links:
- removed link 10_link
- removed link 11_link
- removed link 12_link
- removed link 13_link
- removed link 14_link
- removed link 15_link
- removed link 16_link
- removed link 17_link
- removed link 18_link
- removed link 19_link
- removed link 2_link
- removed link 3_link
- removed link 4_link
- removed link 5_link
- removed link 6_link
- removed link 7_link
- removed link 8_link
- removed link 9_link
- link 0_link: geometry collision cylinder length=0.1 radius=0.6; visual cylinder length=0.1 radius=0.6
- link 1_link: geometry collision cylinder length=0.9 radius=0.2; visual cylinder length=0.9 radius=0.2
- link base_link: geometry collision cylinder length=1 radius=0.6; visual cylinder length=1 radius=0.6
Joints:
- removed joint 10_11_joint
- removed joint 11_12_joint
- removed joint 12_13_joint
- removed joint 13_14_joint
- removed joint 14_15_joint
- removed joint 15_16_joint
- removed joint 16_17_joint
- removed joint 17_18_joint
- removed joint 18_19_joint
- removed joint 1_2_joint
- removed joint 2_3_joint
- removed joint 3_4_joint
- removed joint 4_5_joint
- removed joint 5_6_joint
- removed joint 6_7_joint
- removed joint 7_8_joint
- removed joint 8_9_joint
- removed joint 9_10_joint
- joint 0_1_joint: origin xyz=0 0 0.05 rpy=0 0 0 -> xyz=0 0 0.5 rpy=0 0 0

File: pybullet_data/shapes/4_middle.urdf (robot description, URDF)
Before this commit: robot 4_middle, 21 links, 20 joints
Links:
- removed link 10_link
- removed link 11_link
- removed link 12_link
- removed link 13_link
- removed link 14_link
- removed link 15_link
- removed link 16_link
- removed link 17_link
- removed link 18_link
- removed link 19_link
- removed link 3_link
- removed link 4_link
- removed link 5_link
- removed link 6_link
- removed link 7_link
- removed link 8_link
- removed link 9_link
- link 0_link: geometry collision cylinder length=0.45 radius=0.2; visual cylinder length=0.45 radius=0.2
- link 1_link: geometry collision cylinder length=0.1 radius=0.6; visual cylinder length=0.1 radius=0.6
- link 2_link: geometry collision cylinder length=0.45 radius=0.2; visual cylinder length=0.45 radius=0.2
- link base_link: geometry collision cylinder length=1 radius=0.6; visual cylinder length=1 radius=0.6
Joints:
- removed joint 10_11_joint
- removed joint 11_12_joint
- removed joint 12_13_joint
- removed joint 13_14_joint
- removed joint 14_15_joint
- removed joint 15_16_joint
- removed joint 16_17_joint
- removed joint 17_18_joint
- removed joint 18_19_joint
- removed joint 2_3_joint
- removed joint 3_4_joint
- removed joint 4_5_joint
- removed joint 5_6_joint
- removed joint 6_7_joint
- removed joint 7_8_joint
- removed joint 8_9_joint
- removed joint 9_10_joint
- joint 0_1_joint: origin xyz=0 0 0.05 rpy=0 0 0 -> xyz=0 0 0.275 rpy=0 0 0
- joint 1_2_joint: origin xyz=0 0 0.05 rpy=0 0 0 -> xyz=0 0 0.275 rpy=0 0 0
- joint base_0_joint: origin xyz=0 0 0.05 rpy=0 0 0 -> xyz=0 0 0.225 rpy=0 0 0

File: pybullet_data/shapes/5_top_bottom.urdf (robot description, URDF)
Before this commit: robot 5_top_bottom, 21 links, 20 joints
Links:
- removed link 10_link
- removed link 11_link
- removed link 12_link
- removed link 13_link
- removed link 14_link
- removed link 15_link
- removed link 16_link
- removed link 17_link
- removed link 18_link
- removed link 19_link
- removed link 3_link
- removed link 4_link
- removed link 5_link
- removed link 6_link
- removed link 7_link
- removed link 8_link
- removed link 9_link
- link 0_link: geometry collision cylinder length=0.1 radius=0.6; visual cylinder length=0.1 radius=0.6
- link 1_link: geometry collision cylinder length=0.8 radius=0.2; visual cylinder length=0.8 radius=0.2
- link 2_link: geometry collision cylinder length=0.1 radius=0.6; visual cylinder length=0.1 radius=0.6
- link base_link: geometry collision cylinder length=1 radius=0.6; visual cylinder length=1 radius=0.6
Joints:
- removed joint 10_11_joint
- removed joint 11_12_joint
- removed joint 12_13_joint
- removed joint 13_14_joint
- removed joint 14_15_joint
- removed joint 15_16_joint
- removed joint 16_17_joint
- removed joint 17_18_joint
- removed joint 18_19_joint
- removed joint 2_3_joint
- removed joint 3_4_joint
- removed joint 4_5_joint
- removed joint 5_6_joint
- removed joint 6_7_joint
- removed joint 7_8_joint
- removed joint 8_9_joint
- removed joint 9_10_joint
- joint 0_1_joint: origin xyz=0 0 0.05 rpy=0 0 0 -> xyz=0 0 0.45 rpy=0 0 0
- joint 1_2_joint: origin xyz=0 0 0.05 rpy=0 0 0 -> xyz=0 0 0.45 rpy=0 0 0

Commit message: working every-action-goal plotted

File: pybullet_data/robot.urdf (robot description, URDF)
Before this commit: robot robot, 8 links, 7 joints
Links:
- link left_arm_link: geometry collision box size=1 0.1 0.1; visual box size=1 0.1 0.1
- link left_hand_link: geometry collision box size=1 .1 .1; visual box size=1 .1 .1
- link right_arm_link: geometry collision box size=1 0.1 0.1; visual box size=1 0.1 0.1
- link right_hand_link: geometry collision box size=1 .1 .1; visual box size=1 .1 .1
Joints:
- joint left_arm_left_hand_joint: origin xyz=.5 0 0 rpy=0 0 0 -> xyz=1 0 0 rpy=0 0 0
- joint right_arm_right_hand_joint: origin xyz=.5 0 0 rpy=0 0 0 -> xyz=1 0 0 rpy=0 0 0

File: pybullet_data/shapes/2_T.urdf (robot description, URDF)
Before this commit: robot 5_top_bottom, 4 links, 3 joints
Links:
- removed link 2_link
- link 0_link: geometry collision cylinder length=0.9 radius=0.2; visual cylinder length=0.9 radius=0.2
- link 1_link: geometry collision cylinder length=0.1 radius=0.6; visual cylinder length=0.1 radius=0.6
Joints:
- removed joint 1_2_joint
- joint 0_1_joint: origin xyz=0 0 0.45 rpy=0 0 0 -> xyz=0 0 0.5 rpy=0 0 0
- joint base_0_joint: origin xyz=0 0 0.05 rpy=0 0 0 -> xyz=0 0 0.45 rpy=0 0 0

File: pybullet_data/shapes/5_I.urdf (robot description, URDF)
Before this commit: robot 2_top, 3 links, 2 joints
Links:
- added link 2_link, mass 1; collision cylinder length=0.1 radius=0.6; visual cylinder length=0.1 radius=0.6
- link 0_link: geometry collision cylinder length=0.1 radius=0.6; visual cylinder length=0.1 radius=0.6
- link 1_link: geometry collision cylinder length=0.8 radius=0.2; visual cylinder length=0.8 radius=0.2
Joints:
- added joint 1_2_joint: type fixed, parent 1_link, child 2_link, origin xyz=0 0 0.45 rpy=0 0 0
- joint 0_1_joint: origin xyz=0 0 0.5 rpy=0 0 0 -> xyz=0 0 0.45 rpy=0 0 0
- joint base_0_joint: origin xyz=0 0 0.45 rpy=0 0 0 -> xyz=0 0 0.05 rpy=0 0 0

Commit message: simplified

File: pybullet_data/robot.urdf (robot description, URDF)
Before this commit: robot robot, 8 links, 7 joints
Links:
- removed link left_arm_link
- removed link left_hand_link
- removed link left_shoulder_link
- removed link right_arm_link
- removed link right_hand_link
- removed link right_shoulder_link
- added link arm_link, mass 1; collision box size=2 0.1 0.1; visual box size=2 0.1 0.1
- added link hand_link, mass 1; collision box size=1 .1 .1; visual box size=1 .1 .1
- added link shoulder_link, mass 1; collision box size=.1 0.1 0.1; visual box size=.1 0.1 0.1
Joints:
- removed joint body_left_shoulder_joint
- removed joint body_right_shoulder_joint
- removed joint left_arm_left_hand_joint
- removed joint left_shoulder_left_arm_joint
- removed joint right_arm_right_hand_joint
- removed joint right_shoulder_right_arm_joint
- added joint arm_hand_joint: type fixed, parent arm_link, child hand_link, origin xyz=1.5 0 0 rpy=0 0 -1.5708
- added joint body_shoulder_joint: type continuous, parent body_link, child shoulder_link, origin xyz=0 .5 0 rpy=0 0 0, axis 0 1 0
- added joint shoulder_arm_joint: type prismatic, parent shoulder_link, child arm_link, origin xyz=0 0 0 rpy=0 0 0, axis 1 0 0, limit lower=-0.5 upper=0.5 effort=0 velocity=0

Commit message: simplified, trying to make better combinations

File: pybullet_data/robot.urdf (robot description, URDF)
Before this commit: robot robot, 5 links, 4 joints
Links:
- removed link hand_link
Joints:
- removed joint arm_hand_joint
- joint shoulder_arm_joint: limit lower=-0.5 upper=0.5 effort=0 velocity=0 -> (none); origin xyz=0 0 0 rpy=0 0 0 -> xyz=1 0 0 rpy=0 0 0; type prismatic -> fixed

Commit message: better image gen

File: pybullet_data/robot.urdf (robot description, URDF)
Before this commit: robot robot, 4 links, 3 joints
Joints:
- joint body_shoulder_joint: limit (none) -> lower=-1.57 upper=1.57 effort=99999 velocity=99999; type continuous -> revolute

Commit message: more natural

File: pybullet_data/robot.urdf (robot description, URDF)
Before this commit: robot robot, 4 links, 3 joints
Links:
- removed link arm_link
- removed link body_link
- removed link nose_link
- removed link shoulder_link
- added link arm, mass 0; collision box size=3 0.1 0.1; visual box size=3 0.1 0.1
- added link arm_sensor, mass 0; collision box size=3 0.11 0.11; visual box size=3 0.11 0.11
- added link body, mass 100; collision box size=1 1 1; visual box size=1 1 1
- added link body_sensor, mass 0; collision box size=1.21 1.01 1.01; visual box size=1.21 1.01 1.01
- added link hand, mass 0; collision box size=0.1 2 0.1; visual box size=0.1 2 0.1
- added link hand_sensor, mass 0; collision box size=0.11 2 0.11; visual box size=0.11 2 0.11
- added link nose, mass 0; collision box size=.2 .2 .2; visual box size=.2 .2 .2
- added link shoulder, mass 0; collision box size=.1 0.1 0.1; visual box size=.1 0.1 0.1
Joints:
- added joint arm_arm_sensor_joint: type fixed, parent arm, child arm_sensor, origin xyz=0 0 0 rpy=0 0 0, axis 0 0 0
- added joint arm_hand_joint: type fixed, parent arm, child hand, origin xyz=1.5 0 0 rpy=0 0 0, axis 0 0 1
- added joint body_body_sensor_joint: type fixed, parent body, child body_sensor, origin xyz=.1 0 0 rpy=0 0 0, axis 0 0 0
- added joint hand_hand_sensor_joint: type fixed, parent hand, child hand_sensor, origin xyz=0 0 0 rpy=0 0 0, axis 0 0 0
- joint body_nose_joint: child nose_link -> nose; parent body_link -> body
- joint body_shoulder_joint: axis 0 1 0 -> 0 -1 0; child shoulder_link -> shoulder; limit lower=-1.57 upper=1.57 effort=99999 velocity=99999 -> (none); parent body_link -> body; type revolute -> continuous
- joint shoulder_arm_joint: child arm_link -> arm; origin xyz=1 0 0 rpy=0 0 0 -> xyz=1.5 0 0 rpy=0 0 0; parent shoulder_link -> shoulder

Commit message: kind of working?

File: pybullet_data/robot.urdf (robot description, URDF)
Before this commit: robot robot, 11 links, 10 joints
Links:
- removed link nose
- added link arrow_0, mass 0; collision box size=0.05 0.5 0.001; visual box size=0.05 0.5 0.001
- added link arrow_1, mass 0; collision box size=0.05 0.45 0.001; visual box size=0.05 0.45 0.001
- added link arrow_2, mass 0; collision box size=0.05 0.4 0.001; visual box size=0.05 0.4 0.001
- added link arrow_3, mass 0; collision box size=0.05 0.35 0.001; visual box size=0.05 0.35 0.001
- added link arrow_4, mass 0; collision box size=0.05 0.3 0.001; visual box size=0.05 0.3 0.001
- added link arrow_5, mass 0; collision box size=0.05 0.25 0.001; visual box size=0.05 0.25 0.001
- added link arrow_6, mass 0; collision box size=0.05 0.19999999999999996 0.001; visual box size=0.05 0.19999999999999996 0.001
- added link arrow_7, mass 0; collision box size=0.05 0.14999999999999997 0.001; visual box size=0.05 0.14999999999999997 0.001
- added link arrow_8, mass 0; collision box size=0.05 0.09999999999999998 0.001; visual box size=0.05 0.09999999999999998 0.001
- added link arrow_9, mass 0; collision box size=0.05 0.04999999999999999 0.001; visual box size=0.05 0.04999999999999999 0.001
- added link arrow_base, mass 0; collision box size=0.4 0.2 0.001; visual box size=0.4 0.2 0.001
- link hand: geometry collision box size=0.4 1.6 0.8; visual box size=0.4 1.6 0.8
- link hand_sensor: geometry collision box size=0.42000000000000004 1.62 0.8200000000000001; visual box size=0.42000000000000004 1.62 0.8200000000000001
- link left_arm: geometry collision box size=3 0.4 0.8; visual box size=3 0.4 0.8
- link left_arm_sensor: geometry collision box size=3.02 0.42000000000000004 0.8200000000000001; visual box size=3.02 0.42000000000000004 0.8200000000000001
- link left_shoulder: geometry collision box size=0.4 0.5 0.8; visual box size=0.4 0.5 0.8
- link right_arm: geometry collision box size=3 0.4 0.8; visual box size=3 0.4 0.8
- link right_arm_sensor: geometry collision box size=3.02 0.42000000000000004 0.8200000000000001; visual box size=3.02 0.42000000000000004 0.8200000000000001
- link right_shoulder: geometry collision box size=0.4 0.5 0.8; visual box size=0.4 0.5 0.8
Joints:
- removed joint body_nose_joint
- added joint arrow_0_arrow_1_joint: type fixed, parent arrow_0, child arrow_1, origin xyz=0.025 0 0 rpy=0 0 0, axis 0 0 1
- added joint arrow_1_arrow_2_joint: type fixed, parent arrow_1, child arrow_2, origin xyz=0.025 0 0 rpy=0 0 0, axis 0 0 1
- added joint arrow_2_arrow_3_joint: type fixed, parent arrow_2, child arrow_3, origin xyz=0.025 0 0 rpy=0 0 0, axis 0 0 1
- added joint arrow_3_arrow_4_joint: type fixed, parent arrow_3, child arrow_4, origin xyz=0.025 0 0 rpy=0 0 0, axis 0 0 1
- added joint arrow_4_arrow_5_joint: type fixed, parent arrow_4, child arrow_5, origin xyz=0.025 0 0 rpy=0 0 0, axis 0 0 1
- added joint arrow_5_arrow_6_joint: type fixed, parent arrow_5, child arrow_6, origin xyz=0.025 0 0 rpy=0 0 0, axis 0 0 1
- added joint arrow_6_arrow_7_joint: type fixed, parent arrow_6, child arrow_7, origin xyz=0.025 0 0 rpy=0 0 0, axis 0 0 1
- added joint arrow_7_arrow_8_joint: type fixed, parent arrow_7, child arrow_8, origin xyz=0.025 0 0 rpy=0 0 0, axis 0 0 1
- added joint arrow_8_arrow_9_joint: type fixed, parent arrow_8, child arrow_9, origin xyz=0.025 0 0 rpy=0 0 0, axis 0 0 1
- added joint arrow_base_arrow_0_joint: type fixed, parent arrow_base, child arrow_0, origin xyz=0.2 0 0 rpy=0 0 0, axis 0 0 1
- added joint body_arrow_base_joint: type fixed, parent body, child arrow_base, origin xyz=-0.15 0 0.50000001 rpy=0 0 0, axis 0 0 1
- joint hand_right_arm_joint: origin xyz=-1.5 -1 0 rpy=0 0 0 -> xyz=-1.3 -1 0 rpy=0 0 0
- joint left_arm_hand_joint: origin xyz=1.5 -1 0 rpy=0 0 0 -> xyz=1.3 -1 0 rpy=0 0 0
- joint left_shoulder_left_arm_joint: origin xyz=1.45 0.25 0 rpy=0 0 0 -> xyz=1.3 0.25 0 rpy=0 0 0
- joint right_arm_right_shoulder_joint: origin xyz=-1.45 0.25 0 rpy=0 0 0 -> xyz=-1.3 0.25 0 rpy=0 0 0

Commit message: Working? :O

File: pybullet_data/robot.urdf (robot description, URDF)
Before this commit: robot robot, 21 links, 20 joints
Links:
- removed link body_sensor
- removed link hand_sensor
- removed link left_arm_sensor
- removed link right_arm_sensor
- added link body_sensor_0, mass 0; collision box size=1.02 1.02 1.02; visual box size=1.02 1.02 1.02
- added link hand_sensor_0, mass 0; collision box size=0.42000000000000004 0.8200000000000001 0.8200000000000001; visual box size=0.42000000000000004 0.8200000000000001 0.8200000000000001
- added link hand_sensor_1, mass 0; collision box size=0.42000000000000004 0.8200000000000001 0.8200000000000001; visual box size=0.42000000000000004 0.8200000000000001 0.8200000000000001
- added link left_arm_sensor_0, mass 0; collision box size=1.02 0.42000000000000004 0.8200000000000001; visual box size=1.02 0.42000000000000004 0.8200000000000001
- added link left_arm_sensor_1, mass 0; collision box size=1.02 0.42000000000000004 0.8200000000000001; visual box size=1.02 0.42000000000000004 0.8200000000000001
- added link left_arm_sensor_2, mass 0; collision box size=1.02 0.42000000000000004 0.8200000000000001; visual box size=1.02 0.42000000000000004 0.8200000000000001
- added link right_arm_sensor_0, mass 0; collision box size=1.02 0.42000000000000004 0.8200000000000001; visual box size=1.02 0.42000000000000004 0.8200000000000001
- added link right_arm_sensor_1, mass 0; collision box size=1.02 0.42000000000000004 0.8200000000000001; visual box size=1.02 0.42000000000000004 0.8200000000000001
- added link right_arm_sensor_2, mass 0; collision box size=1.02 0.42000000000000004 0.8200000000000001; visual box size=1.02 0.42000000000000004 0.8200000000000001
Joints:
- removed joint body_body_sensor_joint
- removed joint hand_hand_sensor_joint
- removed joint left_arm_left_arm_sensor_joint
- removed joint right_arm_right_arm_sensor_joint
- added joint body_body_sensor_0_joint: type fixed, parent body, child body_sensor_0, origin xyz=0 0 0 rpy=0 0 0, axis 0 0 0
- added joint hand_hand_sensor_0_joint: type fixed, parent hand, child hand_sensor_0, origin xyz=0 -0.4 0 rpy=0 0 0, axis 0 0 0
- added joint hand_sensor_0_hand_sensor_1_joint: type fixed, parent hand_sensor_0, child hand_sensor_1, origin xyz=0 0.8 0 rpy=0 0 0, axis 0 0 0
- added joint left_arm_left_arm_sensor_0_joint: type fixed, parent left_arm, child left_arm_sensor_0, origin xyz=-1.0 0 0 rpy=0 0 0, axis 0 0 0
- added joint left_arm_sensor_0_left_arm_sensor_1_joint: type fixed, parent left_arm_sensor_0, child left_arm_sensor_1, origin xyz=1.0 0 0 rpy=0 0 0, axis 0 0 0
- added joint left_arm_sensor_1_left_arm_sensor_2_joint: type fixed, parent left_arm_sensor_1, child left_arm_sensor_2, origin xyz=1.0 0 0 rpy=0 0 0, axis 0 0 0
- added joint right_arm_right_arm_sensor_0_joint: type fixed, parent right_arm, child right_arm_sensor_0, origin xyz=-1.0 0 0 rpy=0 0 0, axis 0 0 0
- added joint right_arm_sensor_0_right_arm_sensor_1_joint: type fixed, parent right_arm_sensor_0, child right_arm_sensor_1, origin xyz=1.0 0 0 rpy=0 0 0, axis 0 0 0
- added joint right_arm_sensor_1_right_arm_sensor_2_joint: type fixed, parent right_arm_sensor_1, child right_arm_sensor_2, origin xyz=1.0 0 0 rpy=0 0 0, axis 0 0 0
