Commit message: better test_agent

File: pybullet_data/robot.urdf (robot description, URDF)
Before this commit: robot robot, 26 links, 25 joints
Links:
- removed link body_sensor_0
- removed link hand_sensor_0
- removed link hand_sensor_1
- removed link left_arm_sensor_0
- removed link left_arm_sensor_1
- removed link left_arm_sensor_2
- removed link right_arm_sensor_0
- removed link right_arm_sensor_1
- removed link right_arm_sensor_2
- added link body_sensor_0_bottom, mass 0; collision box size=1.0 1 0.02; visual box size=1.0 1 0.02
- added link body_sensor_0_left, mass 0; collision box size=1.0 0.02 1; visual box size=1.0 0.02 1
- added link body_sensor_0_right, mass 0; collision box size=1.0 0.02 1; visual box size=1.0 0.02 1
- added link body_sensor_0_start, mass 0; collision box size=0.02 1 1; visual box size=0.02 1 1
- added link body_sensor_0_stop, mass 0; collision box size=0.02 1 1; visual box size=0.02 1 1
- added link body_sensor_0_top, mass 0; collision box size=1.0 1 0.02; visual box size=1.0 1 0.02
- added link hand_sensor_0_bottom, mass 0; collision box size=0.02 0.8 0.8; visual box size=0.02 0.8 0.8
- added link hand_sensor_0_left, mass 0; collision box size=0.4 0.8 0.02; visual box size=0.4 0.8 0.02
- added link hand_sensor_0_right, mass 0; collision box size=0.4 0.8 0.02; visual box size=0.4 0.8 0.02
- added link hand_sensor_0_top, mass 0; collision box size=0.02 0.8 0.8; visual box size=0.02 0.8 0.8
- added link hand_sensor_1_bottom, mass 0; collision box size=0.02 0.8 0.8; visual box size=0.02 0.8 0.8
- added link hand_sensor_1_left, mass 0; collision box size=0.4 0.8 0.02; visual box size=0.4 0.8 0.02
- added link hand_sensor_1_right, mass 0; collision box size=0.4 0.8 0.02; visual box size=0.4 0.8 0.02
- added link hand_sensor_1_top, mass 0; collision box size=0.02 0.8 0.8; visual box size=0.02 0.8 0.8
- added link left_arm_sensor_0_bottom, mass 0; collision box size=1.0 0.4 0.02; visual box size=1.0 0.4 0.02
- added link left_arm_sensor_0_left, mass 0; collision box size=1.0 0.02 0.8; visual box size=1.0 0.02 0.8
- added link left_arm_sensor_0_right, mass 0; collision box size=1.0 0.02 0.8; visual box size=1.0 0.02 0.8
- added link left_arm_sensor_0_start, mass 0; collision box size=0.02 0.4 0.8; visual box size=0.02 0.4 0.8
- added link left_arm_sensor_0_top, mass 0; collision box size=1.0 0.4 0.02; visual box size=1.0 0.4 0.02
- added link left_arm_sensor_1_bottom, mass 0; collision box size=1.0 0.4 0.02; visual box size=1.0 0.4 0.02
- added link left_arm_sensor_1_left, mass 0; collision box size=1.0 0.02 0.8; visual box size=1.0 0.02 0.8
- added link left_arm_sensor_1_right, mass 0; collision box size=1.0 0.02 0.8; visual box size=1.0 0.02 0.8
- added link left_arm_sensor_1_top, mass 0; collision box size=1.0 0.4 0.02; visual box size=1.0 0.4 0.02
- added link left_arm_sensor_2_bottom, mass 0; collision box size=1.0 0.4 0.02; visual box size=1.0 0.4 0.02
- added link left_arm_sensor_2_left, mass 0; collision box size=1.0 0.02 0.8; visual box size=1.0 0.02 0.8
- added link left_arm_sensor_2_right, mass 0; collision box size=1.0 0.02 0.8; visual box size=1.0 0.02 0.8
- added link left_arm_sensor_2_stop, mass 0; collision box size=0.02 0.4 0.8; visual box size=0.02 0.4 0.8
- added link left_arm_sensor_2_top, mass 0; collision box size=1.0 0.4 0.02; visual box size=1.0 0.4 0.02
- added link right_arm_sensor_0_bottom, mass 0; collision box size=1.0 0.4 0.02; visual box size=1.0 0.4 0.02
- added link right_arm_sensor_0_left, mass 0; collision box size=1.0 0.02 0.8; visual box size=1.0 0.02 0.8
- added link right_arm_sensor_0_right, mass 0; collision box size=1.0 0.02 0.8; visual box size=1.0 0.02 0.8
- added link right_arm_sensor_0_start, mass 0; collision box size=0.02 0.4 0.8; visual box size=0.02 0.4 0.8
- added link right_arm_sensor_0_top, mass 0; collision box size=1.0 0.4 0.02; visual box size=1.0 0.4 0.02
- added link right_arm_sensor_1_bottom, mass 0; collision box size=1.0 0.4 0.02; visual box size=1.0 0.4 0.02
- added link right_arm_sensor_1_left, mass 0; collision box size=1.0 0.02 0.8; visual box size=1.0 0.02 0.8
- added link right_arm_sensor_1_right, mass 0; collision box size=1.0 0.02 0.8; visual box size=1.0 0.02 0.8
- added link right_arm_sensor_1_top, mass 0; collision box size=1.0 0.4 0.02; visual box size=1.0 0.4 0.02
- added link right_arm_sensor_2_bottom, mass 0; collision box size=1.0 0.4 0.02; visual box size=1.0 0.4 0.02
- added link right_arm_sensor_2_left, mass 0; collision box size=1.0 0.02 0.8; visual box size=1.0 0.02 0.8
- added link right_arm_sensor_2_right, mass 0; collision box size=1.0 0.02 0.8; visual box size=1.0 0.02 0.8
- added link right_arm_sensor_2_stop, mass 0; collision box size=0.02 0.4 0.8; visual box size=0.02 0.4 0.8
- added link right_arm_sensor_2_top, mass 0; collision box size=1.0 0.4 0.02; visual box size=1.0 0.4 0.02
- link arrow_base: geometry collision box size=0.3 0.2 0.001; visual box size=0.3 0.2 0.001
- link left_shoulder: geometry collision box size=0.4 0.3 0.8; visual box size=0.4 0.3 0.8
- link right_shoulder: geometry collision box size=0.4 0.3 0.8; visual box size=0.4 0.3 0.8
Joints:
- removed joint body_body_sensor_0_joint
- removed joint hand_hand_sensor_0_joint
- removed joint hand_sensor_0_hand_sensor_1_joint
- removed joint left_arm_left_arm_sensor_0_joint
- removed joint left_arm_sensor_0_left_arm_sensor_1_joint
- removed joint left_arm_sensor_1_left_arm_sensor_2_joint
- removed joint right_arm_right_arm_sensor_0_joint
- removed joint right_arm_sensor_0_right_arm_sensor_1_joint
- removed joint right_arm_sensor_1_right_arm_sensor_2_joint
- added joint body_body_sensor_0_bottom_joint: type fixed, parent body, child body_sensor_0_bottom, origin xyz=0 0 -0.5 rpy=0 0 0, axis 1 0 0
- added joint body_body_sensor_0_left_joint: type fixed, parent body, child body_sensor_0_left, origin xyz=0 0.5 0 rpy=0 0 0, axis 1 0 0
- added joint body_body_sensor_0_right_joint: type fixed, parent body, child body_sensor_0_right, origin xyz=0 -0.5 0 rpy=0 0 0, axis 1 0 0
- added joint body_body_sensor_0_start_joint: type fixed, parent body, child body_sensor_0_start, origin xyz=0.5 0 0 rpy=0 0 0, axis 1 0 0
- added joint body_body_sensor_0_stop_joint: type fixed, parent body, child body_sensor_0_stop, origin xyz=-0.5 0 0 rpy=0 0 0, axis 1 0 0
- added joint body_body_sensor_0_top_joint: type fixed, parent body, child body_sensor_0_top, origin xyz=0 0 0.5 rpy=0 0 0, axis 1 0 0
- added joint hand_hand_sensor_0_bottom_joint: type fixed, parent hand, child hand_sensor_0_bottom, origin xyz=-0.2 -0.4 0 rpy=0 0 0, axis 0 0 0
- added joint hand_hand_sensor_0_left_joint: type fixed, parent hand, child hand_sensor_0_left, origin xyz=0 -0.4 0.4 rpy=0 0 0, axis 0 0 0
- added joint hand_hand_sensor_0_right_joint: type fixed, parent hand, child hand_sensor_0_right, origin xyz=0 -0.4 -0.4 rpy=0 0 0, axis 0 0 0
- added joint hand_hand_sensor_0_top_joint: type fixed, parent hand, child hand_sensor_0_top, origin xyz=0.2 -0.4 0 rpy=0 0 0, axis 0 0 0
- added joint hand_hand_sensor_1_bottom_joint: type fixed, parent hand, child hand_sensor_1_bottom, origin xyz=-0.2 0.4 0 rpy=0 0 0, axis 0 0 0
- added joint hand_hand_sensor_1_left_joint: type fixed, parent hand, child hand_sensor_1_left, origin xyz=0 0.4 0.4 rpy=0 0 0, axis 0 0 0
- added joint hand_hand_sensor_1_right_joint: type fixed, parent hand, child hand_sensor_1_right, origin xyz=0 0.4 -0.4 rpy=0 0 0, axis 0 0 0
- added joint hand_hand_sensor_1_top_joint: type fixed, parent hand, child hand_sensor_1_top, origin xyz=0.2 0.4 0 rpy=0 0 0, axis 0 0 0
- added joint left_arm_left_arm_sensor_0_bottom_joint: type fixed, parent left_arm, child left_arm_sensor_0_bottom, origin xyz=-1.0 0 -0.4 rpy=0 0 0, axis 1 0 0
- added joint left_arm_left_arm_sensor_0_left_joint: type fixed, parent left_arm, child left_arm_sensor_0_left, origin xyz=-1.0 0.2 0 rpy=0 0 0, axis 1 0 0
- added joint left_arm_left_arm_sensor_0_right_joint: type fixed, parent left_arm, child left_arm_sensor_0_right, origin xyz=-1.0 -0.2 0 rpy=0 0 0, axis 1 0 0
- added joint left_arm_left_arm_sensor_0_start_joint: type fixed, parent left_arm, child left_arm_sensor_0_start, origin xyz=1.5 0 0 rpy=0 0 0, axis 1 0 0
- added joint left_arm_left_arm_sensor_0_top_joint: type fixed, parent left_arm, child left_arm_sensor_0_top, origin xyz=-1.0 0 0.4 rpy=0 0 0, axis 1 0 0
- added joint left_arm_left_arm_sensor_1_bottom_joint: type fixed, parent left_arm, child left_arm_sensor_1_bottom, origin xyz=0.0 0 -0.4 rpy=0 0 0, axis 1 0 0
- added joint left_arm_left_arm_sensor_1_left_joint: type fixed, parent left_arm, child left_arm_sensor_1_left, origin xyz=0.0 0.2 0 rpy=0 0 0, axis 1 0 0
- added joint left_arm_left_arm_sensor_1_right_joint: type fixed, parent left_arm, child left_arm_sensor_1_right, origin xyz=0.0 -0.2 0 rpy=0 0 0, axis 1 0 0
- added joint left_arm_left_arm_sensor_1_top_joint: type fixed, parent left_arm, child left_arm_sensor_1_top, origin xyz=0.0 0 0.4 rpy=0 0 0, axis 1 0 0
- added joint left_arm_left_arm_sensor_2_bottom_joint: type fixed, parent left_arm, child left_arm_sensor_2_bottom, origin xyz=1.0 0 -0.4 rpy=0 0 0, axis 1 0 0
- added joint left_arm_left_arm_sensor_2_left_joint: type fixed, parent left_arm, child left_arm_sensor_2_left, origin xyz=1.0 0.2 0 rpy=0 0 0, axis 1 0 0
- added joint left_arm_left_arm_sensor_2_right_joint: type fixed, parent left_arm, child left_arm_sensor_2_right, origin xyz=1.0 -0.2 0 rpy=0 0 0, axis 1 0 0
- added joint left_arm_left_arm_sensor_2_stop_joint: type fixed, parent left_arm, child left_arm_sensor_2_stop, origin xyz=-1.5 0 0 rpy=0 0 0, axis 1 0 0
- added joint left_arm_left_arm_sensor_2_top_joint: type fixed, parent left_arm, child left_arm_sensor_2_top, origin xyz=1.0 0 0.4 rpy=0 0 0, axis 1 0 0
- added joint right_arm_right_arm_sensor_0_bottom_joint: type fixed, parent right_arm, child right_arm_sensor_0_bottom, origin xyz=-1.0 0 -0.4 rpy=0 0 0, axis 1 0 0
- added joint right_arm_right_arm_sensor_0_left_joint: type fixed, parent right_arm, child right_arm_sensor_0_left, origin xyz=-1.0 0.2 0 rpy=0 0 0, axis 1 0 0
- added joint right_arm_right_arm_sensor_0_right_joint: type fixed, parent right_arm, child right_arm_sensor_0_right, origin xyz=-1.0 -0.2 0 rpy=0 0 0, axis 1 0 0
- added joint right_arm_right_arm_sensor_0_start_joint: type fixed, parent right_arm, child right_arm_sensor_0_start, origin xyz=1.5 0 0 rpy=0 0 0, axis 1 0 0
- added joint right_arm_right_arm_sensor_0_top_joint: type fixed, parent right_arm, child right_arm_sensor_0_top, origin xyz=-1.0 0 0.4 rpy=0 0 0, axis 1 0 0
- added joint right_arm_right_arm_sensor_1_bottom_joint: type fixed, parent right_arm, child right_arm_sensor_1_bottom, origin xyz=0.0 0 -0.4 rpy=0 0 0, axis 1 0 0
- added joint right_arm_right_arm_sensor_1_left_joint: type fixed, parent right_arm, child right_arm_sensor_1_left, origin xyz=0.0 0.2 0 rpy=0 0 0, axis 1 0 0
- added joint right_arm_right_arm_sensor_1_right_joint: type fixed, parent right_arm, child right_arm_sensor_1_right, origin xyz=0.0 -0.2 0 rpy=0 0 0, axis 1 0 0
- added joint right_arm_right_arm_sensor_1_top_joint: type fixed, parent right_arm, child right_arm_sensor_1_top, origin xyz=0.0 0 0.4 rpy=0 0 0, axis 1 0 0
- added joint right_arm_right_arm_sensor_2_bottom_joint: type fixed, parent right_arm, child right_arm_sensor_2_bottom, origin xyz=1.0 0 -0.4 rpy=0 0 0, axis 1 0 0
- added joint right_arm_right_arm_sensor_2_left_joint: type fixed, parent right_arm, child right_arm_sensor_2_left, origin xyz=1.0 0.2 0 rpy=0 0 0, axis 1 0 0
- added joint right_arm_right_arm_sensor_2_right_joint: type fixed, parent right_arm, child right_arm_sensor_2_right, origin xyz=1.0 -0.2 0 rpy=0 0 0, axis 1 0 0
- added joint right_arm_right_arm_sensor_2_stop_joint: type fixed, parent right_arm, child right_arm_sensor_2_stop, origin xyz=-1.5 0 0 rpy=0 0 0, axis 1 0 0
- added joint right_arm_right_arm_sensor_2_top_joint: type fixed, parent right_arm, child right_arm_sensor_2_top, origin xyz=1.0 0 0.4 rpy=0 0 0, axis 1 0 0
- joint arrow_0_arrow_1_joint: origin xyz=0.025 0 0 rpy=0 0 0 -> xyz=0.05 0 0 rpy=0 0 0
- joint arrow_1_arrow_2_joint: origin xyz=0.025 0 0 rpy=0 0 0 -> xyz=0.05 0 0 rpy=0 0 0
- joint arrow_2_arrow_3_joint: origin xyz=0.025 0 0 rpy=0 0 0 -> xyz=0.05 0 0 rpy=0 0 0
- joint arrow_3_arrow_4_joint: origin xyz=0.025 0 0 rpy=0 0 0 -> xyz=0.05 0 0 rpy=0 0 0
- joint arrow_4_arrow_5_joint: origin xyz=0.025 0 0 rpy=0 0 0 -> xyz=0.05 0 0 rpy=0 0 0
- joint arrow_5_arrow_6_joint: origin xyz=0.025 0 0 rpy=0 0 0 -> xyz=0.05 0 0 rpy=0 0 0
- joint arrow_6_arrow_7_joint: origin xyz=0.025 0 0 rpy=0 0 0 -> xyz=0.05 0 0 rpy=0 0 0
- joint arrow_7_arrow_8_joint: origin xyz=0.025 0 0 rpy=0 0 0 -> xyz=0.05 0 0 rpy=0 0 0
- joint arrow_8_arrow_9_joint: origin xyz=0.025 0 0 rpy=0 0 0 -> xyz=0.05 0 0 rpy=0 0 0
- joint arrow_base_arrow_0_joint: origin xyz=0.2 0 0 rpy=0 0 0 -> xyz=0.15 0 0 rpy=0 0 0
- joint body_arrow_base_joint: origin xyz=-0.15 0 0.50000001 rpy=0 0 0 -> xyz=-0.24999999999999997 0 0.50000001 rpy=0 0 0
- joint body_left_shoulder_joint: origin xyz=0 0.75 0 rpy=0 0 0 -> xyz=0 0.65 0 rpy=0 0 0
- joint left_shoulder_left_arm_joint: origin xyz=1.3 0.25 0 rpy=0 0 0 -> xyz=1.3 0.35 0 rpy=0 0 0
- joint right_arm_right_shoulder_joint: origin xyz=-1.3 0.25 0 rpy=0 0 0 -> xyz=-1.3 0.35 0 rpy=0 0 0

Commit message: awesome sensor-plots

File: pybullet_data/robot.urdf (robot description, URDF)
Before this commit: robot robot, 59 links, 58 joints
Links:
- removed link body_sensor_0_bottom
Joints:
- removed joint body_body_sensor_0_bottom_joint

Commit message: 2024_12_07, trying batchnorms again, and multi-step working (big test)

File: pybullet_data/robot.urdf (robot description, URDF)
Before this commit: robot robot, 72 links, 71 joints
Joints:
- joint left_arm_left_hand_joint: axis 0 0 0 -> 0 0 1
- joint left_hand_left_hand_sensor_0_bottom_joint: axis 0 0 0 -> 0 0 1
- joint left_hand_left_hand_sensor_0_left_joint: axis 0 0 0 -> 0 0 1
- joint left_hand_left_hand_sensor_0_right_joint: axis 0 0 0 -> 0 0 1
- joint left_hand_left_hand_sensor_0_stop_joint: axis 0 0 0 -> 0 0 1
- joint left_hand_left_hand_sensor_0_top_joint: axis 0 0 0 -> 0 0 1

File: robot.urdf (robot description, URDF)
Before this commit: robot robot, 72 links, 71 joints
Joints:
- joint left_arm_left_hand_joint: axis 0 0 0 -> 0 0 1
- joint left_hand_left_hand_sensor_0_bottom_joint: axis 0 0 0 -> 0 0 1
- joint left_hand_left_hand_sensor_0_left_joint: axis 0 0 0 -> 0 0 1
- joint left_hand_left_hand_sensor_0_right_joint: axis 0 0 0 -> 0 0 1
- joint left_hand_left_hand_sensor_0_stop_joint: axis 0 0 0 -> 0 0 1
- joint left_hand_left_hand_sensor_0_top_joint: axis 0 0 0 -> 0 0 1
- joint right_arm_right_hand_joint: axis 0 0 0 -> 0 0 1
- joint right_hand_right_hand_sensor_0_bottom_joint: axis 0 0 0 -> 0 0 1
- joint right_hand_right_hand_sensor_0_left_joint: axis 0 0 0 -> 0 0 1
- joint right_hand_right_hand_sensor_0_right_joint: axis 0 0 0 -> 0 0 1
- joint right_hand_right_hand_sensor_0_start_joint: axis 0 0 0 -> 0 0 1
- joint right_hand_right_hand_sensor_0_top_joint: axis 0 0 0 -> 0 0 1

Commit message: 2024_12_17, testing continuousness (big test)

File: pybullet_data/robot.urdf (robot description, URDF)
Before this commit: robot robot, 72 links, 71 joints
Joints:
- joint right_arm_right_hand_joint: axis 0 0 0 -> 0 0 1
- joint right_hand_right_hand_sensor_0_bottom_joint: axis 0 0 0 -> 0 0 1
- joint right_hand_right_hand_sensor_0_left_joint: axis 0 0 0 -> 0 0 1
- joint right_hand_right_hand_sensor_0_right_joint: axis 0 0 0 -> 0 0 1
- joint right_hand_right_hand_sensor_0_start_joint: axis 0 0 0 -> 0 0 1
- joint right_hand_right_hand_sensor_0_top_joint: axis 0 0 0 -> 0 0 1
