Commit message: 2025_01_15, not working, but new robot

File: pybullet_data/robot.urdf (robot description, URDF)
Before this commit: robot robot, 72 links, 71 joints
Links:
- removed link body_sensor_0_left
- removed link body_sensor_0_right
- removed link body_sensor_0_start
- removed link body_sensor_0_stop
- removed link body_sensor_0_top
- removed link body_square_0
- removed link body_square_1
- removed link body_square_10
- removed link body_square_11
- removed link body_square_12
- removed link body_square_13
- removed link body_square_14
- removed link body_square_15
- removed link body_square_16
- removed link body_square_17
- removed link body_square_18
- removed link body_square_19
- removed link body_square_2
- removed link body_square_20
- removed link body_square_21
- removed link body_square_3
- removed link body_square_4
- removed link body_square_5
- removed link body_square_6
- removed link body_square_7
- removed link body_square_8
- removed link body_square_9
- removed link left_arm
- removed link left_arm_sensor_0_bottom
- removed link left_arm_sensor_0_left
- removed link left_arm_sensor_0_right
- removed link left_arm_sensor_0_start
- removed link left_arm_sensor_0_top
- removed link left_arm_sensor_1_bottom
- removed link left_arm_sensor_1_left
- removed link left_arm_sensor_1_right
- removed link left_arm_sensor_1_top
- removed link left_arm_sensor_2_bottom
- removed link left_arm_sensor_2_left
- removed link left_arm_sensor_2_right
- removed link left_arm_sensor_2_stop
- removed link left_arm_sensor_2_top
- removed link left_hand
- removed link left_hand_sensor_0_bottom
- removed link left_hand_sensor_0_left
- removed link left_hand_sensor_0_right
- removed link left_hand_sensor_0_stop
- removed link left_hand_sensor_0_top
- removed link left_shoulder
- removed link right_arm
- removed link right_arm_sensor_0_bottom
- removed link right_arm_sensor_0_left
- removed link right_arm_sensor_0_right
- removed link right_arm_sensor_0_start
- removed link right_arm_sensor_0_top
- removed link right_arm_sensor_1_bottom
- removed link right_arm_sensor_1_left
- removed link right_arm_sensor_1_right
- removed link right_arm_sensor_1_top
- removed link right_arm_sensor_2_bottom
- removed link right_arm_sensor_2_left
- removed link right_arm_sensor_2_right
- removed link right_arm_sensor_2_stop
- removed link right_arm_sensor_2_top
- removed link right_hand
- removed link right_hand_sensor_0_bottom
- removed link right_hand_sensor_0_left
- removed link right_hand_sensor_0_right
- removed link right_hand_sensor_0_start
- removed link right_hand_sensor_0_top
- removed link right_shoulder
- added link arm_1, mass 0.1; collision box size=0.1 0.1 1; visual box size=0.1 0.1 1
- added link arm_2, mass 0.1; collision box size=0.1 0.1 0.75; visual box size=0.1 0.1 0.75
- added link base, mass 100; collision cylinder length=0.1 radius=0.75; visual cylinder length=0.1 radius=0.75
- added link body_face_0, mass 0; collision box size=0.002 0.1111111111111111 0.1111111111111111; visual box size=0.002 0.1111111111111111 0.1111111111111111
- added link body_face_1, mass 0; collision box size=0.002 0.1111111111111111 0.1111111111111111; visual box size=0.002 0.1111111111111111 0.1111111111111111
- added link body_face_10, mass 0; collision box size=0.1111111111111111 0.1111111111111111 0.002; visual box size=0.1111111111111111 0.1111111111111111 0.002
- added link body_face_11, mass 0; collision box size=0.1111111111111111 0.1111111111111111 0.002; visual box size=0.1111111111111111 0.1111111111111111 0.002
- added link body_face_12, mass 0; collision box size=0.1111111111111111 0.1111111111111111 0.002; visual box size=0.1111111111111111 0.1111111111111111 0.002
- added link body_face_13, mass 0; collision box size=0.1111111111111111 0.1111111111111111 0.002; visual box size=0.1111111111111111 0.1111111111111111 0.002
- added link body_face_14, mass 0; collision box size=0.1111111111111111 0.1111111111111111 0.002; visual box size=0.1111111111111111 0.1111111111111111 0.002
- added link body_face_15, mass 0; collision box size=0.1111111111111111 0.1111111111111111 0.002; visual box size=0.1111111111111111 0.1111111111111111 0.002
- added link body_face_16, mass 0; collision box size=0.1111111111111111 0.1111111111111111 0.002; visual box size=0.1111111111111111 0.1111111111111111 0.002
- added link body_face_17, mass 0; collision box size=0.1111111111111111 0.1111111111111111 0.002; visual box size=0.1111111111111111 0.1111111111111111 0.002
- added link body_face_18, mass 0; collision box size=0.1111111111111111 0.1111111111111111 0.002; visual box size=0.1111111111111111 0.1111111111111111 0.002
- added link body_face_19, mass 0; collision box size=0.1111111111111111 0.1111111111111111 0.002; visual box size=0.1111111111111111 0.1111111111111111 0.002
- added link body_face_2, mass 0; collision box size=0.002 0.1111111111111111 0.1111111111111111; visual box size=0.002 0.1111111111111111 0.1111111111111111
- added link body_face_20, mass 0; collision box size=0.1111111111111111 0.1111111111111111 0.002; visual box size=0.1111111111111111 0.1111111111111111 0.002
- added link body_face_21, mass 0; collision box size=0.1111111111111111 0.1111111111111111 0.002; visual box size=0.1111111111111111 0.1111111111111111 0.002
- added link body_face_3, mass 0; collision box size=0.002 0.1111111111111111 0.1111111111111111; visual box size=0.002 0.1111111111111111 0.1111111111111111
- added link body_face_4, mass 0; collision box size=0.002 0.1111111111111111 0.1111111111111111; visual box size=0.002 0.1111111111111111 0.1111111111111111
- added link body_face_5, mass 0; collision box size=0.002 0.1111111111111111 0.1111111111111111; visual box size=0.002 0.1111111111111111 0.1111111111111111
- added link body_face_6, mass 0; collision box size=0.002 0.1111111111111111 0.1111111111111111; visual box size=0.002 0.1111111111111111 0.1111111111111111
- added link body_face_7, mass 0; collision box size=0.002 0.1111111111111111 0.1111111111111111; visual box size=0.002 0.1111111111111111 0.1111111111111111
- added link body_face_8, mass 0; collision box size=0.002 0.1111111111111111 0.1111111111111111; visual box size=0.002 0.1111111111111111 0.1111111111111111
- added link body_face_9, mass 0; collision box size=0.1111111111111111 0.1111111111111111 0.002; visual box size=0.1111111111111111 0.1111111111111111 0.002
- added link elbow_pitch, mass 0.1; collision box size=0.1 0.1 0.1; visual box size=0.1 0.1 0.1
- added link hand_0, mass 0.1; collision box size=0.5 0.46411047216403317 0.1; visual box size=0.5 0.46411047216403317 0.1
- added link hand_0_sensor_0_bottom, mass 0; collision box size=0.5 0.46411047216403317 0.02; visual box size=0.5 0.46411047216403317 0.02
- added link hand_0_sensor_0_start, mass 0; collision box size=0.02 0.46411047216403317 0.1; visual box size=0.02 0.46411047216403317 0.1
- added link hand_0_sensor_0_stop, mass 0; collision box size=0.02 0.46411047216403317 0.1; visual box size=0.02 0.46411047216403317 0.1
- added link hand_0_sensor_0_top, mass 0; collision box size=0.5 0.46411047216403317 0.02; visual box size=0.5 0.46411047216403317 0.02
- added link hand_1, mass 0.1; collision box size=0.5 0.46411047216403317 0.1; visual box size=0.5 0.46411047216403317 0.1
- added link hand_10, mass 0.1; collision box size=0.5 0.46411047216403317 0.1; visual box size=0.5 0.46411047216403317 0.1
- added link hand_10_sensor_0_bottom, mass 0; collision box size=0.5 0.46411047216403317 0.02; visual box size=0.5 0.46411047216403317 0.02
- added link hand_10_sensor_0_start, mass 0; collision box size=0.02 0.46411047216403317 0.1; visual box size=0.02 0.46411047216403317 0.1
- added link hand_10_sensor_0_stop, mass 0; collision box size=0.02 0.46411047216403317 0.1; visual box size=0.02 0.46411047216403317 0.1
- added link hand_10_sensor_0_top, mass 0; collision box size=0.5 0.46411047216403317 0.02; visual box size=0.5 0.46411047216403317 0.02
- added link hand_11, mass 0.1; collision box size=0.5 0.46411047216403317 0.1; visual box size=0.5 0.46411047216403317 0.1
- added link hand_11_sensor_0_bottom, mass 0; collision box size=0.5 0.46411047216403317 0.02; visual box size=0.5 0.46411047216403317 0.02
- added link hand_11_sensor_0_start, mass 0; collision box size=0.02 0.46411047216403317 0.1; visual box size=0.02 0.46411047216403317 0.1
- added link hand_11_sensor_0_stop, mass 0; collision box size=0.02 0.46411047216403317 0.1; visual box size=0.02 0.46411047216403317 0.1
- added link hand_11_sensor_0_top, mass 0; collision box size=0.5 0.46411047216403317 0.02; visual box size=0.5 0.46411047216403317 0.02
- added link hand_1_sensor_0_bottom, mass 0; collision box size=0.5 0.46411047216403317 0.02; visual box size=0.5 0.46411047216403317 0.02
- added link hand_1_sensor_0_start, mass 0; collision box size=0.02 0.46411047216403317 0.1; visual box size=0.02 0.46411047216403317 0.1
- added link hand_1_sensor_0_stop, mass 0; collision box size=0.02 0.46411047216403317 0.1; visual box size=0.02 0.46411047216403317 0.1
- added link hand_1_sensor_0_top, mass 0; collision box size=0.5 0.46411047216403317 0.02; visual box size=0.5 0.46411047216403317 0.02
- added link hand_2, mass 0.1; collision box size=0.5 0.46411047216403317 0.1; visual box size=0.5 0.46411047216403317 0.1
- added link hand_2_sensor_0_bottom, mass 0; collision box size=0.5 0.46411047216403317 0.02; visual box size=0.5 0.46411047216403317 0.02
- added link hand_2_sensor_0_start, mass 0; collision box size=0.02 0.46411047216403317 0.1; visual box size=0.02 0.46411047216403317 0.1
- added link hand_2_sensor_0_stop, mass 0; collision box size=0.02 0.46411047216403317 0.1; visual box size=0.02 0.46411047216403317 0.1
- added link hand_2_sensor_0_top, mass 0; collision box size=0.5 0.46411047216403317 0.02; visual box size=0.5 0.46411047216403317 0.02
- added link hand_3, mass 0.1; collision box size=0.5 0.46411047216403317 0.1; visual box size=0.5 0.46411047216403317 0.1
- added link hand_3_sensor_0_bottom, mass 0; collision box size=0.5 0.46411047216403317 0.02; visual box size=0.5 0.46411047216403317 0.02
- added link hand_3_sensor_0_start, mass 0; collision box size=0.02 0.46411047216403317 0.1; visual box size=0.02 0.46411047216403317 0.1
- added link hand_3_sensor_0_stop, mass 0; collision box size=0.02 0.46411047216403317 0.1; visual box size=0.02 0.46411047216403317 0.1
- added link hand_3_sensor_0_top, mass 0; collision box size=0.5 0.46411047216403317 0.02; visual box size=0.5 0.46411047216403317 0.02
- added link hand_4, mass 0.1; collision box size=0.5 0.46411047216403317 0.1; visual box size=0.5 0.46411047216403317 0.1
- added link hand_4_sensor_0_bottom, mass 0; collision box size=0.5 0.46411047216403317 0.02; visual box size=0.5 0.46411047216403317 0.02
- added link hand_4_sensor_0_start, mass 0; collision box size=0.02 0.46411047216403317 0.1; visual box size=0.02 0.46411047216403317 0.1
- added link hand_4_sensor_0_stop, mass 0; collision box size=0.02 0.46411047216403317 0.1; visual box size=0.02 0.46411047216403317 0.1
- added link hand_4_sensor_0_top, mass 0; collision box size=0.5 0.46411047216403317 0.02; visual box size=0.5 0.46411047216403317 0.02
- added link hand_5, mass 0.1; collision box size=0.5 0.46411047216403317 0.1; visual box size=0.5 0.46411047216403317 0.1
- added link hand_5_sensor_0_bottom, mass 0; collision box size=0.5 0.46411047216403317 0.02; visual box size=0.5 0.46411047216403317 0.02
- added link hand_5_sensor_0_start, mass 0; collision box size=0.02 0.46411047216403317 0.1; visual box size=0.02 0.46411047216403317 0.1
- added link hand_5_sensor_0_stop, mass 0; collision box size=0.02 0.46411047216403317 0.1; visual box size=0.02 0.46411047216403317 0.1
- added link hand_5_sensor_0_top, mass 0; collision box size=0.5 0.46411047216403317 0.02; visual box size=0.5 0.46411047216403317 0.02
- added link hand_6, mass 0.1; collision box size=0.5 0.46411047216403317 0.1; visual box size=0.5 0.46411047216403317 0.1
- added link hand_6_sensor_0_bottom, mass 0; collision box size=0.5 0.46411047216403317 0.02; visual box size=0.5 0.46411047216403317 0.02
- added link hand_6_sensor_0_start, mass 0; collision box size=0.02 0.46411047216403317 0.1; visual box size=0.02 0.46411047216403317 0.1
- added link hand_6_sensor_0_stop, mass 0; collision box size=0.02 0.46411047216403317 0.1; visual box size=0.02 0.46411047216403317 0.1
- added link hand_6_sensor_0_top, mass 0; collision box size=0.5 0.46411047216403317 0.02; visual box size=0.5 0.46411047216403317 0.02
- added link hand_7, mass 0.1; collision box size=0.5 0.46411047216403317 0.1; visual box size=0.5 0.46411047216403317 0.1
- added link hand_7_sensor_0_bottom, mass 0; collision box size=0.5 0.46411047216403317 0.02; visual box size=0.5 0.46411047216403317 0.02
- added link hand_7_sensor_0_start, mass 0; collision box size=0.02 0.46411047216403317 0.1; visual box size=0.02 0.46411047216403317 0.1
- added link hand_7_sensor_0_stop, mass 0; collision box size=0.02 0.46411047216403317 0.1; visual box size=0.02 0.46411047216403317 0.1
- added link hand_7_sensor_0_top, mass 0; collision box size=0.5 0.46411047216403317 0.02; visual box size=0.5 0.46411047216403317 0.02
- added link hand_8, mass 0.1; collision box size=0.5 0.46411047216403317 0.1; visual box size=0.5 0.46411047216403317 0.1
- added link hand_8_sensor_0_bottom, mass 0; collision box size=0.5 0.46411047216403317 0.02; visual box size=0.5 0.46411047216403317 0.02
- added link hand_8_sensor_0_start, mass 0; collision box size=0.02 0.46411047216403317 0.1; visual box size=0.02 0.46411047216403317 0.1
- added link hand_8_sensor_0_stop, mass 0; collision box size=0.02 0.46411047216403317 0.1; visual box size=0.02 0.46411047216403317 0.1
- added link hand_8_sensor_0_top, mass 0; collision box size=0.5 0.46411047216403317 0.02; visual box size=0.5 0.46411047216403317 0.02
- added link hand_9, mass 0.1; collision box size=0.5 0.46411047216403317 0.1; visual box size=0.5 0.46411047216403317 0.1
- added link hand_9_sensor_0_bottom, mass 0; collision box size=0.5 0.46411047216403317 0.02; visual box size=0.5 0.46411047216403317 0.02
- added link hand_9_sensor_0_start, mass 0; collision box size=0.02 0.46411047216403317 0.1; visual box size=0.02 0.46411047216403317 0.1
- added link hand_9_sensor_0_stop, mass 0; collision box size=0.02 0.46411047216403317 0.1; visual box size=0.02 0.46411047216403317 0.1
- added link hand_9_sensor_0_top, mass 0; collision box size=0.5 0.46411047216403317 0.02; visual box size=0.5 0.46411047216403317 0.02
- added link shoulder_pitch, mass 0.1; collision box size=0.2 0.1 0.1; visual box size=0.2 0.1 0.1
- added link shoulder_roll, mass 0.1; collision box size=0.1 0.1 0.1; visual box size=0.1 0.1 0.1
- link body: mass 100 -> 0.1; geometry collision box size=1 1 2; visual box size=1 1 2
Joints:
- removed joint body_body_sensor_0_left_joint
- removed joint body_body_sensor_0_right_joint
- removed joint body_body_sensor_0_start_joint
- removed joint body_body_sensor_0_stop_joint
- removed joint body_body_sensor_0_top_joint
- removed joint body_body_square_0_joint
- removed joint body_body_square_10_joint
- removed joint body_body_square_11_joint
- removed joint body_body_square_12_joint
- removed joint body_body_square_13_joint
- removed joint body_body_square_14_joint
- removed joint body_body_square_15_joint
- removed joint body_body_square_16_joint
- removed joint body_body_square_17_joint
- removed joint body_body_square_18_joint
- removed joint body_body_square_19_joint
- removed joint body_body_square_1_joint
- removed joint body_body_square_20_joint
- removed joint body_body_square_21_joint
- removed joint body_body_square_2_joint
- removed joint body_body_square_3_joint
- removed joint body_body_square_4_joint
- removed joint body_body_square_5_joint
- removed joint body_body_square_6_joint
- removed joint body_body_square_7_joint
- removed joint body_body_square_8_joint
- removed joint body_body_square_9_joint
- removed joint body_left_shoulder_joint
- removed joint body_right_shoulder_joint
- removed joint left_arm_left_arm_sensor_0_bottom_joint
- removed joint left_arm_left_arm_sensor_0_left_joint
- removed joint left_arm_left_arm_sensor_0_right_joint
- removed joint left_arm_left_arm_sensor_0_start_joint
- removed joint left_arm_left_arm_sensor_0_top_joint
- removed joint left_arm_left_arm_sensor_1_bottom_joint
- removed joint left_arm_left_arm_sensor_1_left_joint
- removed joint left_arm_left_arm_sensor_1_right_joint
- removed joint left_arm_left_arm_sensor_1_top_joint
- removed joint left_arm_left_arm_sensor_2_bottom_joint
- removed joint left_arm_left_arm_sensor_2_left_joint
- removed joint left_arm_left_arm_sensor_2_right_joint
- removed joint left_arm_left_arm_sensor_2_stop_joint
- removed joint left_arm_left_arm_sensor_2_top_joint
- removed joint left_arm_left_hand_joint
- removed joint left_hand_left_hand_sensor_0_bottom_joint
- removed joint left_hand_left_hand_sensor_0_left_joint
- removed joint left_hand_left_hand_sensor_0_right_joint
- removed joint left_hand_left_hand_sensor_0_stop_joint
- removed joint left_hand_left_hand_sensor_0_top_joint
- removed joint left_shoulder_left_arm_joint
- removed joint right_arm_right_arm_sensor_0_bottom_joint
- removed joint right_arm_right_arm_sensor_0_left_joint
- removed joint right_arm_right_arm_sensor_0_right_joint
- removed joint right_arm_right_arm_sensor_0_start_joint
- removed joint right_arm_right_arm_sensor_0_top_joint
- removed joint right_arm_right_arm_sensor_1_bottom_joint
- removed joint right_arm_right_arm_sensor_1_left_joint
- removed joint right_arm_right_arm_sensor_1_right_joint
- removed joint right_arm_right_arm_sensor_1_top_joint
- removed joint right_arm_right_arm_sensor_2_bottom_joint
- removed joint right_arm_right_arm_sensor_2_left_joint
- removed joint right_arm_right_arm_sensor_2_right_joint
- removed joint right_arm_right_arm_sensor_2_stop_joint
- removed joint right_arm_right_arm_sensor_2_top_joint
- removed joint right_arm_right_hand_joint
- removed joint right_hand_right_hand_sensor_0_bottom_joint
- removed joint right_hand_right_hand_sensor_0_left_joint
- removed joint right_hand_right_hand_sensor_0_right_joint
- removed joint right_hand_right_hand_sensor_0_start_joint
- removed joint right_hand_right_hand_sensor_0_top_joint
- removed joint right_shoulder_right_arm_joint
- added joint arm_1_elbow_pitch_joint: type revolute, parent arm_1, child elbow_pitch, origin xyz=0 0 0.55 rpy=0 0 0, axis 1 0 0, limit lower=-1.5 upper=0 effort=100 velocity=10
- added joint arm_2_hand_0_joint: type fixed, parent arm_2, child hand_0, origin xyz=0.2 -0.19999999999999996 2.0 rpy=-0.0 0 0, axis 0 0 1
- added joint arm_2_hand_10_joint: type fixed, parent arm_2, child hand_10, origin xyz=0.2 -0.8928203230275509 1.6 rpy=-5.235987755982989 0 0, axis 0 0 1
- added joint arm_2_hand_11_joint: type fixed, parent arm_2, child hand_11, origin xyz=0.2 -0.6000000000000003 1.8928203230275507 rpy=-5.759586531581287 0 0, axis 0 0 1
- added joint arm_2_hand_1_joint: type fixed, parent arm_2, child hand_1, origin xyz=0.2 0.2 1.8928203230275509 rpy=-0.5235987755982988 0 0, axis 0 0 1
- added joint arm_2_hand_2_joint: type fixed, parent arm_2, child hand_2, origin xyz=0.2 0.49282032302755097 1.6 rpy=-1.0471975511965976 0 0, axis 0 0 1
- added joint arm_2_hand_3_joint: type fixed, parent arm_2, child hand_3, origin xyz=0.2 0.6000000000000001 1.2 rpy=-1.5707963267948966 0 0, axis 0 0 1
- added joint arm_2_hand_4_joint: type fixed, parent arm_2, child hand_4, origin xyz=0.2 0.4928203230275511 0.8 rpy=-2.0943951023931953 0 0, axis 0 0 1
- added joint arm_2_hand_5_joint: type fixed, parent arm_2, child hand_5, origin xyz=0.2 0.2 0.5071796769724489 rpy=-2.6179938779914944 0 0, axis 0 0 1
- added joint arm_2_hand_6_joint: type fixed, parent arm_2, child hand_6, origin xyz=0.2 -0.19999999999999984 0.3999999999999999 rpy=-3.141592653589793 0 0, axis 0 0 1
- added joint arm_2_hand_7_joint: type fixed, parent arm_2, child hand_7, origin xyz=0.2 -0.5999999999999998 0.5071796769724488 rpy=-3.665191429188092 0 0, axis 0 0 1
- added joint arm_2_hand_8_joint: type fixed, parent arm_2, child hand_8, origin xyz=0.2 -0.8928203230275508 0.7999999999999996 rpy=-4.1887902047863905 0 0, axis 0 0 1
- added joint arm_2_hand_9_joint: type fixed, parent arm_2, child hand_9, origin xyz=0.2 -1.0 1.1999999999999997 rpy=-4.71238898038469 0 0, axis 0 0 1
- added joint base_body_joint: type continuous, parent base, child body, origin xyz=0 0 1.05 rpy=0 0 0, axis 0 0 1
- added joint body_body_face_0_joint: type fixed, parent body, child body_face_0, origin xyz=0.501 -0.33333333333333337 0.6111111111111112 rpy=0 0 0, axis 0 0 1
- added joint body_body_face_10_joint: type fixed, parent body, child body_face_10, origin xyz=0.11111111111111116 -0.1111111111111111 1.001 rpy=0 0 0, axis 0 0 1
- added joint body_body_face_11_joint: type fixed, parent body, child body_face_11, origin xyz=0.2222222222222222 -0.1111111111111111 1.001 rpy=0 0 0, axis 0 0 1
- added joint body_body_face_12_joint: type fixed, parent body, child body_face_12, origin xyz=-0.33333333333333337 0.0 1.001 rpy=0 0 0, axis 0 0 1
- added joint body_body_face_13_joint: type fixed, parent body, child body_face_13, origin xyz=-0.2222222222222222 0.0 1.001 rpy=0 0 0, axis 0 0 1
- added joint body_body_face_14_joint: type fixed, parent body, child body_face_14, origin xyz=-0.1111111111111111 0.0 1.001 rpy=0 0 0, axis 0 0 1
- added joint body_body_face_15_joint: type fixed, parent body, child body_face_15, origin xyz=0.0 0.0 1.001 rpy=0 0 0, axis 0 0 1
- added joint body_body_face_16_joint: type fixed, parent body, child body_face_16, origin xyz=0.11111111111111116 0.0 1.001 rpy=0 0 0, axis 0 0 1
- added joint body_body_face_17_joint: type fixed, parent body, child body_face_17, origin xyz=0.2222222222222222 0.0 1.001 rpy=0 0 0, axis 0 0 1
- added joint body_body_face_18_joint: type fixed, parent body, child body_face_18, origin xyz=0.33333333333333337 0.0 1.001 rpy=0 0 0, axis 0 0 1
- added joint body_body_face_19_joint: type fixed, parent body, child body_face_19, origin xyz=0.11111111111111116 0.11111111111111116 1.001 rpy=0 0 0, axis 0 0 1
- added joint body_body_face_1_joint: type fixed, parent body, child body_face_1, origin xyz=0.501 -0.2222222222222222 0.7222222222222222 rpy=0 0 0, axis 0 0 1
- added joint body_body_face_20_joint: type fixed, parent body, child body_face_20, origin xyz=0.2222222222222222 0.11111111111111116 1.001 rpy=0 0 0, axis 0 0 1
- added joint body_body_face_21_joint: type fixed, parent body, child body_face_21, origin xyz=0.11111111111111116 0.2222222222222222 1.001 rpy=0 0 0, axis 0 0 1
- added joint body_body_face_2_joint: type fixed, parent body, child body_face_2, origin xyz=0.501 -0.1111111111111111 0.6111111111111112 rpy=0 0 0, axis 0 0 1
- added joint body_body_face_3_joint: type fixed, parent body, child body_face_3, origin xyz=0.501 -0.1111111111111111 0.2777777777777778 rpy=0 0 0, axis 0 0 1
- added joint body_body_face_4_joint: type fixed, parent body, child body_face_4, origin xyz=0.501 0.0 0.2777777777777778 rpy=0 0 0, axis 0 0 1
- added joint body_body_face_5_joint: type fixed, parent body, child body_face_5, origin xyz=0.501 0.11111111111111116 0.6111111111111112 rpy=0 0 0, axis 0 0 1
- added joint body_body_face_6_joint: type fixed, parent body, child body_face_6, origin xyz=0.501 0.11111111111111116 0.2777777777777778 rpy=0 0 0, axis 0 0 1
- added joint body_body_face_7_joint: type fixed, parent body, child body_face_7, origin xyz=0.501 0.2222222222222222 0.7222222222222222 rpy=0 0 0, axis 0 0 1
- added joint body_body_face_8_joint: type fixed, parent body, child body_face_8, origin xyz=0.501 0.33333333333333337 0.6111111111111112 rpy=0 0 0, axis 0 0 1
- added joint body_body_face_9_joint: type fixed, parent body, child body_face_9, origin xyz=0.11111111111111116 -0.2222222222222222 1.001 rpy=0 0 0, axis 0 0 1
- added joint body_shoulder_pitch_joint: type revolute, parent body, child shoulder_pitch, origin xyz=0.5 -0.55 0 rpy=0 0 0, axis 0 -1 0, limit lower=-1.5 upper=0 effort=100 velocity=10
- added joint elbow_pitch_arm_2_joint: type fixed, parent elbow_pitch, child arm_2, origin xyz=0 0.15 0.35 rpy=-0.5 0 0, axis 0 -1 0
- added joint hand_0_hand_0_sensor_0_bottom_joint: type fixed, parent hand_0, child hand_0_sensor_0_bottom, origin xyz=0 0 -0.05 rpy=0 0 0, axis 0 0 1
- added joint hand_0_hand_0_sensor_0_start_joint: type fixed, parent hand_0, child hand_0_sensor_0_start, origin xyz=0.25 0 0 rpy=0 0 0, axis 0 0 1
- added joint hand_0_hand_0_sensor_0_stop_joint: type fixed, parent hand_0, child hand_0_sensor_0_stop, origin xyz=-0.25 0 0 rpy=0 0 0, axis 0 0 1
- added joint hand_0_hand_0_sensor_0_top_joint: type fixed, parent hand_0, child hand_0_sensor_0_top, origin xyz=0 0 0.05 rpy=0 0 0, axis 0 0 1
- added joint hand_10_hand_10_sensor_0_bottom_joint: type fixed, parent hand_10, child hand_10_sensor_0_bottom, origin xyz=0 0 -0.05 rpy=0 0 0, axis 0 0 1
- added joint hand_10_hand_10_sensor_0_start_joint: type fixed, parent hand_10, child hand_10_sensor_0_start, origin xyz=0.25 0 0 rpy=0 0 0, axis 0 0 1
- added joint hand_10_hand_10_sensor_0_stop_joint: type fixed, parent hand_10, child hand_10_sensor_0_stop, origin xyz=-0.25 0 0 rpy=0 0 0, axis 0 0 1
- added joint hand_10_hand_10_sensor_0_top_joint: type fixed, parent hand_10, child hand_10_sensor_0_top, origin xyz=0 0 0.05 rpy=0 0 0, axis 0 0 1
- added joint hand_11_hand_11_sensor_0_bottom_joint: type fixed, parent hand_11, child hand_11_sensor_0_bottom, origin xyz=0 0 -0.05 rpy=0 0 0, axis 0 0 1
- added joint hand_11_hand_11_sensor_0_start_joint: type fixed, parent hand_11, child hand_11_sensor_0_start, origin xyz=0.25 0 0 rpy=0 0 0, axis 0 0 1
- added joint hand_11_hand_11_sensor_0_stop_joint: type fixed, parent hand_11, child hand_11_sensor_0_stop, origin xyz=-0.25 0 0 rpy=0 0 0, axis 0 0 1
- added joint hand_11_hand_11_sensor_0_top_joint: type fixed, parent hand_11, child hand_11_sensor_0_top, origin xyz=0 0 0.05 rpy=0 0 0, axis 0 0 1
- added joint hand_1_hand_1_sensor_0_bottom_joint: type fixed, parent hand_1, child hand_1_sensor_0_bottom, origin xyz=0 0 -0.05 rpy=0 0 0, axis 0 0 1
- added joint hand_1_hand_1_sensor_0_start_joint: type fixed, parent hand_1, child hand_1_sensor_0_start, origin xyz=0.25 0 0 rpy=0 0 0, axis 0 0 1
- added joint hand_1_hand_1_sensor_0_stop_joint: type fixed, parent hand_1, child hand_1_sensor_0_stop, origin xyz=-0.25 0 0 rpy=0 0 0, axis 0 0 1
- added joint hand_1_hand_1_sensor_0_top_joint: type fixed, parent hand_1, child hand_1_sensor_0_top, origin xyz=0 0 0.05 rpy=0 0 0, axis 0 0 1
- added joint hand_2_hand_2_sensor_0_bottom_joint: type fixed, parent hand_2, child hand_2_sensor_0_bottom, origin xyz=0 0 -0.05 rpy=0 0 0, axis 0 0 1
- added joint hand_2_hand_2_sensor_0_start_joint: type fixed, parent hand_2, child hand_2_sensor_0_start, origin xyz=0.25 0 0 rpy=0 0 0, axis 0 0 1
- added joint hand_2_hand_2_sensor_0_stop_joint: type fixed, parent hand_2, child hand_2_sensor_0_stop, origin xyz=-0.25 0 0 rpy=0 0 0, axis 0 0 1
- added joint hand_2_hand_2_sensor_0_top_joint: type fixed, parent hand_2, child hand_2_sensor_0_top, origin xyz=0 0 0.05 rpy=0 0 0, axis 0 0 1
- added joint hand_3_hand_3_sensor_0_bottom_joint: type fixed, parent hand_3, child hand_3_sensor_0_bottom, origin xyz=0 0 -0.05 rpy=0 0 0, axis 0 0 1
- added joint hand_3_hand_3_sensor_0_start_joint: type fixed, parent hand_3, child hand_3_sensor_0_start, origin xyz=0.25 0 0 rpy=0 0 0, axis 0 0 1
- added joint hand_3_hand_3_sensor_0_stop_joint: type fixed, parent hand_3, child hand_3_sensor_0_stop, origin xyz=-0.25 0 0 rpy=0 0 0, axis 0 0 1
- added joint hand_3_hand_3_sensor_0_top_joint: type fixed, parent hand_3, child hand_3_sensor_0_top, origin xyz=0 0 0.05 rpy=0 0 0, axis 0 0 1
- added joint hand_4_hand_4_sensor_0_bottom_joint: type fixed, parent hand_4, child hand_4_sensor_0_bottom, origin xyz=0 0 -0.05 rpy=0 0 0, axis 0 0 1
- added joint hand_4_hand_4_sensor_0_start_joint: type fixed, parent hand_4, child hand_4_sensor_0_start, origin xyz=0.25 0 0 rpy=0 0 0, axis 0 0 1
- added joint hand_4_hand_4_sensor_0_stop_joint: type fixed, parent hand_4, child hand_4_sensor_0_stop, origin xyz=-0.25 0 0 rpy=0 0 0, axis 0 0 1
- added joint hand_4_hand_4_sensor_0_top_joint: type fixed, parent hand_4, child hand_4_sensor_0_top, origin xyz=0 0 0.05 rpy=0 0 0, axis 0 0 1
- added joint hand_5_hand_5_sensor_0_bottom_joint: type fixed, parent hand_5, child hand_5_sensor_0_bottom, origin xyz=0 0 -0.05 rpy=0 0 0, axis 0 0 1
- added joint hand_5_hand_5_sensor_0_start_joint: type fixed, parent hand_5, child hand_5_sensor_0_start, origin xyz=0.25 0 0 rpy=0 0 0, axis 0 0 1
- added joint hand_5_hand_5_sensor_0_stop_joint: type fixed, parent hand_5, child hand_5_sensor_0_stop, origin xyz=-0.25 0 0 rpy=0 0 0, axis 0 0 1
- added joint hand_5_hand_5_sensor_0_top_joint: type fixed, parent hand_5, child hand_5_sensor_0_top, origin xyz=0 0 0.05 rpy=0 0 0, axis 0 0 1
- added joint hand_6_hand_6_sensor_0_bottom_joint: type fixed, parent hand_6, child hand_6_sensor_0_bottom, origin xyz=0 0 -0.05 rpy=0 0 0, axis 0 0 1
- added joint hand_6_hand_6_sensor_0_start_joint: type fixed, parent hand_6, child hand_6_sensor_0_start, origin xyz=0.25 0 0 rpy=0 0 0, axis 0 0 1
- added joint hand_6_hand_6_sensor_0_stop_joint: type fixed, parent hand_6, child hand_6_sensor_0_stop, origin xyz=-0.25 0 0 rpy=0 0 0, axis 0 0 1
- added joint hand_6_hand_6_sensor_0_top_joint: type fixed, parent hand_6, child hand_6_sensor_0_top, origin xyz=0 0 0.05 rpy=0 0 0, axis 0 0 1
- added joint hand_7_hand_7_sensor_0_bottom_joint: type fixed, parent hand_7, child hand_7_sensor_0_bottom, origin xyz=0 0 -0.05 rpy=0 0 0, axis 0 0 1
- added joint hand_7_hand_7_sensor_0_start_joint: type fixed, parent hand_7, child hand_7_sensor_0_start, origin xyz=0.25 0 0 rpy=0 0 0, axis 0 0 1
- added joint hand_7_hand_7_sensor_0_stop_joint: type fixed, parent hand_7, child hand_7_sensor_0_stop, origin xyz=-0.25 0 0 rpy=0 0 0, axis 0 0 1
- added joint hand_7_hand_7_sensor_0_top_joint: type fixed, parent hand_7, child hand_7_sensor_0_top, origin xyz=0 0 0.05 rpy=0 0 0, axis 0 0 1
- added joint hand_8_hand_8_sensor_0_bottom_joint: type fixed, parent hand_8, child hand_8_sensor_0_bottom, origin xyz=0 0 -0.05 rpy=0 0 0, axis 0 0 1
- added joint hand_8_hand_8_sensor_0_start_joint: type fixed, parent hand_8, child hand_8_sensor_0_start, origin xyz=0.25 0 0 rpy=0 0 0, axis 0 0 1
- added joint hand_8_hand_8_sensor_0_stop_joint: type fixed, parent hand_8, child hand_8_sensor_0_stop, origin xyz=-0.25 0 0 rpy=0 0 0, axis 0 0 1
- added joint hand_8_hand_8_sensor_0_top_joint: type fixed, parent hand_8, child hand_8_sensor_0_top, origin xyz=0 0 0.05 rpy=0 0 0, axis 0 0 1
- added joint hand_9_hand_9_sensor_0_bottom_joint: type fixed, parent hand_9, child hand_9_sensor_0_bottom, origin xyz=0 0 -0.05 rpy=0 0 0, axis 0 0 1
- added joint hand_9_hand_9_sensor_0_start_joint: type fixed, parent hand_9, child hand_9_sensor_0_start, origin xyz=0.25 0 0 rpy=0 0 0, axis 0 0 1
- added joint hand_9_hand_9_sensor_0_stop_joint: type fixed, parent hand_9, child hand_9_sensor_0_stop, origin xyz=-0.25 0 0 rpy=0 0 0, axis 0 0 1
- added joint hand_9_hand_9_sensor_0_top_joint: type fixed, parent hand_9, child hand_9_sensor_0_top, origin xyz=0 0 0.05 rpy=0 0 0, axis 0 0 1
- added joint shoulder_pitch_shoulder_roll_joint: type revolute, parent shoulder_pitch, child shoulder_roll, origin xyz=0.15 0 0 rpy=0 0 0, axis 1 0 0, limit lower=0 upper=1.5 effort=100 velocity=10
- added joint shoulder_roll_arm_1_joint: type fixed, parent shoulder_roll, child arm_1, origin xyz=0 0 0.55 rpy=0 0 0, axis 0 -1 0
