Commit message: 2025_01_19, decent with new robot, but still bad

File: pybullet_data/robot.urdf (robot description, URDF)
Before this commit: robot robot, 89 links, 88 joints
Links:
- removed link arm_2
- removed link elbow_pitch
- removed link shoulder_roll
- link arm_1: mass 0.1 -> 10; geometry collision box size=0.1 1.5 0.1; visual box size=0.1 1.5 0.1
- link body: mass 0.1 -> 10
- link hand_0: mass 0.1 -> 1
- link hand_1: mass 0.1 -> 1
- link hand_10: mass 0.1 -> 1
- link hand_11: mass 0.1 -> 1
- link hand_2: mass 0.1 -> 1
- link hand_3: mass 0.1 -> 1
- link hand_4: mass 0.1 -> 1
- link hand_5: mass 0.1 -> 1
- link hand_6: mass 0.1 -> 1
- link hand_7: mass 0.1 -> 1
- link hand_8: mass 0.1 -> 1
- link hand_9: mass 0.1 -> 1
- link shoulder_pitch: mass 0.1 -> 10
Joints:
- removed joint arm_1_elbow_pitch_joint
- removed joint arm_2_hand_0_joint
- removed joint arm_2_hand_10_joint
- removed joint arm_2_hand_11_joint
- removed joint arm_2_hand_1_joint
- removed joint arm_2_hand_2_joint
- removed joint arm_2_hand_3_joint
- removed joint arm_2_hand_4_joint
- removed joint arm_2_hand_5_joint
- removed joint arm_2_hand_6_joint
- removed joint arm_2_hand_7_joint
- removed joint arm_2_hand_8_joint
- removed joint arm_2_hand_9_joint
- removed joint elbow_pitch_arm_2_joint
- removed joint shoulder_pitch_shoulder_roll_joint
- removed joint shoulder_roll_arm_1_joint
- added joint arm_1_hand_0_joint: type fixed, parent arm_1, child hand_0, origin xyz=0.2 -1.4 1.4000000000000001 rpy=-0.0 -0.4 0.0, axis 0 0 1
- added joint arm_1_hand_10_joint: type fixed, parent arm_1, child hand_10, origin xyz=0.2 -2.092820323027551 1.0000000000000002 rpy=-5.235987755982989 -0.20000000000000007 -0.34641016151377546, axis 0 0 1
- added joint arm_1_hand_11_joint: type fixed, parent arm_1, child hand_11, origin xyz=0.2 -1.8000000000000003 1.2928203230275508 rpy=-5.759586531581287 -0.34641016151377535 -0.20000000000000018, axis 0 0 1
- added joint arm_1_hand_1_joint: type fixed, parent arm_1, child hand_1, origin xyz=0.2 -1.0 1.2928203230275512 rpy=-0.5235987755982988 -0.3464101615137755 0.19999999999999998, axis 0 0 1
- added joint arm_1_hand_2_joint: type fixed, parent arm_1, child hand_2, origin xyz=0.2 -0.707179676972449 1.0000000000000002 rpy=-1.0471975511965976 -0.20000000000000007 0.34641016151377546, axis 0 0 1
- added joint arm_1_hand_3_joint: type fixed, parent arm_1, child hand_3, origin xyz=0.2 -0.5999999999999999 0.6000000000000001 rpy=-1.5707963267948966 -2.4492935982947065e-17 0.4, axis 0 0 1
- added joint arm_1_hand_4_joint: type fixed, parent arm_1, child hand_4, origin xyz=0.2 -0.7071796769724489 0.20000000000000023 rpy=-2.0943951023931953 0.19999999999999993 0.3464101615137755, axis 0 0 1
- added joint arm_1_hand_5_joint: type fixed, parent arm_1, child hand_5, origin xyz=0.2 -1.0 -0.09282032302755094 rpy=-2.6179938779914944 0.3464101615137755 0.19999999999999998, axis 0 0 1
- added joint arm_1_hand_6_joint: type fixed, parent arm_1, child hand_6, origin xyz=0.2 -1.4 -0.19999999999999996 rpy=-3.141592653589793 0.4 4.898587196589413e-17, axis 0 0 1
- added joint arm_1_hand_7_joint: type fixed, parent arm_1, child hand_7, origin xyz=0.2 -1.7999999999999998 -0.09282032302755105 rpy=-3.665191429188092 0.34641016151377557 -0.1999999999999999, axis 0 0 1
- added joint arm_1_hand_8_joint: type fixed, parent arm_1, child hand_8, origin xyz=0.2 -2.0928203230275506 0.19999999999999973 rpy=-4.1887902047863905 0.20000000000000018 -0.34641016151377535, axis 0 0 1
- added joint arm_1_hand_9_joint: type fixed, parent arm_1, child hand_9, origin xyz=0.2 -2.2 0.6 rpy=-4.71238898038469 7.347880794884119e-17 -0.4, axis 0 0 1
- added joint shoulder_pitch_arm_1_joint: type prismatic, parent shoulder_pitch, child arm_1, origin xyz=0.15 0 0.7 rpy=-1.5707 0 0, axis 0 -1 0, limit lower=-1 upper=0 effort=100 velocity=10
- joint base_body_joint: limit (none) -> lower=0 upper=0 effort=0 velocity=0
