Commit message: 2025_02_19, big test. Finding problems in head-arm bots.

File: pybullet_data/robot_two_side_arm.urdf (robot description, URDF)
Before this commit: robot robot, 72 links, 71 joints
Links:
- removed link body_square_0
- removed link body_square_1
- removed link body_square_10
- removed link body_square_11
- removed link body_square_12
- removed link body_square_13
- removed link body_square_14
- removed link body_square_15
- removed link body_square_16
- removed link body_square_17
- removed link body_square_18
- removed link body_square_19
- removed link body_square_2
- removed link body_square_20
- removed link body_square_21
- removed link body_square_3
- removed link body_square_4
- removed link body_square_5
- removed link body_square_6
- removed link body_square_7
- removed link body_square_8
- removed link body_square_9
- added link body_face_0, mass 0; collision box size=0.002 0.1111111111111111 0.1111111111111111; visual box size=0.002 0.1111111111111111 0.1111111111111111
- added link body_face_1, mass 0; collision box size=0.002 0.1111111111111111 0.1111111111111111; visual box size=0.002 0.1111111111111111 0.1111111111111111
- added link body_face_2, mass 0; collision box size=0.002 0.1111111111111111 0.1111111111111111; visual box size=0.002 0.1111111111111111 0.1111111111111111
- added link body_face_3, mass 0; collision box size=0.002 0.1111111111111111 0.1111111111111111; visual box size=0.002 0.1111111111111111 0.1111111111111111
- added link body_face_4, mass 0; collision box size=0.002 0.1111111111111111 0.1111111111111111; visual box size=0.002 0.1111111111111111 0.1111111111111111
- added link body_face_5, mass 0; collision box size=0.002 0.1111111111111111 0.1111111111111111; visual box size=0.002 0.1111111111111111 0.1111111111111111
- added link body_face_6, mass 0; collision box size=0.002 0.1111111111111111 0.1111111111111111; visual box size=0.002 0.1111111111111111 0.1111111111111111
- added link body_face_7, mass 0; collision box size=0.002 0.1111111111111111 0.1111111111111111; visual box size=0.002 0.1111111111111111 0.1111111111111111
- added link body_face_8, mass 0; collision box size=0.002 0.1111111111111111 0.1111111111111111; visual box size=0.002 0.1111111111111111 0.1111111111111111
Joints:
- removed joint body_body_square_0_joint
- removed joint body_body_square_10_joint
- removed joint body_body_square_11_joint
- removed joint body_body_square_12_joint
- removed joint body_body_square_13_joint
- removed joint body_body_square_14_joint
- removed joint body_body_square_15_joint
- removed joint body_body_square_16_joint
- removed joint body_body_square_17_joint
- removed joint body_body_square_18_joint
- removed joint body_body_square_19_joint
- removed joint body_body_square_1_joint
- removed joint body_body_square_20_joint
- removed joint body_body_square_21_joint
- removed joint body_body_square_2_joint
- removed joint body_body_square_3_joint
- removed joint body_body_square_4_joint
- removed joint body_body_square_5_joint
- removed joint body_body_square_6_joint
- removed joint body_body_square_7_joint
- removed joint body_body_square_8_joint
- removed joint body_body_square_9_joint
- added joint body_body_face_0_joint: type fixed, parent body, child body_face_0, origin xyz=0.501 -0.33333333333333337 0.11111111111111116 rpy=0 0 0, axis 0 0 1
- added joint body_body_face_1_joint: type fixed, parent body, child body_face_1, origin xyz=0.501 -0.2222222222222222 0.2222222222222222 rpy=0 0 0, axis 0 0 1
- added joint body_body_face_2_joint: type fixed, parent body, child body_face_2, origin xyz=0.501 -0.1111111111111111 0.11111111111111116 rpy=0 0 0, axis 0 0 1
- added joint body_body_face_3_joint: type fixed, parent body, child body_face_3, origin xyz=0.501 -0.1111111111111111 -0.2222222222222222 rpy=0 0 0, axis 0 0 1
- added joint body_body_face_4_joint: type fixed, parent body, child body_face_4, origin xyz=0.501 0.0 -0.2222222222222222 rpy=0 0 0, axis 0 0 1
- added joint body_body_face_5_joint: type fixed, parent body, child body_face_5, origin xyz=0.501 0.11111111111111116 0.11111111111111116 rpy=0 0 0, axis 0 0 1
- added joint body_body_face_6_joint: type fixed, parent body, child body_face_6, origin xyz=0.501 0.11111111111111116 -0.2222222222222222 rpy=0 0 0, axis 0 0 1
- added joint body_body_face_7_joint: type fixed, parent body, child body_face_7, origin xyz=0.501 0.2222222222222222 0.2222222222222222 rpy=0 0 0, axis 0 0 1
- added joint body_body_face_8_joint: type fixed, parent body, child body_face_8, origin xyz=0.501 0.33333333333333337 0.11111111111111116 rpy=0 0 0, axis 0 0 1
- joint body_joint_1_joint: limit (none) -> lower=0 upper=0 effort=0 velocity=0
- joint body_joint_2_joint: limit (none) -> lower=0 upper=0 effort=0 velocity=0
