Commit message: starting again!

File: pybullet_data/shapes/1_pole.urdf (robot description, URDF)
Before this commit: robot 5_cone, 21 links, 20 joints
Links:
- link 0_link: geometry collision cylinder length=0.05 radius=0.2; visual cylinder length=0.05 radius=0.2
- link 10_link: geometry collision cylinder length=0.05 radius=0.2; visual cylinder length=0.05 radius=0.2
- link 11_link: geometry collision cylinder length=0.05 radius=0.2; visual cylinder length=0.05 radius=0.2
- link 12_link: geometry collision cylinder length=0.05 radius=0.2; visual cylinder length=0.05 radius=0.2
- link 13_link: geometry collision cylinder length=0.05 radius=0.2; visual cylinder length=0.05 radius=0.2
- link 14_link: geometry collision cylinder length=0.05 radius=0.2; visual cylinder length=0.05 radius=0.2
- link 15_link: geometry collision cylinder length=0.05 radius=0.2; visual cylinder length=0.05 radius=0.2
- link 16_link: geometry collision cylinder length=0.05 radius=0.2; visual cylinder length=0.05 radius=0.2
- link 17_link: geometry collision cylinder length=0.05 radius=0.2; visual cylinder length=0.05 radius=0.2
- link 18_link: geometry collision cylinder length=0.05 radius=0.2; visual cylinder length=0.05 radius=0.2
- link 19_link: geometry collision cylinder length=0.05 radius=0.2; visual cylinder length=0.05 radius=0.2
- link 1_link: geometry collision cylinder length=0.05 radius=0.2; visual cylinder length=0.05 radius=0.2
- link 2_link: geometry collision cylinder length=0.05 radius=0.2; visual cylinder length=0.05 radius=0.2
- link 3_link: geometry collision cylinder length=0.05 radius=0.2; visual cylinder length=0.05 radius=0.2
- link 4_link: geometry collision cylinder length=0.05 radius=0.2; visual cylinder length=0.05 radius=0.2
- link 5_link: geometry collision cylinder length=0.05 radius=0.2; visual cylinder length=0.05 radius=0.2
- link 6_link: geometry collision cylinder length=0.05 radius=0.2; visual cylinder length=0.05 radius=0.2
- link 7_link: geometry collision cylinder length=0.05 radius=0.2; visual cylinder length=0.05 radius=0.2
- link 8_link: geometry collision cylinder length=0.05 radius=0.2; visual cylinder length=0.05 radius=0.2
- link 9_link: geometry collision cylinder length=0.05 radius=0.2; visual cylinder length=0.05 radius=0.2

File: pybullet_data/shapes/2_top.urdf (robot description, URDF)
Before this commit: robot 4_flat_top, 21 links, 20 joints
Links:
- link 18_link: geometry collision cylinder length=0.05 radius=0.6; visual cylinder length=0.05 radius=0.6

File: pybullet_data/shapes/3_bottom.urdf (robot description, URDF)
Before this commit: robot 3_flat_bottom, 21 links, 20 joints
Links:
- link 1_link: geometry collision cylinder length=0.05 radius=0.6; visual cylinder length=0.05 radius=0.6

File: pybullet_data/shapes/4_middle.urdf (robot description, URDF)
Before this commit: robot 1_cylinder, 21 links, 20 joints
Links:
- link 0_link: geometry collision cylinder length=0.05 radius=0.2; visual cylinder length=0.05 radius=0.2
- link 11_link: geometry collision cylinder length=0.05 radius=0.2; visual cylinder length=0.05 radius=0.2
- link 12_link: geometry collision cylinder length=0.05 radius=0.2; visual cylinder length=0.05 radius=0.2
- link 13_link: geometry collision cylinder length=0.05 radius=0.2; visual cylinder length=0.05 radius=0.2
- link 14_link: geometry collision cylinder length=0.05 radius=0.2; visual cylinder length=0.05 radius=0.2
- link 15_link: geometry collision cylinder length=0.05 radius=0.2; visual cylinder length=0.05 radius=0.2
- link 16_link: geometry collision cylinder length=0.05 radius=0.2; visual cylinder length=0.05 radius=0.2
- link 17_link: geometry collision cylinder length=0.05 radius=0.2; visual cylinder length=0.05 radius=0.2
- link 18_link: geometry collision cylinder length=0.05 radius=0.2; visual cylinder length=0.05 radius=0.2
- link 19_link: geometry collision cylinder length=0.05 radius=0.2; visual cylinder length=0.05 radius=0.2
- link 1_link: geometry collision cylinder length=0.05 radius=0.2; visual cylinder length=0.05 radius=0.2
- link 2_link: geometry collision cylinder length=0.05 radius=0.2; visual cylinder length=0.05 radius=0.2
- link 3_link: geometry collision cylinder length=0.05 radius=0.2; visual cylinder length=0.05 radius=0.2
- link 4_link: geometry collision cylinder length=0.05 radius=0.2; visual cylinder length=0.05 radius=0.2
- link 5_link: geometry collision cylinder length=0.05 radius=0.2; visual cylinder length=0.05 radius=0.2
- link 6_link: geometry collision cylinder length=0.05 radius=0.2; visual cylinder length=0.05 radius=0.2
- link 7_link: geometry collision cylinder length=0.05 radius=0.2; visual cylinder length=0.05 radius=0.2
- link 8_link: geometry collision cylinder length=0.05 radius=0.2; visual cylinder length=0.05 radius=0.2

File: pybullet_data/shapes/5_top_bottom.urdf (robot description, URDF)
Before this commit: robot 6_cone_inverted, 21 links, 20 joints
Links:
- link 0_link: geometry collision cylinder length=0.05 radius=0.6; visual cylinder length=0.05 radius=0.6
- link 10_link: geometry collision cylinder length=0.05 radius=0.2; visual cylinder length=0.05 radius=0.2
- link 11_link: geometry collision cylinder length=0.05 radius=0.2; visual cylinder length=0.05 radius=0.2
- link 12_link: geometry collision cylinder length=0.05 radius=0.2; visual cylinder length=0.05 radius=0.2
- link 13_link: geometry collision cylinder length=0.05 radius=0.2; visual cylinder length=0.05 radius=0.2
- link 14_link: geometry collision cylinder length=0.05 radius=0.2; visual cylinder length=0.05 radius=0.2
- link 15_link: geometry collision cylinder length=0.05 radius=0.2; visual cylinder length=0.05 radius=0.2
- link 16_link: geometry collision cylinder length=0.05 radius=0.2; visual cylinder length=0.05 radius=0.2
- link 17_link: geometry collision cylinder length=0.05 radius=0.2; visual cylinder length=0.05 radius=0.2
- link 18_link: geometry collision cylinder length=0.05 radius=0.6; visual cylinder length=0.05 radius=0.6
- link 1_link: geometry collision cylinder length=0.05 radius=0.6; visual cylinder length=0.05 radius=0.6
- link 2_link: geometry collision cylinder length=0.05 radius=0.2; visual cylinder length=0.05 radius=0.2
- link 3_link: geometry collision cylinder length=0.05 radius=0.2; visual cylinder length=0.05 radius=0.2
- link 4_link: geometry collision cylinder length=0.05 radius=0.2; visual cylinder length=0.05 radius=0.2
- link 5_link: geometry collision cylinder length=0.05 radius=0.2; visual cylinder length=0.05 radius=0.2
- link 6_link: geometry collision cylinder length=0.05 radius=0.2; visual cylinder length=0.05 radius=0.2
- link 7_link: geometry collision cylinder length=0.05 radius=0.2; visual cylinder length=0.05 radius=0.2
- link 8_link: geometry collision cylinder length=0.05 radius=0.2; visual cylinder length=0.05 radius=0.2
- link 9_link: geometry collision cylinder length=0.05 radius=0.2; visual cylinder length=0.05 radius=0.2
