Commit message: working wellish

File: pybullet_data/shapes/1_SQUARE.urdf (robot description, URDF)
Before this commit: robot 1_square, 6 links, 5 joints
Joints:
- joint joint1: origin xyz=0 .6 0 rpy=0 0 0 -> xyz=0 -.6 0 rpy=0 0 0
- joint joint3: origin xyz=0 -.6 0 rpy=0 0 0 -> xyz=0 .6 0 rpy=0 0 0

File: pybullet_data/shapes/2_UP.urdf (robot description, URDF)
Before this commit: robot 2_up, 7 links, 6 joints
Joints:
- joint joint1: origin xyz=0 .6 0 rpy=0 0 0 -> xyz=0 -.6 0 rpy=0 0 0
- joint joint3: origin xyz=0 -.6 0 rpy=0 0 0 -> xyz=0 .6 0 rpy=0 0 0

File: pybullet_data/shapes/3_DOWN.urdf (robot description, URDF)
Before this commit: robot 2_up, 7 links, 6 joints
Joints:
- joint joint1: origin xyz=0 .6 0 rpy=0 0 0 -> xyz=0 -.6 0 rpy=0 0 0
- joint joint3: origin xyz=0 -.6 0 rpy=0 0 0 -> xyz=0 .6 0 rpy=0 0 0

File: pybullet_data/shapes/4_LEFT.urdf (robot description, URDF)
Before this commit: robot 2_up, 7 links, 6 joints
Joints:
- joint joint1: origin xyz=0 .6 0 rpy=0 0 0 -> xyz=0 -.6 0 rpy=0 0 0
- joint joint3: origin xyz=0 -.6 0 rpy=0 0 0 -> xyz=0 .6 0 rpy=0 0 0

File: pybullet_data/shapes/5_RIGHT.urdf (robot description, URDF)
Before this commit: robot 2_up, 7 links, 6 joints
Joints:
- joint joint1: origin xyz=0 .6 0 rpy=0 0 0 -> xyz=0 -.6 0 rpy=0 0 0
- joint joint3: origin xyz=0 -.6 0 rpy=0 0 0 -> xyz=0 .6 0 rpy=0 0 0
