Commit message: 2025_02_13, functioning, but clearly something wrong in gauging success

File: robot_one_arm.urdf (robot description, URDF)
Before this commit: robot robot, 37 links, 36 joints
Links:
- removed link arm_sensor_0_stop
- removed link hand_1_sensor_0_top
- removed link shoulder_sensor_0_bottom
- link arm: mass 10 -> 2
- link hand_1: mass 10 -> 2
- link shoulder: mass 10 -> 2; geometry collision box size=0.4 0.4 0.6; visual box size=0.4 0.4 0.6
- link shoulder_sensor_0_left: geometry collision box size=0.4 0.02 0.6; visual box size=0.4 0.02 0.6
- link shoulder_sensor_0_right: geometry collision box size=0.4 0.02 0.6; visual box size=0.4 0.02 0.6
- link shoulder_sensor_0_start: geometry collision box size=0.02 0.4 0.6; visual box size=0.02 0.4 0.6
- link shoulder_sensor_0_stop: geometry collision box size=0.02 0.4 0.6; visual box size=0.02 0.4 0.6
Joints:
- removed joint arm_arm_sensor_0_stop_joint
- removed joint hand_1_hand_1_sensor_0_top_joint
- removed joint shoulder_shoulder_sensor_0_bottom_joint
- joint body_shoulder_joint: origin xyz=0 0 0.7 rpy=0 0 0 -> xyz=0 0 0.8 rpy=0 0 0
- joint shoulder_arm_joint: origin xyz=1.575 0 0.2 rpy=0 0 0 -> xyz=1.575 0 0.1 rpy=0 0 0
- joint shoulder_shoulder_sensor_0_top_joint: origin xyz=0 0 0.4 rpy=0 0 0 -> xyz=0 0 0.3 rpy=0 0 0
