Commit message: 2025_03_06, no test. Updated variable names, implemented any number of joints. Now: Acceleration!

File: robot_four_side_arm.urdf (robot description, URDF)
Before this commit: robot robot, 74 links, 73 joints
Links:
- added link back_left_wheel, mass 0.1; collision cylinder length=0.1 radius=0.1; visual cylinder length=0.1 radius=0.1
- added link back_right_wheel, mass 0.1; collision cylinder length=0.1 radius=0.1; visual cylinder length=0.1 radius=0.1
- added link from_left_wheel, mass 0.1; collision cylinder length=0.1 radius=0.1; visual cylinder length=0.1 radius=0.1
- added link from_right_wheel, mass 0.1; collision cylinder length=0.1 radius=0.1; visual cylinder length=0.1 radius=0.1
Joints:
- added joint body_back_left_wheel_joint: type fixed, parent body, child back_left_wheel, origin xyz=-0.35 0.5 -0.4 rpy=1.5708 0 0, axis 1 0 0
- added joint body_back_right_wheel_joint: type fixed, parent body, child back_right_wheel, origin xyz=-0.35 -0.5 -0.4 rpy=1.5708 0 0, axis 1 0 0
- added joint body_from_left_wheel_joint: type fixed, parent body, child from_left_wheel, origin xyz=0.35 0.5 -0.4 rpy=1.5708 0 0, axis 1 0 0
- added joint body_from_right_wheel_joint: type fixed, parent body, child from_right_wheel, origin xyz=0.35 -0.5 -0.4 rpy=1.5708 0 0, axis 1 0 0

File: robot_two_head_arm_f.urdf (robot description, URDF)
Before this commit: robot robot, 105 links, 104 joints
Links:
- added link back_left_wheel, mass 0.1; collision cylinder length=0.1 radius=0.1; visual cylinder length=0.1 radius=0.1
- added link back_right_wheel, mass 0.1; collision cylinder length=0.1 radius=0.1; visual cylinder length=0.1 radius=0.1
- added link from_left_wheel, mass 0.1; collision cylinder length=0.1 radius=0.1; visual cylinder length=0.1 radius=0.1
- added link from_right_wheel, mass 0.1; collision cylinder length=0.1 radius=0.1; visual cylinder length=0.1 radius=0.1
Joints:
- added joint body_back_left_wheel_joint: type fixed, parent body, child back_left_wheel, origin xyz=-0.35 0.5 -0.4 rpy=1.5708 0 0, axis 1 0 0
- added joint body_back_right_wheel_joint: type fixed, parent body, child back_right_wheel, origin xyz=-0.35 -0.5 -0.4 rpy=1.5708 0 0, axis 1 0 0
- added joint body_from_left_wheel_joint: type fixed, parent body, child from_left_wheel, origin xyz=0.35 0.5 -0.4 rpy=1.5708 0 0, axis 1 0 0
- added joint body_from_right_wheel_joint: type fixed, parent body, child from_right_wheel, origin xyz=0.35 -0.5 -0.4 rpy=1.5708 0 0, axis 1 0 0

File: robot_two_head_arm_g.urdf (robot description, URDF)
Before this commit: robot robot, 105 links, 104 joints
Links:
- added link back_left_wheel, mass 0.1; collision cylinder length=0.1 radius=0.1; visual cylinder length=0.1 radius=0.1
- added link back_right_wheel, mass 0.1; collision cylinder length=0.1 radius=0.1; visual cylinder length=0.1 radius=0.1
- added link from_left_wheel, mass 0.1; collision cylinder length=0.1 radius=0.1; visual cylinder length=0.1 radius=0.1
- added link from_right_wheel, mass 0.1; collision cylinder length=0.1 radius=0.1; visual cylinder length=0.1 radius=0.1
Joints:
- added joint body_back_left_wheel_joint: type fixed, parent body, child back_left_wheel, origin xyz=-0.35 0.5 -0.4 rpy=1.5708 0 0, axis 1 0 0
- added joint body_back_right_wheel_joint: type fixed, parent body, child back_right_wheel, origin xyz=-0.35 -0.5 -0.4 rpy=1.5708 0 0, axis 1 0 0
- added joint body_from_left_wheel_joint: type fixed, parent body, child from_left_wheel, origin xyz=0.35 0.5 -0.4 rpy=1.5708 0 0, axis 1 0 0
- added joint body_from_right_wheel_joint: type fixed, parent body, child from_right_wheel, origin xyz=0.35 -0.5 -0.4 rpy=1.5708 0 0, axis 1 0 0

File: robot_two_side_arm.urdf (robot description, URDF)
Before this commit: robot robot, 72 links, 71 joints
Links:
- added link back_left_wheel, mass 0.1; collision cylinder length=0.1 radius=0.1; visual cylinder length=0.1 radius=0.1
- added link back_right_wheel, mass 0.1; collision cylinder length=0.1 radius=0.1; visual cylinder length=0.1 radius=0.1
- added link from_left_wheel, mass 0.1; collision cylinder length=0.1 radius=0.1; visual cylinder length=0.1 radius=0.1
- added link from_right_wheel, mass 0.1; collision cylinder length=0.1 radius=0.1; visual cylinder length=0.1 radius=0.1
Joints:
- added joint body_back_left_wheel_joint: type fixed, parent body, child back_left_wheel, origin xyz=-0.35 0.5 -0.4 rpy=1.5708 0 0, axis 1 0 0
- added joint body_back_right_wheel_joint: type fixed, parent body, child back_right_wheel, origin xyz=-0.35 -0.5 -0.4 rpy=1.5708 0 0, axis 1 0 0
- added joint body_from_left_wheel_joint: type fixed, parent body, child from_left_wheel, origin xyz=0.35 0.5 -0.4 rpy=1.5708 0 0, axis 1 0 0
- added joint body_from_right_wheel_joint: type fixed, parent body, child from_right_wheel, origin xyz=0.35 -0.5 -0.4 rpy=1.5708 0 0, axis 1 0 0
