Commit message: 2025_03_26. Big test, great results. But, pushing left/right doesn't make object move across vision.

File: robot_two_head_arm_a.urdf (robot description, URDF)
Before this commit: robot robot, 43 links, 42 joints
Links:
- removed link arm_sensor_0_start
- link hand: geometry collision box size=1 0.6000000000000001 1.25; visual box size=1 0.6000000000000001 1.25
- link hand_sensor_0_bottom: geometry collision box size=1.0 0.6000000000000001 0.02; visual box size=1.0 0.6000000000000001 0.02
- link hand_sensor_0_start: geometry collision box size=0.02 0.6000000000000001 1.25; visual box size=0.02 0.6000000000000001 1.25
- link hand_sensor_0_stop: geometry collision box size=0.02 0.6000000000000001 1.25; visual box size=0.02 0.6000000000000001 1.25
- link hand_sensor_0_top: geometry collision box size=1.0 0.6000000000000001 0.02; visual box size=1.0 0.6000000000000001 0.02
Joints:
- removed joint arm_arm_sensor_0_start_joint
- joint hand_hand_sensor_0_left_joint: origin xyz=0 0.1 0 rpy=0 0 0 -> xyz=0 0.30000000000000004 0 rpy=0 0 0
- joint hand_hand_sensor_0_right_joint: origin xyz=0 -0.1 0 rpy=0 0 0 -> xyz=0 -0.30000000000000004 0 rpy=0 0 0

Commit message: 2025_03_31. Big test, failed: the harder left/right seems impossible.

File: robot_two_head_arm_a.urdf (robot description, URDF)
Before this commit: robot robot, 42 links, 41 joints
Links:
- removed link joint_1_sensor_0_left
- removed link joint_1_sensor_0_right
- removed link joint_1_sensor_0_start
- removed link joint_1_sensor_0_stop
- removed link joint_2_sensor_0_left
- removed link joint_2_sensor_0_right
- removed link joint_2_sensor_0_stop
- removed link joint_2_sensor_0_top
Joints:
- removed joint joint_1_joint_1_sensor_0_left_joint
- removed joint joint_1_joint_1_sensor_0_right_joint
- removed joint joint_1_joint_1_sensor_0_start_joint
- removed joint joint_1_joint_1_sensor_0_stop_joint
- removed joint joint_2_joint_2_sensor_0_left_joint
- removed joint joint_2_joint_2_sensor_0_right_joint
- removed joint joint_2_joint_2_sensor_0_stop_joint
- removed joint joint_2_joint_2_sensor_0_top_joint
