Commit message: 2025_07_16. Big test. Trying different touch-hyperparameters.

File: robot_2.urdf (robot description, URDF)
Before this commit: robot robot, 65 links, 64 joints
Links:
- removed link hand_sensor_0_stop
- added link hand_sensor_1_bottom, mass 0; collision box size=0.14285714285714285 0.6000000000000001 0.03; visual box size=0.14285714285714285 0.6000000000000001 0.03
- added link hand_sensor_1_left, mass 0; collision box size=0.14285714285714285 0.03 1.25; visual box size=0.14285714285714285 0.03 1.25
- added link hand_sensor_1_right, mass 0; collision box size=0.14285714285714285 0.03 1.25; visual box size=0.14285714285714285 0.03 1.25
- added link hand_sensor_1_top, mass 0; collision box size=0.14285714285714285 0.6000000000000001 0.03; visual box size=0.14285714285714285 0.6000000000000001 0.03
- added link hand_sensor_2_bottom, mass 0; collision box size=0.14285714285714285 0.6000000000000001 0.03; visual box size=0.14285714285714285 0.6000000000000001 0.03
- added link hand_sensor_2_left, mass 0; collision box size=0.14285714285714285 0.03 1.25; visual box size=0.14285714285714285 0.03 1.25
- added link hand_sensor_2_right, mass 0; collision box size=0.14285714285714285 0.03 1.25; visual box size=0.14285714285714285 0.03 1.25
- added link hand_sensor_2_top, mass 0; collision box size=0.14285714285714285 0.6000000000000001 0.03; visual box size=0.14285714285714285 0.6000000000000001 0.03
- added link hand_sensor_3_bottom, mass 0; collision box size=0.14285714285714285 0.6000000000000001 0.03; visual box size=0.14285714285714285 0.6000000000000001 0.03
- added link hand_sensor_3_left, mass 0; collision box size=0.14285714285714285 0.03 1.25; visual box size=0.14285714285714285 0.03 1.25
- added link hand_sensor_3_right, mass 0; collision box size=0.14285714285714285 0.03 1.25; visual box size=0.14285714285714285 0.03 1.25
- added link hand_sensor_3_top, mass 0; collision box size=0.14285714285714285 0.6000000000000001 0.03; visual box size=0.14285714285714285 0.6000000000000001 0.03
- added link hand_sensor_4_bottom, mass 0; collision box size=0.14285714285714285 0.6000000000000001 0.03; visual box size=0.14285714285714285 0.6000000000000001 0.03
- added link hand_sensor_4_left, mass 0; collision box size=0.14285714285714285 0.03 1.25; visual box size=0.14285714285714285 0.03 1.25
- added link hand_sensor_4_right, mass 0; collision box size=0.14285714285714285 0.03 1.25; visual box size=0.14285714285714285 0.03 1.25
- added link hand_sensor_4_top, mass 0; collision box size=0.14285714285714285 0.6000000000000001 0.03; visual box size=0.14285714285714285 0.6000000000000001 0.03
- added link hand_sensor_5_bottom, mass 0; collision box size=0.14285714285714285 0.6000000000000001 0.03; visual box size=0.14285714285714285 0.6000000000000001 0.03
- added link hand_sensor_5_left, mass 0; collision box size=0.14285714285714285 0.03 1.25; visual box size=0.14285714285714285 0.03 1.25
- added link hand_sensor_5_right, mass 0; collision box size=0.14285714285714285 0.03 1.25; visual box size=0.14285714285714285 0.03 1.25
- added link hand_sensor_5_top, mass 0; collision box size=0.14285714285714285 0.6000000000000001 0.03; visual box size=0.14285714285714285 0.6000000000000001 0.03
- added link hand_sensor_6_bottom, mass 0; collision box size=0.14285714285714285 0.6000000000000001 0.03; visual box size=0.14285714285714285 0.6000000000000001 0.03
- added link hand_sensor_6_left, mass 0; collision box size=0.14285714285714285 0.03 1.25; visual box size=0.14285714285714285 0.03 1.25
- added link hand_sensor_6_right, mass 0; collision box size=0.14285714285714285 0.03 1.25; visual box size=0.14285714285714285 0.03 1.25
- added link hand_sensor_6_stop, mass 0; collision box size=0.03 0.6000000000000001 1.25; visual box size=0.03 0.6000000000000001 1.25
- added link hand_sensor_6_top, mass 0; collision box size=0.14285714285714285 0.6000000000000001 0.03; visual box size=0.14285714285714285 0.6000000000000001 0.03
- link arm: geometry collision box size=1.75 0.2 0.2; visual box size=1.75 0.2 0.2
- link arm_outline_1: geometry collision box size=1.75 0.005 0.005; visual box size=1.75 0.005 0.005
- link arm_outline_2: geometry collision box size=1.75 0.005 0.005; visual box size=1.75 0.005 0.005
- link arm_outline_3: geometry collision box size=1.75 0.005 0.005; visual box size=1.75 0.005 0.005
- link arm_outline_4: geometry collision box size=1.75 0.005 0.005; visual box size=1.75 0.005 0.005
- link arm_sensor_0_bottom: geometry collision box size=1.75 0.2 0.03; visual box size=1.75 0.2 0.03
- link arm_sensor_0_left: geometry collision box size=1.75 0.03 0.2; visual box size=1.75 0.03 0.2
- link arm_sensor_0_right: geometry collision box size=1.75 0.03 0.2; visual box size=1.75 0.03 0.2
- link arm_sensor_0_top: geometry collision box size=1.75 0.2 0.03; visual box size=1.75 0.2 0.03
- link hand_sensor_0_bottom: geometry collision box size=0.14285714285714285 0.6000000000000001 0.03; visual box size=0.14285714285714285 0.6000000000000001 0.03
- link hand_sensor_0_left: geometry collision box size=0.14285714285714285 0.03 1.25; visual box size=0.14285714285714285 0.03 1.25
- link hand_sensor_0_right: geometry collision box size=0.14285714285714285 0.03 1.25; visual box size=0.14285714285714285 0.03 1.25
- link hand_sensor_0_top: geometry collision box size=0.14285714285714285 0.6000000000000001 0.03; visual box size=0.14285714285714285 0.6000000000000001 0.03
Joints:
- removed joint hand_hand_sensor_0_stop_joint
- added joint hand_hand_sensor_1_bottom_joint: type fixed, parent hand, child hand_sensor_1_bottom, origin xyz=-0.28571428571428575 0 -0.625 rpy=0 0 0, axis 0 1 0
- added joint hand_hand_sensor_1_left_joint: type fixed, parent hand, child hand_sensor_1_left, origin xyz=-0.28571428571428575 0.30000000000000004 0 rpy=0 0 0, axis 0 1 0
- added joint hand_hand_sensor_1_right_joint: type fixed, parent hand, child hand_sensor_1_right, origin xyz=-0.28571428571428575 -0.30000000000000004 0 rpy=0 0 0, axis 0 1 0
- added joint hand_hand_sensor_1_top_joint: type fixed, parent hand, child hand_sensor_1_top, origin xyz=-0.28571428571428575 0 0.625 rpy=0 0 0, axis 0 1 0
- added joint hand_hand_sensor_2_bottom_joint: type fixed, parent hand, child hand_sensor_2_bottom, origin xyz=-0.1428571428571429 0 -0.625 rpy=0 0 0, axis 0 1 0
- added joint hand_hand_sensor_2_left_joint: type fixed, parent hand, child hand_sensor_2_left, origin xyz=-0.1428571428571429 0.30000000000000004 0 rpy=0 0 0, axis 0 1 0
- added joint hand_hand_sensor_2_right_joint: type fixed, parent hand, child hand_sensor_2_right, origin xyz=-0.1428571428571429 -0.30000000000000004 0 rpy=0 0 0, axis 0 1 0
- added joint hand_hand_sensor_2_top_joint: type fixed, parent hand, child hand_sensor_2_top, origin xyz=-0.1428571428571429 0 0.625 rpy=0 0 0, axis 0 1 0
- added joint hand_hand_sensor_3_bottom_joint: type fixed, parent hand, child hand_sensor_3_bottom, origin xyz=-5.551115123125783e-17 0 -0.625 rpy=0 0 0, axis 0 1 0
- added joint hand_hand_sensor_3_left_joint: type fixed, parent hand, child hand_sensor_3_left, origin xyz=-5.551115123125783e-17 0.30000000000000004 0 rpy=0 0 0, axis 0 1 0
- added joint hand_hand_sensor_3_right_joint: type fixed, parent hand, child hand_sensor_3_right, origin xyz=-5.551115123125783e-17 -0.30000000000000004 0 rpy=0 0 0, axis 0 1 0
- added joint hand_hand_sensor_3_top_joint: type fixed, parent hand, child hand_sensor_3_top, origin xyz=-5.551115123125783e-17 0 0.625 rpy=0 0 0, axis 0 1 0
- added joint hand_hand_sensor_4_bottom_joint: type fixed, parent hand, child hand_sensor_4_bottom, origin xyz=0.1428571428571428 0 -0.625 rpy=0 0 0, axis 0 1 0
- added joint hand_hand_sensor_4_left_joint: type fixed, parent hand, child hand_sensor_4_left, origin xyz=0.1428571428571428 0.30000000000000004 0 rpy=0 0 0, axis 0 1 0
- added joint hand_hand_sensor_4_right_joint: type fixed, parent hand, child hand_sensor_4_right, origin xyz=0.1428571428571428 -0.30000000000000004 0 rpy=0 0 0, axis 0 1 0
- added joint hand_hand_sensor_4_top_joint: type fixed, parent hand, child hand_sensor_4_top, origin xyz=0.1428571428571428 0 0.625 rpy=0 0 0, axis 0 1 0
- added joint hand_hand_sensor_5_bottom_joint: type fixed, parent hand, child hand_sensor_5_bottom, origin xyz=0.28571428571428564 0 -0.625 rpy=0 0 0, axis 0 1 0
- added joint hand_hand_sensor_5_left_joint: type fixed, parent hand, child hand_sensor_5_left, origin xyz=0.28571428571428564 0.30000000000000004 0 rpy=0 0 0, axis 0 1 0
- added joint hand_hand_sensor_5_right_joint: type fixed, parent hand, child hand_sensor_5_right, origin xyz=0.28571428571428564 -0.30000000000000004 0 rpy=0 0 0, axis 0 1 0
- added joint hand_hand_sensor_5_top_joint: type fixed, parent hand, child hand_sensor_5_top, origin xyz=0.28571428571428564 0 0.625 rpy=0 0 0, axis 0 1 0
- added joint hand_hand_sensor_6_bottom_joint: type fixed, parent hand, child hand_sensor_6_bottom, origin xyz=0.4285714285714285 0 -0.625 rpy=0 0 0, axis 0 1 0
- added joint hand_hand_sensor_6_left_joint: type fixed, parent hand, child hand_sensor_6_left, origin xyz=0.4285714285714285 0.30000000000000004 0 rpy=0 0 0, axis 0 1 0
- added joint hand_hand_sensor_6_right_joint: type fixed, parent hand, child hand_sensor_6_right, origin xyz=0.4285714285714285 -0.30000000000000004 0 rpy=0 0 0, axis 0 1 0
- added joint hand_hand_sensor_6_stop_joint: type fixed, parent hand, child hand_sensor_6_stop, origin xyz=-0.5 0 0 rpy=0 0 0, axis 0 1 0
- added joint hand_hand_sensor_6_top_joint: type fixed, parent hand, child hand_sensor_6_top, origin xyz=0.4285714285714285 0 0.625 rpy=0 0 0, axis 0 1 0
- joint arm_arm_outline_5_joint: origin xyz=0.6475 0.10250000000000001 0 rpy=0 0 0 -> xyz=0.8724999999999999 0.10250000000000001 0 rpy=0 0 0
- joint arm_arm_outline_6_joint: origin xyz=0.6475 -0.10250000000000001 0 rpy=0 0 0 -> xyz=0.8724999999999999 -0.10250000000000001 0 rpy=0 0 0
- joint arm_arm_outline_7_joint: origin xyz=0.6475 0 -0.10250000000000001 rpy=0 0 0 -> xyz=0.8724999999999999 0 -0.10250000000000001 rpy=0 0 0
- joint arm_hand_joint: origin xyz=1.15 0 -0.525 rpy=0 0 0 -> xyz=1.375 0 -0.525 rpy=0 0 0
- joint hand_hand_sensor_0_bottom_joint: origin xyz=0 0 -0.625 rpy=0 0 0 -> xyz=-0.4285714285714286 0 -0.625 rpy=0 0 0
- joint hand_hand_sensor_0_left_joint: origin xyz=0 0.30000000000000004 0 rpy=0 0 0 -> xyz=-0.4285714285714286 0.30000000000000004 0 rpy=0 0 0
- joint hand_hand_sensor_0_right_joint: origin xyz=0 -0.30000000000000004 0 rpy=0 0 0 -> xyz=-0.4285714285714286 -0.30000000000000004 0 rpy=0 0 0
- joint hand_hand_sensor_0_top_joint: origin xyz=0 0 0.625 rpy=0 0 0 -> xyz=-0.4285714285714286 0 0.625 rpy=0 0 0
- joint joint_2_arm_joint: origin xyz=0.75 0 0 rpy=0 0 0 -> xyz=0.975 0 0 rpy=0 0 0
