Commit message: adjusted awarding, adding face-mask

File: robot.urdf (robot description, URDF)
Before this commit: robot robot, 58 links, 57 joints
Links:
- link arrow_0: geometry collision box size=0.05 0.5 0.02; visual box size=0.05 0.5 0.02
- link arrow_1: geometry collision box size=0.05 0.45 0.02; visual box size=0.05 0.45 0.02
- link arrow_2: geometry collision box size=0.05 0.4 0.02; visual box size=0.05 0.4 0.02
- link arrow_3: geometry collision box size=0.05 0.35 0.02; visual box size=0.05 0.35 0.02
- link arrow_4: geometry collision box size=0.05 0.3 0.02; visual box size=0.05 0.3 0.02
- link arrow_5: geometry collision box size=0.05 0.25 0.02; visual box size=0.05 0.25 0.02
- link arrow_6: geometry collision box size=0.05 0.19999999999999996 0.02; visual box size=0.05 0.19999999999999996 0.02
- link arrow_7: geometry collision box size=0.05 0.14999999999999997 0.02; visual box size=0.05 0.14999999999999997 0.02
- link arrow_8: geometry collision box size=0.05 0.09999999999999998 0.02; visual box size=0.05 0.09999999999999998 0.02
- link arrow_9: geometry collision box size=0.05 0.04999999999999999 0.02; visual box size=0.05 0.04999999999999999 0.02
- link arrow_base: geometry collision box size=0.3 0.2 0.02; visual box size=0.3 0.2 0.02
Joints:
- joint body_arrow_base_joint: origin xyz=-0.24999999999999997 0 0.50000001 rpy=0 0 0 -> xyz=-0.24999999999999997 0 0.51 rpy=0 0 0

Commit message: still working

File: robot.urdf (robot description, URDF)
Before this commit: robot robot, 58 links, 57 joints
Links:
- removed link arrow_0
- removed link arrow_1
- removed link arrow_2
- removed link arrow_3
- removed link arrow_4
- removed link arrow_5
- removed link arrow_6
- removed link arrow_7
- removed link arrow_8
- removed link arrow_9
- removed link arrow_base
- added link body_square_0, mass 0; collision box size=0.002 0.1111111111111111 0.1111111111111111; visual box size=0.002 0.1111111111111111 0.1111111111111111
- added link body_square_1, mass 0; collision box size=0.002 0.1111111111111111 0.1111111111111111; visual box size=0.002 0.1111111111111111 0.1111111111111111
- added link body_square_10, mass 0; collision box size=0.1111111111111111 0.1111111111111111 0.002; visual box size=0.1111111111111111 0.1111111111111111 0.002
- added link body_square_11, mass 0; collision box size=0.1111111111111111 0.1111111111111111 0.002; visual box size=0.1111111111111111 0.1111111111111111 0.002
- added link body_square_12, mass 0; collision box size=0.1111111111111111 0.1111111111111111 0.002; visual box size=0.1111111111111111 0.1111111111111111 0.002
- added link body_square_13, mass 0; collision box size=0.1111111111111111 0.1111111111111111 0.002; visual box size=0.1111111111111111 0.1111111111111111 0.002
- added link body_square_14, mass 0; collision box size=0.1111111111111111 0.1111111111111111 0.002; visual box size=0.1111111111111111 0.1111111111111111 0.002
- added link body_square_15, mass 0; collision box size=0.1111111111111111 0.1111111111111111 0.002; visual box size=0.1111111111111111 0.1111111111111111 0.002
- added link body_square_16, mass 0; collision box size=0.1111111111111111 0.1111111111111111 0.002; visual box size=0.1111111111111111 0.1111111111111111 0.002
- added link body_square_17, mass 0; collision box size=0.1111111111111111 0.1111111111111111 0.002; visual box size=0.1111111111111111 0.1111111111111111 0.002
- added link body_square_18, mass 0; collision box size=0.1111111111111111 0.1111111111111111 0.002; visual box size=0.1111111111111111 0.1111111111111111 0.002
- added link body_square_19, mass 0; collision box size=0.1111111111111111 0.1111111111111111 0.002; visual box size=0.1111111111111111 0.1111111111111111 0.002
- added link body_square_2, mass 0; collision box size=0.002 0.1111111111111111 0.1111111111111111; visual box size=0.002 0.1111111111111111 0.1111111111111111
- added link body_square_3, mass 0; collision box size=0.002 0.1111111111111111 0.1111111111111111; visual box size=0.002 0.1111111111111111 0.1111111111111111
- added link body_square_4, mass 0; collision box size=0.002 0.1111111111111111 0.1111111111111111; visual box size=0.002 0.1111111111111111 0.1111111111111111
- added link body_square_5, mass 0; collision box size=0.002 0.1111111111111111 0.1111111111111111; visual box size=0.002 0.1111111111111111 0.1111111111111111
- added link body_square_6, mass 0; collision box size=0.002 0.1111111111111111 0.1111111111111111; visual box size=0.002 0.1111111111111111 0.1111111111111111
- added link body_square_7, mass 0; collision box size=0.002 0.1111111111111111 0.1111111111111111; visual box size=0.002 0.1111111111111111 0.1111111111111111
- added link body_square_8, mass 0; collision box size=0.002 0.1111111111111111 0.1111111111111111; visual box size=0.002 0.1111111111111111 0.1111111111111111
- added link body_square_9, mass 0; collision box size=0.1111111111111111 0.1111111111111111 0.002; visual box size=0.1111111111111111 0.1111111111111111 0.002
Joints:
- removed joint arrow_0_arrow_1_joint
- removed joint arrow_1_arrow_2_joint
- removed joint arrow_2_arrow_3_joint
- removed joint arrow_3_arrow_4_joint
- removed joint arrow_4_arrow_5_joint
- removed joint arrow_5_arrow_6_joint
- removed joint arrow_6_arrow_7_joint
- removed joint arrow_7_arrow_8_joint
- removed joint arrow_8_arrow_9_joint
- removed joint arrow_base_arrow_0_joint
- removed joint body_arrow_base_joint
- added joint body_body_square_0_joint: type fixed, parent body, child body_square_0, origin xyz=0.501 -0.33333333333333337 0.11111111111111116 rpy=0 0 0, axis 0 0 1
- added joint body_body_square_10_joint: type fixed, parent body, child body_square_10, origin xyz=0.2222222222222222 -0.1111111111111111 0.501 rpy=0 0 0, axis 0 0 1
- added joint body_body_square_11_joint: type fixed, parent body, child body_square_11, origin xyz=-0.33333333333333337 0.0 0.501 rpy=0 0 0, axis 0 0 1
- added joint body_body_square_12_joint: type fixed, parent body, child body_square_12, origin xyz=-0.2222222222222222 0.0 0.501 rpy=0 0 0, axis 0 0 1
- added joint body_body_square_13_joint: type fixed, parent body, child body_square_13, origin xyz=-0.1111111111111111 0.0 0.501 rpy=0 0 0, axis 0 0 1
- added joint body_body_square_14_joint: type fixed, parent body, child body_square_14, origin xyz=0.0 0.0 0.501 rpy=0 0 0, axis 0 0 1
- added joint body_body_square_15_joint: type fixed, parent body, child body_square_15, origin xyz=0.11111111111111116 0.0 0.501 rpy=0 0 0, axis 0 0 1
- added joint body_body_square_16_joint: type fixed, parent body, child body_square_16, origin xyz=0.2222222222222222 0.0 0.501 rpy=0 0 0, axis 0 0 1
- added joint body_body_square_17_joint: type fixed, parent body, child body_square_17, origin xyz=0.33333333333333337 0.0 0.501 rpy=0 0 0, axis 0 0 1
- added joint body_body_square_18_joint: type fixed, parent body, child body_square_18, origin xyz=0.2222222222222222 0.11111111111111116 0.501 rpy=0 0 0, axis 0 0 1
- added joint body_body_square_19_joint: type fixed, parent body, child body_square_19, origin xyz=0.11111111111111116 0.2222222222222222 0.501 rpy=0 0 0, axis 0 0 1
- added joint body_body_square_1_joint: type fixed, parent body, child body_square_1, origin xyz=0.501 -0.2222222222222222 0.2222222222222222 rpy=0 0 0, axis 0 0 1
- added joint body_body_square_2_joint: type fixed, parent body, child body_square_2, origin xyz=0.501 -0.1111111111111111 0.11111111111111116 rpy=0 0 0, axis 0 0 1
- added joint body_body_square_3_joint: type fixed, parent body, child body_square_3, origin xyz=0.501 -0.1111111111111111 -0.2222222222222222 rpy=0 0 0, axis 0 0 1
- added joint body_body_square_4_joint: type fixed, parent body, child body_square_4, origin xyz=0.501 0.0 -0.2222222222222222 rpy=0 0 0, axis 0 0 1
- added joint body_body_square_5_joint: type fixed, parent body, child body_square_5, origin xyz=0.501 0.11111111111111116 0.11111111111111116 rpy=0 0 0, axis 0 0 1
- added joint body_body_square_6_joint: type fixed, parent body, child body_square_6, origin xyz=0.501 0.11111111111111116 -0.2222222222222222 rpy=0 0 0, axis 0 0 1
- added joint body_body_square_7_joint: type fixed, parent body, child body_square_7, origin xyz=0.501 0.2222222222222222 0.2222222222222222 rpy=0 0 0, axis 0 0 1
- added joint body_body_square_8_joint: type fixed, parent body, child body_square_8, origin xyz=0.501 0.33333333333333337 0.11111111111111116 rpy=0 0 0, axis 0 0 1
- added joint body_body_square_9_joint: type fixed, parent body, child body_square_9, origin xyz=0.11111111111111116 -0.2222222222222222 0.501 rpy=0 0 0, axis 0 0 1

Commit message: tried cube-objects

File: robot.urdf (robot description, URDF)
Before this commit: robot robot, 67 links, 66 joints
Links:
- removed link hand
- removed link hand_sensor_0_bottom
- removed link hand_sensor_0_left
- removed link hand_sensor_0_right
- removed link hand_sensor_0_top
- removed link hand_sensor_1_bottom
- removed link hand_sensor_1_left
- removed link hand_sensor_1_right
- removed link hand_sensor_1_top
- added link left_hand, mass 0.1; collision box size=0.4 0.7 0.5; visual box size=0.4 0.7 0.5
- added link left_hand_sensor_0_bottom, mass 0; collision box size=0.02 0.7 0.5; visual box size=0.02 0.7 0.5
- added link left_hand_sensor_0_left, mass 0; collision box size=0.4 0.7 0.02; visual box size=0.4 0.7 0.02
- added link left_hand_sensor_0_right, mass 0; collision box size=0.4 0.7 0.02; visual box size=0.4 0.7 0.02
- added link left_hand_sensor_0_stop, mass 0; collision box size=0.4 0.02 0.5; visual box size=0.4 0.02 0.5
- added link left_hand_sensor_0_top, mass 0; collision box size=0.02 0.7 0.5; visual box size=0.02 0.7 0.5
- added link right_hand, mass 0.1; collision box size=0.4 0.7 0.5; visual box size=0.4 0.7 0.5
- added link right_hand_sensor_0_bottom, mass 0; collision box size=0.02 0.7 0.5; visual box size=0.02 0.7 0.5
- added link right_hand_sensor_0_left, mass 0; collision box size=0.4 0.7 0.02; visual box size=0.4 0.7 0.02
- added link right_hand_sensor_0_right, mass 0; collision box size=0.4 0.7 0.02; visual box size=0.4 0.7 0.02
- added link right_hand_sensor_0_start, mass 0; collision box size=0.4 0.02 0.5; visual box size=0.4 0.02 0.5
- added link right_hand_sensor_0_top, mass 0; collision box size=0.02 0.7 0.5; visual box size=0.02 0.7 0.5
- link left_arm: geometry collision box size=3 0.4 0.5; visual box size=3 0.4 0.5
- link left_arm_sensor_0_left: geometry collision box size=1.0 0.02 0.5; visual box size=1.0 0.02 0.5
- link left_arm_sensor_0_right: geometry collision box size=1.0 0.02 0.5; visual box size=1.0 0.02 0.5
- link left_arm_sensor_0_start: geometry collision box size=0.02 0.4 0.5; visual box size=0.02 0.4 0.5
- link left_arm_sensor_1_left: geometry collision box size=1.0 0.02 0.5; visual box size=1.0 0.02 0.5
- link left_arm_sensor_1_right: geometry collision box size=1.0 0.02 0.5; visual box size=1.0 0.02 0.5
- link left_arm_sensor_2_left: geometry collision box size=1.0 0.02 0.5; visual box size=1.0 0.02 0.5
- link left_arm_sensor_2_right: geometry collision box size=1.0 0.02 0.5; visual box size=1.0 0.02 0.5
- link left_arm_sensor_2_stop: geometry collision box size=0.02 0.4 0.5; visual box size=0.02 0.4 0.5
- link left_shoulder: geometry collision box size=0.4 0.3 0.5; visual box size=0.4 0.3 0.5
- link right_arm: geometry collision box size=3 0.4 0.5; visual box size=3 0.4 0.5
- link right_arm_sensor_0_left: geometry collision box size=1.0 0.02 0.5; visual box size=1.0 0.02 0.5
- link right_arm_sensor_0_right: geometry collision box size=1.0 0.02 0.5; visual box size=1.0 0.02 0.5
- link right_arm_sensor_0_start: geometry collision box size=0.02 0.4 0.5; visual box size=0.02 0.4 0.5
- link right_arm_sensor_1_left: geometry collision box size=1.0 0.02 0.5; visual box size=1.0 0.02 0.5
- link right_arm_sensor_1_right: geometry collision box size=1.0 0.02 0.5; visual box size=1.0 0.02 0.5
- link right_arm_sensor_2_left: geometry collision box size=1.0 0.02 0.5; visual box size=1.0 0.02 0.5
- link right_arm_sensor_2_right: geometry collision box size=1.0 0.02 0.5; visual box size=1.0 0.02 0.5
- link right_arm_sensor_2_stop: geometry collision box size=0.02 0.4 0.5; visual box size=0.02 0.4 0.5
- link right_shoulder: geometry collision box size=0.4 0.3 0.5; visual box size=0.4 0.3 0.5
Joints:
- removed joint hand_hand_sensor_0_bottom_joint
- removed joint hand_hand_sensor_0_left_joint
- removed joint hand_hand_sensor_0_right_joint
- removed joint hand_hand_sensor_0_top_joint
- removed joint hand_hand_sensor_1_bottom_joint
- removed joint hand_hand_sensor_1_left_joint
- removed joint hand_hand_sensor_1_right_joint
- removed joint hand_hand_sensor_1_top_joint
- removed joint hand_right_arm_joint
- removed joint left_arm_hand_joint
- removed joint right_arm_right_shoulder_joint
- added joint body_right_shoulder_joint: type continuous, parent body, child right_shoulder, origin xyz=0 -0.65 0 rpy=0 0 0, axis 0 -1 0
- added joint left_arm_left_hand_joint: type fixed, parent left_arm, child left_hand, origin xyz=1.3 -0.55 0 rpy=0 0 0, axis 0 0 0
- added joint left_hand_left_hand_sensor_0_bottom_joint: type fixed, parent left_hand, child left_hand_sensor_0_bottom, origin xyz=-0.2 0 0 rpy=0 0 0, axis 0 0 0
- added joint left_hand_left_hand_sensor_0_left_joint: type fixed, parent left_hand, child left_hand_sensor_0_left, origin xyz=0 0 0.25 rpy=0 0 0, axis 0 0 0
- added joint left_hand_left_hand_sensor_0_right_joint: type fixed, parent left_hand, child left_hand_sensor_0_right, origin xyz=0 0 -0.25 rpy=0 0 0, axis 0 0 0
- added joint left_hand_left_hand_sensor_0_stop_joint: type fixed, parent left_hand, child left_hand_sensor_0_stop, origin xyz=0 -0.35 0 rpy=0 0 0, axis 0 0 0
- added joint left_hand_left_hand_sensor_0_top_joint: type fixed, parent left_hand, child left_hand_sensor_0_top, origin xyz=0.2 0 0 rpy=0 0 0, axis 0 0 0
- added joint right_arm_right_hand_joint: type fixed, parent right_arm, child right_hand, origin xyz=1.3 0.55 0 rpy=0 0 0, axis 0 0 0
- added joint right_hand_right_hand_sensor_0_bottom_joint: type fixed, parent right_hand, child right_hand_sensor_0_bottom, origin xyz=-0.2 0 0 rpy=0 0 0, axis 0 0 0
- added joint right_hand_right_hand_sensor_0_left_joint: type fixed, parent right_hand, child right_hand_sensor_0_left, origin xyz=0 0 0.25 rpy=0 0 0, axis 0 0 0
- added joint right_hand_right_hand_sensor_0_right_joint: type fixed, parent right_hand, child right_hand_sensor_0_right, origin xyz=0 0 -0.25 rpy=0 0 0, axis 0 0 0
- added joint right_hand_right_hand_sensor_0_start_joint: type fixed, parent right_hand, child right_hand_sensor_0_start, origin xyz=0 0.35 0 rpy=0 0 0, axis 0 0 0
- added joint right_hand_right_hand_sensor_0_top_joint: type fixed, parent right_hand, child right_hand_sensor_0_top, origin xyz=0.2 0 0 rpy=0 0 0, axis 0 0 0
- added joint right_shoulder_right_arm_joint: type fixed, parent right_shoulder, child right_arm, origin xyz=1.3 -0.35 0 rpy=0 0 0, axis 1 0 0
- joint left_arm_left_arm_sensor_0_bottom_joint: origin xyz=-1.0 0 -0.4 rpy=0 0 0 -> xyz=-1.0 0 -0.25 rpy=0 0 0
- joint left_arm_left_arm_sensor_0_top_joint: origin xyz=-1.0 0 0.4 rpy=0 0 0 -> xyz=-1.0 0 0.25 rpy=0 0 0
- joint left_arm_left_arm_sensor_1_bottom_joint: origin xyz=0.0 0 -0.4 rpy=0 0 0 -> xyz=0.0 0 -0.25 rpy=0 0 0
- joint left_arm_left_arm_sensor_1_top_joint: origin xyz=0.0 0 0.4 rpy=0 0 0 -> xyz=0.0 0 0.25 rpy=0 0 0
- joint left_arm_left_arm_sensor_2_bottom_joint: origin xyz=1.0 0 -0.4 rpy=0 0 0 -> xyz=1.0 0 -0.25 rpy=0 0 0
- joint left_arm_left_arm_sensor_2_top_joint: origin xyz=1.0 0 0.4 rpy=0 0 0 -> xyz=1.0 0 0.25 rpy=0 0 0
- joint right_arm_right_arm_sensor_0_bottom_joint: origin xyz=-1.0 0 -0.4 rpy=0 0 0 -> xyz=-1.0 0 -0.25 rpy=0 0 0
- joint right_arm_right_arm_sensor_0_top_joint: origin xyz=-1.0 0 0.4 rpy=0 0 0 -> xyz=-1.0 0 0.25 rpy=0 0 0
- joint right_arm_right_arm_sensor_1_bottom_joint: origin xyz=0.0 0 -0.4 rpy=0 0 0 -> xyz=0.0 0 -0.25 rpy=0 0 0
- joint right_arm_right_arm_sensor_1_top_joint: origin xyz=0.0 0 0.4 rpy=0 0 0 -> xyz=0.0 0 0.25 rpy=0 0 0
- joint right_arm_right_arm_sensor_2_bottom_joint: origin xyz=1.0 0 -0.4 rpy=0 0 0 -> xyz=1.0 0 -0.25 rpy=0 0 0
- joint right_arm_right_arm_sensor_2_top_joint: origin xyz=1.0 0 0.4 rpy=0 0 0 -> xyz=1.0 0 0.25 rpy=0 0 0

Commit message: 3d-interactive-plotting LDA

File: robot.urdf (robot description, URDF)
Before this commit: robot robot, 70 links, 69 joints
Links:
- added link body_square_20, mass 0; collision box size=0.1111111111111111 0.1111111111111111 0.002; visual box size=0.1111111111111111 0.1111111111111111 0.002
- added link body_square_21, mass 0; collision box size=0.1111111111111111 0.1111111111111111 0.002; visual box size=0.1111111111111111 0.1111111111111111 0.002
Joints:
- added joint body_body_square_20_joint: type fixed, parent body, child body_square_20, origin xyz=0.2222222222222222 0.11111111111111116 0.501 rpy=0 0 0, axis 0 0 1
- added joint body_body_square_21_joint: type fixed, parent body, child body_square_21, origin xyz=0.11111111111111116 0.2222222222222222 0.501 rpy=0 0 0, axis 0 0 1
- joint body_body_square_10_joint: origin xyz=0.2222222222222222 -0.1111111111111111 0.501 rpy=0 0 0 -> xyz=0.11111111111111116 -0.1111111111111111 0.501 rpy=0 0 0
- joint body_body_square_11_joint: origin xyz=-0.33333333333333337 0.0 0.501 rpy=0 0 0 -> xyz=0.2222222222222222 -0.1111111111111111 0.501 rpy=0 0 0
- joint body_body_square_12_joint: origin xyz=-0.2222222222222222 0.0 0.501 rpy=0 0 0 -> xyz=-0.33333333333333337 0.0 0.501 rpy=0 0 0
- joint body_body_square_13_joint: origin xyz=-0.1111111111111111 0.0 0.501 rpy=0 0 0 -> xyz=-0.2222222222222222 0.0 0.501 rpy=0 0 0
- joint body_body_square_14_joint: origin xyz=0.0 0.0 0.501 rpy=0 0 0 -> xyz=-0.1111111111111111 0.0 0.501 rpy=0 0 0
- joint body_body_square_15_joint: origin xyz=0.11111111111111116 0.0 0.501 rpy=0 0 0 -> xyz=0.0 0.0 0.501 rpy=0 0 0
- joint body_body_square_16_joint: origin xyz=0.2222222222222222 0.0 0.501 rpy=0 0 0 -> xyz=0.11111111111111116 0.0 0.501 rpy=0 0 0
- joint body_body_square_17_joint: origin xyz=0.33333333333333337 0.0 0.501 rpy=0 0 0 -> xyz=0.2222222222222222 0.0 0.501 rpy=0 0 0
- joint body_body_square_18_joint: origin xyz=0.2222222222222222 0.11111111111111116 0.501 rpy=0 0 0 -> xyz=0.33333333333333337 0.0 0.501 rpy=0 0 0
- joint body_body_square_19_joint: origin xyz=0.11111111111111116 0.2222222222222222 0.501 rpy=0 0 0 -> xyz=0.11111111111111116 0.11111111111111116 0.501 rpy=0 0 0

Commit message: 2025_01_20, new robot for better 3d thought (big test)

File: robot.urdf (robot description, URDF)
Before this commit: robot robot, 72 links, 71 joints
Links:
- link body: geometry collision box size=1 1 2.5; visual box size=1 1 2.5
- link body_sensor_0_left: geometry collision box size=1.0 0.02 2.5; visual box size=1.0 0.02 2.5
- link body_sensor_0_right: geometry collision box size=1.0 0.02 2.5; visual box size=1.0 0.02 2.5
- link body_sensor_0_start: geometry collision box size=0.02 1 2.5; visual box size=0.02 1 2.5
- link body_sensor_0_stop: geometry collision box size=0.02 1 2.5; visual box size=0.02 1 2.5
Joints:
- joint body_body_sensor_0_top_joint: origin xyz=0 0 0.5 rpy=0 0 0 -> xyz=0 0 1.25 rpy=0 0 0
- joint body_left_shoulder_joint: origin xyz=0 0.65 0 rpy=0 0 0 -> xyz=0 0.65 -0.75 rpy=0 0 0
- joint body_right_shoulder_joint: origin xyz=0 -0.65 0 rpy=0 0 0 -> xyz=0 -0.65 -0.75 rpy=0 0 0

Commit message: 2025_10_14. Working, maybe final?

File: robot.urdf (robot description, URDF)
Before this commit: robot robot, 69 links, 68 joints
Links:
- removed link body_face_front_0
- removed link body_face_front_1
- removed link body_face_front_2
- removed link body_face_front_3
- removed link body_face_front_4
- removed link body_face_front_5
- removed link body_face_front_6
- removed link body_face_front_7
- removed link body_face_front_8
Joints:
- removed joint body_body_face_front_0_joint
- removed joint body_body_face_front_1_joint
- removed joint body_body_face_front_2_joint
- removed joint body_body_face_front_3_joint
- removed joint body_body_face_front_4_joint
- removed joint body_body_face_front_5_joint
- removed joint body_body_face_front_6_joint
- removed joint body_body_face_front_7_joint
- removed joint body_body_face_front_8_joint

File: robot_2.urdf (robot description, URDF)
Before this commit: robot robot, 69 links, 68 joints
Links:
- removed link body_face_front_0
- removed link body_face_front_1
- removed link body_face_front_2
- removed link body_face_front_3
- removed link body_face_front_4
- removed link body_face_front_5
- removed link body_face_front_6
- removed link body_face_front_7
- removed link body_face_front_8
- link arm: geometry collision box size=1.75 0.2 0.2; visual box size=1.75 0.2 0.2
- link arm_outline_1: geometry collision box size=1.75 0.005 0.005; visual box size=1.75 0.005 0.005
- link arm_outline_2: geometry collision box size=1.75 0.005 0.005; visual box size=1.75 0.005 0.005
- link arm_outline_3: geometry collision box size=1.75 0.005 0.005; visual box size=1.75 0.005 0.005
- link arm_outline_4: geometry collision box size=1.75 0.005 0.005; visual box size=1.75 0.005 0.005
- link arm_sensor_0_bottom: geometry collision box size=1.75 0.2 0.03; visual box size=1.75 0.2 0.03
- link arm_sensor_0_left: geometry collision box size=1.75 0.03 0.2; visual box size=1.75 0.03 0.2
- link arm_sensor_0_right: geometry collision box size=1.75 0.03 0.2; visual box size=1.75 0.03 0.2
- link arm_sensor_0_top: geometry collision box size=1.75 0.2 0.03; visual box size=1.75 0.2 0.03
Joints:
- removed joint body_body_face_front_0_joint
- removed joint body_body_face_front_1_joint
- removed joint body_body_face_front_2_joint
- removed joint body_body_face_front_3_joint
- removed joint body_body_face_front_4_joint
- removed joint body_body_face_front_5_joint
- removed joint body_body_face_front_6_joint
- removed joint body_body_face_front_7_joint
- removed joint body_body_face_front_8_joint
- joint arm_arm_outline_5_joint: origin xyz=0.7474999999999999 0.10250000000000001 0 rpy=0 0 0 -> xyz=0.8724999999999999 0.10250000000000001 0 rpy=0 0 0
- joint arm_arm_outline_6_joint: origin xyz=0.7474999999999999 -0.10250000000000001 0 rpy=0 0 0 -> xyz=0.8724999999999999 -0.10250000000000001 0 rpy=0 0 0
- joint arm_arm_outline_7_joint: origin xyz=0.7474999999999999 0 -0.10250000000000001 rpy=0 0 0 -> xyz=0.8724999999999999 0 -0.10250000000000001 rpy=0 0 0
- joint arm_hand_joint: origin xyz=1.25 0 -0.525 rpy=0 0 0 -> xyz=1.375 0 -0.525 rpy=0 0 0
- joint joint_2_arm_joint: origin xyz=0.85 0 0 rpy=0 0 0 -> xyz=0.975 0 0 rpy=0 0 0
