Commit message: 2025_02_27, big test. Problem discovered: arm gets stuck!

File: pybullet_data/robots/robot_one_head_arm.urdf (robot description, URDF)
Before this commit: robot robot, 47 links, 46 joints
Links:
- link joint_1: geometry collision box size=0.4 0.4 0.6000000000000001; visual box size=0.4 0.4 0.6000000000000001
- link joint_1_sensor_0_left: geometry collision box size=0.4 0.02 0.6000000000000001; visual box size=0.4 0.02 0.6000000000000001
- link joint_1_sensor_0_right: geometry collision box size=0.4 0.02 0.6000000000000001; visual box size=0.4 0.02 0.6000000000000001
- link joint_1_sensor_0_start: geometry collision box size=0.02 0.4 0.6000000000000001; visual box size=0.02 0.4 0.6000000000000001
- link joint_1_sensor_0_stop: geometry collision box size=0.02 0.4 0.6000000000000001; visual box size=0.02 0.4 0.6000000000000001
Joints:
- joint joint_1_arm_joint: origin xyz=1.575 0 0.1 rpy=0 0 0 -> xyz=1.575 0 0.10000000000000003 rpy=0 0 0
- joint joint_1_joint_1_sensor_0_top_joint: origin xyz=0 0 0.3 rpy=0 0 0 -> xyz=0 0 0.30000000000000004 rpy=0 0 0

File: pybullet_data/robots/robot_two_head_arm.urdf (robot description, URDF)
Before this commit: robot robot, 53 links, 52 joints
Joints:
- joint joint_1_joint_2_joint: origin xyz=0 0 0.3 rpy=0 0 0 -> xyz=0 0 0.30000000000000004 rpy=0 0 0

File: pybullet_data/robots/robot_two_head_arm_b.urdf (robot description, URDF)
Before this commit: robot robot, 65 links, 64 joints
Joints:
- joint joint_1_joint_2_joint: origin xyz=0 0 0.3 rpy=0 0 0 -> xyz=0 0 0.30000000000000004 rpy=0 0 0

Commit message: 2025_03_01, big test, failed. Trying considerations and bigger cnn. Found problems in goal-detections.

File: pybullet_data/robots/robot_one_head_arm.urdf (robot description, URDF)
Before this commit: robot robot, 47 links, 46 joints
Links:
- removed link joint_1_sensor_0_start
Joints:
- removed joint joint_1_joint_1_sensor_0_start_joint

File: pybullet_data/robots/robot_two_head_arm.urdf (robot description, URDF)
Before this commit: robot robot, 53 links, 52 joints
Links:
- removed link joint_1_sensor_0_top
- removed link joint_2_sensor_0_start
Joints:
- removed joint joint_1_joint_1_sensor_0_top_joint
- removed joint joint_2_joint_2_sensor_0_start_joint

File: pybullet_data/robots/robot_two_head_arm_b.urdf (robot description, URDF)
Before this commit: robot robot, 65 links, 64 joints
Links:
- removed link hand_1_sensor_0_left
- removed link hand_1_sensor_0_right
- removed link joint_1_sensor_0_top
- removed link joint_2_sensor_0_start
- added link hand_1_sensor_0_top, mass 0; collision box size=0.4 1.3 0.02; visual box size=0.4 1.3 0.02
- added link hand_2_sensor_0_top, mass 0; collision box size=1.0 0.4 0.02; visual box size=1.0 0.4 0.02
- added link hand_3_sensor_0_top, mass 0; collision box size=1.0 0.4 0.02; visual box size=1.0 0.4 0.02
Joints:
- removed joint hand_1_hand_1_sensor_0_left_joint
- removed joint hand_1_hand_1_sensor_0_right_joint
- removed joint joint_1_joint_1_sensor_0_top_joint
- removed joint joint_2_joint_2_sensor_0_start_joint
- added joint hand_1_hand_1_sensor_0_top_joint: type fixed, parent hand_1, child hand_1_sensor_0_top, origin xyz=0 0 0.5 rpy=0 0 0, axis 0 1 0
- added joint hand_2_hand_2_sensor_0_top_joint: type fixed, parent hand_2, child hand_2_sensor_0_top, origin xyz=0 0 0.5 rpy=0 0 0, axis 0 1 0
- added joint hand_3_hand_3_sensor_0_top_joint: type fixed, parent hand_3, child hand_3_sensor_0_top, origin xyz=0 0 0.5 rpy=0 0 0, axis 0 1 0

File: pybullet_data/robots/robot_two_head_arm_c.urdf (robot description, URDF)
Before this commit: robot robot, 124 links, 123 joints
Links:
- removed link hand_part_0_sensor_0_left
- removed link hand_part_0_sensor_0_right
- removed link hand_part_1_sensor_0_start
- removed link hand_part_1_sensor_0_stop
- removed link hand_part_2_sensor_0_start
- removed link hand_part_2_sensor_0_stop
- removed link hand_part_3_sensor_0_start
- removed link hand_part_3_sensor_0_stop
- removed link hand_part_4_sensor_0_start
- removed link hand_part_4_sensor_0_stop
- removed link hand_part_5_sensor_0_start
- removed link hand_part_5_sensor_0_stop
- removed link hand_part_6_sensor_0_start
- removed link hand_part_6_sensor_0_stop
- removed link hand_part_7_sensor_0_start
- removed link hand_part_7_sensor_0_stop
- removed link hand_part_8_sensor_0_start
- removed link hand_part_8_sensor_0_stop
- removed link hand_part_9_sensor_0_start
- removed link hand_part_9_sensor_0_stop
- removed link joint_1_sensor_0_top
- removed link joint_2_sensor_0_start
- removed link wrist_sensor_0_bottom
- removed link wrist_sensor_0_top
- link hand_part_0: geometry collision box size=0.2 0.6180339887498948 0.25; visual box size=0.2 0.6180339887498948 0.25
- link hand_part_0_sensor_0_bottom: geometry collision box size=0.2 0.6180339887498948 0.02; visual box size=0.2 0.6180339887498948 0.02
- link hand_part_0_sensor_0_start: geometry collision box size=0.02 0.6180339887498948 0.25; visual box size=0.02 0.6180339887498948 0.25
- link hand_part_0_sensor_0_stop: geometry collision box size=0.02 0.6180339887498948 0.25; visual box size=0.02 0.6180339887498948 0.25
- link hand_part_0_sensor_0_top: geometry collision box size=0.2 0.6180339887498948 0.02; visual box size=0.2 0.6180339887498948 0.02
- link hand_part_1: geometry collision box size=0.6180339887498948 0.2 0.25; visual box size=0.6180339887498948 0.2 0.25
- link hand_part_1_sensor_0_bottom: geometry collision box size=0.6180339887498948 0.2 0.02; visual box size=0.6180339887498948 0.2 0.02
- link hand_part_1_sensor_0_left: geometry collision box size=0.6180339887498948 0.02 0.25; visual box size=0.6180339887498948 0.02 0.25
- link hand_part_1_sensor_0_right: geometry collision box size=0.6180339887498948 0.02 0.25; visual box size=0.6180339887498948 0.02 0.25
- link hand_part_1_sensor_0_top: geometry collision box size=0.6180339887498948 0.2 0.02; visual box size=0.6180339887498948 0.2 0.02
- link hand_part_2: geometry collision box size=0.6180339887498948 0.2 0.25; visual box size=0.6180339887498948 0.2 0.25
- link hand_part_2_sensor_0_bottom: geometry collision box size=0.6180339887498948 0.2 0.02; visual box size=0.6180339887498948 0.2 0.02
- link hand_part_2_sensor_0_left: geometry collision box size=0.6180339887498948 0.02 0.25; visual box size=0.6180339887498948 0.02 0.25
- link hand_part_2_sensor_0_right: geometry collision box size=0.6180339887498948 0.02 0.25; visual box size=0.6180339887498948 0.02 0.25
- link hand_part_2_sensor_0_top: geometry collision box size=0.6180339887498948 0.2 0.02; visual box size=0.6180339887498948 0.2 0.02
- link hand_part_3: geometry collision box size=0.6180339887498948 0.2 0.25; visual box size=0.6180339887498948 0.2 0.25
- link hand_part_3_sensor_0_bottom: geometry collision box size=0.6180339887498948 0.2 0.02; visual box size=0.6180339887498948 0.2 0.02
- link hand_part_3_sensor_0_left: geometry collision box size=0.6180339887498948 0.02 0.25; visual box size=0.6180339887498948 0.02 0.25
- link hand_part_3_sensor_0_right: geometry collision box size=0.6180339887498948 0.02 0.25; visual box size=0.6180339887498948 0.02 0.25
- link hand_part_3_sensor_0_top: geometry collision box size=0.6180339887498948 0.2 0.02; visual box size=0.6180339887498948 0.2 0.02
- link hand_part_4: geometry collision box size=0.6180339887498948 0.2 0.25; visual box size=0.6180339887498948 0.2 0.25
- link hand_part_4_sensor_0_bottom: geometry collision box size=0.6180339887498948 0.2 0.02; visual box size=0.6180339887498948 0.2 0.02
- link hand_part_4_sensor_0_left: geometry collision box size=0.6180339887498948 0.02 0.25; visual box size=0.6180339887498948 0.02 0.25
- link hand_part_4_sensor_0_right: geometry collision box size=0.6180339887498948 0.02 0.25; visual box size=0.6180339887498948 0.02 0.25
- link hand_part_4_sensor_0_top: geometry collision box size=0.6180339887498948 0.2 0.02; visual box size=0.6180339887498948 0.2 0.02
- link hand_part_5: geometry collision box size=0.6180339887498948 0.2 0.25; visual box size=0.6180339887498948 0.2 0.25
- link hand_part_5_sensor_0_bottom: geometry collision box size=0.6180339887498948 0.2 0.02; visual box size=0.6180339887498948 0.2 0.02
- link hand_part_5_sensor_0_left: geometry collision box size=0.6180339887498948 0.02 0.25; visual box size=0.6180339887498948 0.02 0.25
- link hand_part_5_sensor_0_right: geometry collision box size=0.6180339887498948 0.02 0.25; visual box size=0.6180339887498948 0.02 0.25
- link hand_part_5_sensor_0_top: geometry collision box size=0.6180339887498948 0.2 0.02; visual box size=0.6180339887498948 0.2 0.02
- link hand_part_6: geometry collision box size=0.6180339887498948 0.2 0.25; visual box size=0.6180339887498948 0.2 0.25
- link hand_part_6_sensor_0_bottom: geometry collision box size=0.6180339887498948 0.2 0.02; visual box size=0.6180339887498948 0.2 0.02
- link hand_part_6_sensor_0_left: geometry collision box size=0.6180339887498948 0.02 0.25; visual box size=0.6180339887498948 0.02 0.25
- link hand_part_6_sensor_0_right: geometry collision box size=0.6180339887498948 0.02 0.25; visual box size=0.6180339887498948 0.02 0.25
- link hand_part_6_sensor_0_top: geometry collision box size=0.6180339887498948 0.2 0.02; visual box size=0.6180339887498948 0.2 0.02
- link hand_part_7: geometry collision box size=0.6180339887498948 0.2 0.25; visual box size=0.6180339887498948 0.2 0.25
- link hand_part_7_sensor_0_bottom: geometry collision box size=0.6180339887498948 0.2 0.02; visual box size=0.6180339887498948 0.2 0.02
- link hand_part_7_sensor_0_left: geometry collision box size=0.6180339887498948 0.02 0.25; visual box size=0.6180339887498948 0.02 0.25
- link hand_part_7_sensor_0_right: geometry collision box size=0.6180339887498948 0.02 0.25; visual box size=0.6180339887498948 0.02 0.25
- link hand_part_7_sensor_0_top: geometry collision box size=0.6180339887498948 0.2 0.02; visual box size=0.6180339887498948 0.2 0.02
- link hand_part_8: geometry collision box size=0.6180339887498948 0.2 0.25; visual box size=0.6180339887498948 0.2 0.25
- link hand_part_8_sensor_0_bottom: geometry collision box size=0.6180339887498948 0.2 0.02; visual box size=0.6180339887498948 0.2 0.02
- link hand_part_8_sensor_0_left: geometry collision box size=0.6180339887498948 0.02 0.25; visual box size=0.6180339887498948 0.02 0.25
- link hand_part_8_sensor_0_right: geometry collision box size=0.6180339887498948 0.02 0.25; visual box size=0.6180339887498948 0.02 0.25
- link hand_part_8_sensor_0_top: geometry collision box size=0.6180339887498948 0.2 0.02; visual box size=0.6180339887498948 0.2 0.02
- link hand_part_9: geometry collision box size=0.6180339887498948 0.2 0.25; visual box size=0.6180339887498948 0.2 0.25
- link hand_part_9_sensor_0_bottom: geometry collision box size=0.6180339887498948 0.2 0.02; visual box size=0.6180339887498948 0.2 0.02
- link hand_part_9_sensor_0_left: geometry collision box size=0.6180339887498948 0.02 0.25; visual box size=0.6180339887498948 0.02 0.25
- link hand_part_9_sensor_0_right: geometry collision box size=0.6180339887498948 0.02 0.25; visual box size=0.6180339887498948 0.02 0.25
- link hand_part_9_sensor_0_top: geometry collision box size=0.6180339887498948 0.2 0.02; visual box size=0.6180339887498948 0.2 0.02
Joints:
- removed joint hand_part_0_hand_part_0_sensor_0_left_joint
- removed joint hand_part_0_hand_part_0_sensor_0_right_joint
- removed joint hand_part_1_hand_part_1_sensor_0_start_joint
- removed joint hand_part_1_hand_part_1_sensor_0_stop_joint
- removed joint hand_part_2_hand_part_2_sensor_0_start_joint
- removed joint hand_part_2_hand_part_2_sensor_0_stop_joint
- removed joint hand_part_3_hand_part_3_sensor_0_start_joint
- removed joint hand_part_3_hand_part_3_sensor_0_stop_joint
- removed joint hand_part_4_hand_part_4_sensor_0_start_joint
- removed joint hand_part_4_hand_part_4_sensor_0_stop_joint
- removed joint hand_part_5_hand_part_5_sensor_0_start_joint
- removed joint hand_part_5_hand_part_5_sensor_0_stop_joint
- removed joint hand_part_6_hand_part_6_sensor_0_start_joint
- removed joint hand_part_6_hand_part_6_sensor_0_stop_joint
- removed joint hand_part_7_hand_part_7_sensor_0_start_joint
- removed joint hand_part_7_hand_part_7_sensor_0_stop_joint
- removed joint hand_part_8_hand_part_8_sensor_0_start_joint
- removed joint hand_part_8_hand_part_8_sensor_0_stop_joint
- removed joint hand_part_9_hand_part_9_sensor_0_start_joint
- removed joint hand_part_9_hand_part_9_sensor_0_stop_joint
- removed joint joint_1_joint_1_sensor_0_top_joint
- removed joint joint_2_joint_2_sensor_0_start_joint
- removed joint wrist_wrist_sensor_0_bottom_joint
- removed joint wrist_wrist_sensor_0_top_joint
- joint hand_part_0_hand_part_1_joint: origin xyz=-0.14530850560107214 0.4472135954999579 0 rpy=0 0 -0.9424777960769379 -> xyz=-0.1816356320013402 0.5590169943749475 0 rpy=0 0 -0.9424777960769379
- joint hand_part_0_hand_part_2_joint: origin xyz=-0.5257311121191336 0.7236067977499789 0 rpy=0 0 -0.3141592653589793 -> xyz=-0.6571638901489171 0.9045084971874737 0 rpy=0 0 -0.3141592653589793
- joint hand_part_0_hand_part_3_joint: origin xyz=-0.9959593139531121 0.723606797749979 0 rpy=0 0 0.3141592653589793 -> xyz=-1.2449491424413903 0.9045084971874738 0 rpy=0 0 0.3141592653589793
- joint hand_part_0_hand_part_4_joint: origin xyz=-1.3763819204711736 0.44721359549995804 0 rpy=0 0 0.9424777960769379 -> xyz=-1.7204774005889671 0.5590169943749476 0 rpy=0 0 0.9424777960769379
- joint hand_part_0_hand_part_5_joint: origin xyz=-1.5216904260722457 9.317666547912739e-17 0 rpy=0 0 1.5707963267948966 -> xyz=-1.9021130325903073 1.1647083184890926e-16 0 rpy=0 0 1.5707963267948966
- joint hand_part_0_hand_part_6_joint: origin xyz=-1.3763819204711736 -0.44721359549995787 0 rpy=0 0 2.199114857512855 -> xyz=-1.7204774005889671 -0.5590169943749473 0 rpy=0 0 2.199114857512855
- joint hand_part_0_hand_part_7_joint: origin xyz=-0.9959593139531121 -0.7236067977499789 0 rpy=0 0 2.827433388230814 -> xyz=-1.2449491424413903 -0.9045084971874737 0 rpy=0 0 2.827433388230814
- joint hand_part_0_hand_part_8_joint: origin xyz=-0.5257311121191337 -0.723606797749979 0 rpy=0 0 3.4557519189487724 -> xyz=-0.6571638901489173 -0.9045084971874738 0 rpy=0 0 3.4557519189487724
- joint hand_part_0_hand_part_9_joint: origin xyz=-0.14530850560107225 -0.4472135954999581 0 rpy=0 0 4.084070449666731 -> xyz=-0.1816356320013403 -0.5590169943749477 0 rpy=0 0 4.084070449666731

File: pybullet_data/robots/robot_two_head_arm_d.urdf (robot description, URDF)
Before this commit: robot robot, 82 links, 81 joints
Links:
- removed link hand_1_sensor_0_top
- removed link hand_2_sensor_0_top
- removed link hand_3_sensor_0_top
- removed link hand_4
- removed link hand_4_sensor_0_bottom
- removed link hand_4_sensor_0_left
- removed link hand_4_sensor_0_right
- removed link hand_4_sensor_0_start
- removed link hand_4_sensor_0_stop
- removed link hand_4_sensor_0_top
- removed link joint_1_sensor_0_top
- removed link joint_2_sensor_0_start
- link palm: geometry collision box size=0.2 1.5 0.2; visual box size=0.2 1.5 0.2
- link palm_sensor_0_bottom: geometry collision box size=0.2 1.5 0.02; visual box size=0.2 1.5 0.02
- link palm_sensor_0_start: geometry collision box size=0.02 1.5 0.2; visual box size=0.02 1.5 0.2
- link palm_sensor_0_stop: geometry collision box size=0.02 1.5 0.2; visual box size=0.02 1.5 0.2
- link palm_sensor_0_top: geometry collision box size=0.2 1.5 0.02; visual box size=0.2 1.5 0.02
Joints:
- removed joint hand_1_hand_1_sensor_0_top_joint
- removed joint hand_2_hand_2_sensor_0_top_joint
- removed joint hand_3_hand_3_sensor_0_top_joint
- removed joint hand_4_hand_4_sensor_0_bottom_joint
- removed joint hand_4_hand_4_sensor_0_left_joint
- removed joint hand_4_hand_4_sensor_0_right_joint
- removed joint hand_4_hand_4_sensor_0_start_joint
- removed joint hand_4_hand_4_sensor_0_stop_joint
- removed joint hand_4_hand_4_sensor_0_top_joint
- removed joint joint_1_joint_1_sensor_0_top_joint
- removed joint joint_2_joint_2_sensor_0_start_joint
- removed joint palm_hand_4_joint
- joint arm_palm_joint: origin xyz=0.575 0 0 rpy=0 0 0 -> xyz=0.125 0 0 rpy=0 0 0
- joint palm_hand_1_joint: origin xyz=0.7000000000000001 0 -0.7 rpy=0 0 0 -> xyz=1.15 0 -0.7 rpy=0 0 0
- joint palm_hand_2_joint: origin xyz=-0.7000000000000001 0 -0.7 rpy=0 0 0 -> xyz=0 0.65 -0.7 rpy=0 0 0
- joint palm_hand_3_joint: origin xyz=0 0.7000000000000001 -0.7 rpy=0 0 0 -> xyz=0 -0.65 -0.7 rpy=0 0 0
- joint palm_palm_sensor_0_left_joint: origin xyz=0 0.8 0 rpy=0 0 0 -> xyz=0 0.75 0 rpy=0 0 0
- joint palm_palm_sensor_0_right_joint: origin xyz=0 -0.8 0 rpy=0 0 0 -> xyz=0 -0.75 0 rpy=0 0 0
