Commit message: 2025_03_06, big test. Complete cnn for image-out doesn't seem to help.

File: pybullet_data/robots/robot_two_head_arm_e.urdf (robot description, URDF)
Before this commit: robot robot, 94 links, 93 joints
Links:
- removed link hand_1_a
- removed link hand_1_a_sensor_0_bottom
- removed link hand_1_a_sensor_0_left
- removed link hand_1_a_sensor_0_right
- removed link hand_1_a_sensor_0_start
- removed link hand_1_a_sensor_0_stop
- removed link hand_1_a_sensor_0_top
- removed link hand_2_a
- removed link hand_2_a_sensor_0_bottom
- removed link hand_2_a_sensor_0_left
- removed link hand_2_a_sensor_0_right
- removed link hand_2_a_sensor_0_start
- removed link hand_2_a_sensor_0_stop
- removed link hand_2_a_sensor_0_top
- removed link hand_3_a
- removed link hand_3_a_sensor_0_bottom
- removed link hand_3_a_sensor_0_left
- removed link hand_3_a_sensor_0_right
- removed link hand_3_a_sensor_0_start
- removed link hand_3_a_sensor_0_stop
- removed link hand_3_a_sensor_0_top
- removed link hand_3_b
- removed link hand_3_b_sensor_0_bottom
- removed link hand_3_b_sensor_0_left
- removed link hand_3_b_sensor_0_right
- removed link hand_3_b_sensor_0_start
- removed link hand_3_b_sensor_0_stop
- removed link hand_3_b_sensor_0_top
- removed link hand_3_c
- removed link hand_3_c_sensor_0_bottom
- removed link hand_3_c_sensor_0_left
- removed link hand_3_c_sensor_0_right
- removed link hand_3_c_sensor_0_start
- removed link hand_3_c_sensor_0_stop
- removed link hand_3_c_sensor_0_top
- added link finger_1_3, mass 2; collision box size=0.2 0.2 1.5; visual box size=0.2 0.2 1.5
- added link finger_1_3_sensor_0_bottom, mass 0; collision box size=0.2 0.2 0.02; visual box size=0.2 0.2 0.02
- added link finger_1_3_sensor_0_left, mass 0; collision box size=0.2 0.02 1.5; visual box size=0.2 0.02 1.5
- added link finger_1_3_sensor_0_right, mass 0; collision box size=0.2 0.02 1.5; visual box size=0.2 0.02 1.5
- added link finger_1_3_sensor_0_start, mass 0; collision box size=0.02 0.2 1.5; visual box size=0.02 0.2 1.5
- added link finger_1_3_sensor_0_stop, mass 0; collision box size=0.02 0.2 1.5; visual box size=0.02 0.2 1.5
- added link finger_1_3_sensor_0_top, mass 0; collision box size=0.2 0.2 0.02; visual box size=0.2 0.2 0.02
- added link finger_2_3, mass 2; collision box size=0.2 0.2 0.5; visual box size=0.2 0.2 0.5
- added link finger_2_3_sensor_0_bottom, mass 0; collision box size=0.2 0.2 0.02; visual box size=0.2 0.2 0.02
- added link finger_2_3_sensor_0_left, mass 0; collision box size=0.2 0.02 0.5; visual box size=0.2 0.02 0.5
- added link finger_2_3_sensor_0_right, mass 0; collision box size=0.2 0.02 0.5; visual box size=0.2 0.02 0.5
- added link finger_2_3_sensor_0_start, mass 0; collision box size=0.02 0.2 0.5; visual box size=0.02 0.2 0.5
- added link finger_2_3_sensor_0_stop, mass 0; collision box size=0.02 0.2 0.5; visual box size=0.02 0.2 0.5
- added link finger_2_3_sensor_0_top, mass 0; collision box size=0.2 0.2 0.02; visual box size=0.2 0.2 0.02
Joints:
- removed joint arm_hand_3_a_joint
- removed joint hand_1_a_hand_1_a_sensor_0_bottom_joint
- removed joint hand_1_a_hand_1_a_sensor_0_left_joint
- removed joint hand_1_a_hand_1_a_sensor_0_right_joint
- removed joint hand_1_a_hand_1_a_sensor_0_start_joint
- removed joint hand_1_a_hand_1_a_sensor_0_stop_joint
- removed joint hand_1_a_hand_1_a_sensor_0_top_joint
- removed joint hand_2_a_hand_2_a_sensor_0_bottom_joint
- removed joint hand_2_a_hand_2_a_sensor_0_left_joint
- removed joint hand_2_a_hand_2_a_sensor_0_right_joint
- removed joint hand_2_a_hand_2_a_sensor_0_start_joint
- removed joint hand_2_a_hand_2_a_sensor_0_stop_joint
- removed joint hand_2_a_hand_2_a_sensor_0_top_joint
- removed joint hand_3_a_hand_3_a_sensor_0_bottom_joint
- removed joint hand_3_a_hand_3_a_sensor_0_left_joint
- removed joint hand_3_a_hand_3_a_sensor_0_right_joint
- removed joint hand_3_a_hand_3_a_sensor_0_start_joint
- removed joint hand_3_a_hand_3_a_sensor_0_stop_joint
- removed joint hand_3_a_hand_3_a_sensor_0_top_joint
- removed joint hand_3_a_hand_3_b_joint
- removed joint hand_3_b_hand_3_b_sensor_0_bottom_joint
- removed joint hand_3_b_hand_3_b_sensor_0_left_joint
- removed joint hand_3_b_hand_3_b_sensor_0_right_joint
- removed joint hand_3_b_hand_3_b_sensor_0_start_joint
- removed joint hand_3_b_hand_3_b_sensor_0_stop_joint
- removed joint hand_3_b_hand_3_b_sensor_0_top_joint
- removed joint hand_3_b_hand_3_c_joint
- removed joint hand_3_c_hand_3_c_sensor_0_bottom_joint
- removed joint hand_3_c_hand_3_c_sensor_0_left_joint
- removed joint hand_3_c_hand_3_c_sensor_0_right_joint
- removed joint hand_3_c_hand_3_c_sensor_0_start_joint
- removed joint hand_3_c_hand_3_c_sensor_0_stop_joint
- removed joint hand_3_c_hand_3_c_sensor_0_top_joint
- removed joint palm_1_hand_1_a_joint
- removed joint palm_2_hand_2_a_joint
- added joint arm_finger_1_3_joint: type fixed, parent arm, child finger_1_3, origin xyz=2.079769465589431 0 -0.2565151074942517 rpy=0 -1.2217304763960306 0, axis 0 1 0
- added joint finger_1_3_finger_1_3_sensor_0_bottom_joint: type fixed, parent finger_1_3, child finger_1_3_sensor_0_bottom, origin xyz=0 0 -0.75 rpy=0 0 0, axis 0 1 0
- added joint finger_1_3_finger_1_3_sensor_0_left_joint: type fixed, parent finger_1_3, child finger_1_3_sensor_0_left, origin xyz=0 0.1 0 rpy=0 0 0, axis 0 1 0
- added joint finger_1_3_finger_1_3_sensor_0_right_joint: type fixed, parent finger_1_3, child finger_1_3_sensor_0_right, origin xyz=0 -0.1 0 rpy=0 0 0, axis 0 1 0
- added joint finger_1_3_finger_1_3_sensor_0_start_joint: type fixed, parent finger_1_3, child finger_1_3_sensor_0_start, origin xyz=0.1 0 0 rpy=0 0 0, axis 0 1 0
- added joint finger_1_3_finger_1_3_sensor_0_stop_joint: type fixed, parent finger_1_3, child finger_1_3_sensor_0_stop, origin xyz=-0.1 0 0 rpy=0 0 0, axis 0 1 0
- added joint finger_1_3_finger_1_3_sensor_0_top_joint: type fixed, parent finger_1_3, child finger_1_3_sensor_0_top, origin xyz=0 0 0.75 rpy=0 0 0, axis 0 1 0
- added joint finger_1_3_finger_2_3_joint: type fixed, parent finger_1_3, child finger_2_3, origin xyz=0.810424031024606 0 -0.48309205425341406 rpy=0 -0.4363323129985824 0, axis 0 1 0
- added joint finger_2_3_finger_2_3_sensor_0_bottom_joint: type fixed, parent finger_2_3, child finger_2_3_sensor_0_bottom, origin xyz=0 0 -0.25 rpy=0 0 0, axis 0 1 0
- added joint finger_2_3_finger_2_3_sensor_0_left_joint: type fixed, parent finger_2_3, child finger_2_3_sensor_0_left, origin xyz=0 0.1 0 rpy=0 0 0, axis 0 1 0
- added joint finger_2_3_finger_2_3_sensor_0_right_joint: type fixed, parent finger_2_3, child finger_2_3_sensor_0_right, origin xyz=0 -0.1 0 rpy=0 0 0, axis 0 1 0
- added joint finger_2_3_finger_2_3_sensor_0_start_joint: type fixed, parent finger_2_3, child finger_2_3_sensor_0_start, origin xyz=0.1 0 0 rpy=0 0 0, axis 0 1 0
- added joint finger_2_3_finger_2_3_sensor_0_stop_joint: type fixed, parent finger_2_3, child finger_2_3_sensor_0_stop, origin xyz=-0.1 0 0 rpy=0 0 0, axis 0 1 0
- added joint finger_2_3_finger_2_3_sensor_0_top_joint: type fixed, parent finger_2_3, child finger_2_3_sensor_0_top, origin xyz=0 0 0.25 rpy=0 0 0, axis 0 1 0
