Commit message: 2025_03_07, big test. accelerated joints works. But: notice ec and ef are the same!

File: pybullet_data/robots/robot_four_side_arm.urdf (robot description, URDF)
Before this commit: robot robot, 78 links, 77 joints
Joints:
- joint body_joint_1_joint: limit lower=0 upper=0 effort=0 velocity=0 -> lower=0 upper=1.5707963267948966 effort=999 velocity=999
- joint body_joint_3_joint: limit lower=0 upper=0 effort=0 velocity=0 -> lower=0 upper=1.5707963267948966 effort=999 velocity=999
- joint joint_1_joint_2_joint: limit lower=0 upper=0 effort=0 velocity=0 -> lower=-0.7853981633974483 upper=0.7853981633974483 effort=999 velocity=999
- joint joint_3_joint_4_joint: limit lower=0 upper=0 effort=0 velocity=0 -> lower=-0.7853981633974483 upper=0.7853981633974483 effort=999 velocity=999

File: pybullet_data/robots/robot_two_head_arm_f.urdf (robot description, URDF)
Before this commit: robot robot, 109 links, 108 joints
Joints:
- joint body_joint_1_joint: limit lower=0 upper=0 effort=0 velocity=0 -> lower=-0.7853981633974483 upper=0.7853981633974483 effort=999 velocity=999
- joint joint_1_joint_2_joint: limit lower=0 upper=0 effort=0 velocity=0 -> lower=-1.5707963267948966 upper=0 effort=999 velocity=999

File: pybullet_data/robots/robot_two_head_arm_g.urdf (robot description, URDF)
Before this commit: robot robot, 109 links, 108 joints
Joints:
- joint body_joint_1_joint: limit lower=0 upper=0 effort=0 velocity=0 -> lower=-0.7853981633974483 upper=0.7853981633974483 effort=999 velocity=999
- joint joint_1_joint_2_joint: limit lower=0 upper=0 effort=0 velocity=0 -> lower=-1.5707963267948966 upper=0 effort=999 velocity=999

File: pybullet_data/robots/robot_two_side_arm.urdf (robot description, URDF)
Before this commit: robot robot, 76 links, 75 joints
Joints:
- joint body_joint_1_joint: limit lower=0 upper=0 effort=0 velocity=0 -> lower=0 upper=1.5707963267948966 effort=999 velocity=999
- joint body_joint_2_joint: limit lower=0 upper=0 effort=0 velocity=0 -> lower=0 upper=1.5707963267948966 effort=999 velocity=999
