Commit message: 2025_03_13. Big test, longer episodes. OMG WOW!

File: pybullet_data/robots/robot_two_head_arm_g.urdf (robot description, URDF)
Before this commit: robot robot, 109 links, 108 joints
Links:
- added link hand_part_11_sensor_0_start, mass 0; collision box size=0.02 0.2 1; visual box size=0.02 0.2 1
- added link hand_part_5_sensor_0_stop, mass 0; collision box size=0.02 0.2 1; visual box size=0.02 0.2 1
Joints:
- added joint hand_part_11_hand_part_11_sensor_0_start_joint: type fixed, parent hand_part_11, child hand_part_11_sensor_0_start, origin xyz=0.19509032201612825 0 0 rpy=0 0 0, axis 0 1 0
- added joint hand_part_5_hand_part_5_sensor_0_stop_joint: type fixed, parent hand_part_5, child hand_part_5_sensor_0_stop, origin xyz=-0.19509032201612825 0 0 rpy=0 0 0, axis 0 1 0
