Commit message: 2025_03_21. Big test: Working awesomely!

File: pybullet_data/robots/robot_two_head_arm_a.urdf (robot description, URDF)
Before this commit: robot robot, 54 links, 53 joints
Links:
- added link hand_sensor_0_bottom, mass 0; collision box size=1.0 0.2 0.02; visual box size=1.0 0.2 0.02
- added link hand_sensor_0_top, mass 0; collision box size=1.0 0.2 0.02; visual box size=1.0 0.2 0.02
- link arm: geometry collision box size=1.75 0.2 0.2; visual box size=1.75 0.2 0.2
- link arm_sensor_0_bottom: geometry collision box size=1.75 0.2 0.02; visual box size=1.75 0.2 0.02
- link arm_sensor_0_left: geometry collision box size=1.75 0.02 0.2; visual box size=1.75 0.02 0.2
- link arm_sensor_0_right: geometry collision box size=1.75 0.02 0.2; visual box size=1.75 0.02 0.2
- link arm_sensor_0_top: geometry collision box size=1.75 0.2 0.02; visual box size=1.75 0.2 0.02
- link hand: geometry collision box size=1 0.2 1.25; visual box size=1 0.2 1.25
- link hand_sensor_0_left: geometry collision box size=1.0 0.02 1.25; visual box size=1.0 0.02 1.25
- link hand_sensor_0_right: geometry collision box size=1.0 0.02 1.25; visual box size=1.0 0.02 1.25
- link hand_sensor_0_start: geometry collision box size=0.02 0.2 1.25; visual box size=0.02 0.2 1.25
- link hand_sensor_0_stop: geometry collision box size=0.02 0.2 1.25; visual box size=0.02 0.2 1.25
Joints:
- added joint hand_hand_sensor_0_bottom_joint: type fixed, parent hand, child hand_sensor_0_bottom, origin xyz=0 0 -0.625 rpy=0 0 0, axis 0 1 0
- added joint hand_hand_sensor_0_top_joint: type fixed, parent hand, child hand_sensor_0_top, origin xyz=0 0 0.625 rpy=0 0 0, axis 0 1 0
- joint arm_arm_sensor_0_start_joint: origin xyz=1.375 0 0 rpy=0 0 0 -> xyz=0.875 0 0 rpy=0 0 0
- joint arm_hand_joint: origin xyz=0.875 0 -0.6 rpy=0 0 0 -> xyz=1.375 0 -0.525 rpy=0 0 0
- joint joint_2_arm_joint: origin xyz=1.475 0 0 rpy=0 0 0 -> xyz=0.975 0 0 rpy=0 0 0

File: pybullet_data/robots/robot_two_head_arm_b.urdf (robot description, URDF)
Before this commit: robot robot, 111 links, 110 joints
Links:
- removed link hand_part_0
- removed link hand_part_0_sensor_0_bottom
- removed link hand_part_0_sensor_0_start
- removed link hand_part_0_sensor_0_stop
- removed link hand_part_0_sensor_0_top
- removed link hand_part_1
- removed link hand_part_11
- removed link hand_part_11_sensor_0_bottom
- removed link hand_part_11_sensor_0_left
- removed link hand_part_11_sensor_0_right
- removed link hand_part_11_sensor_0_start
- removed link hand_part_11_sensor_0_top
- removed link hand_part_12
- removed link hand_part_12_sensor_0_bottom
- removed link hand_part_12_sensor_0_left
- removed link hand_part_12_sensor_0_right
- removed link hand_part_12_sensor_0_top
- removed link hand_part_13
- removed link hand_part_13_sensor_0_bottom
- removed link hand_part_13_sensor_0_left
- removed link hand_part_13_sensor_0_right
- removed link hand_part_13_sensor_0_top
- removed link hand_part_14
- removed link hand_part_14_sensor_0_bottom
- removed link hand_part_14_sensor_0_left
- removed link hand_part_14_sensor_0_right
- removed link hand_part_14_sensor_0_top
- removed link hand_part_15
- removed link hand_part_15_sensor_0_bottom
- removed link hand_part_15_sensor_0_left
- removed link hand_part_15_sensor_0_right
- removed link hand_part_15_sensor_0_top
- removed link hand_part_1_sensor_0_bottom
- removed link hand_part_1_sensor_0_left
- removed link hand_part_1_sensor_0_right
- removed link hand_part_1_sensor_0_top
- removed link hand_part_2
- removed link hand_part_2_sensor_0_bottom
- removed link hand_part_2_sensor_0_left
- removed link hand_part_2_sensor_0_right
- removed link hand_part_2_sensor_0_top
- removed link hand_part_3
- removed link hand_part_3_sensor_0_bottom
- removed link hand_part_3_sensor_0_left
- removed link hand_part_3_sensor_0_right
- removed link hand_part_3_sensor_0_top
- removed link hand_part_4
- removed link hand_part_4_sensor_0_bottom
- removed link hand_part_4_sensor_0_left
- removed link hand_part_4_sensor_0_right
- removed link hand_part_4_sensor_0_top
- removed link hand_part_5
- removed link hand_part_5_sensor_0_bottom
- removed link hand_part_5_sensor_0_left
- removed link hand_part_5_sensor_0_right
- removed link hand_part_5_sensor_0_stop
- removed link hand_part_5_sensor_0_top
- removed link wrist
- removed link wrist_sensor_0_left
- removed link wrist_sensor_0_right
- removed link wrist_sensor_0_start
- removed link wrist_sensor_0_stop
- added link hand, mass 2; collision box size=1 1 1.25; visual box size=1 1 1.25
- added link hand_sensor_0_bottom, mass 0; collision box size=1.0 1 0.02; visual box size=1.0 1 0.02
- added link hand_sensor_0_left, mass 0; collision box size=1.0 0.02 1.25; visual box size=1.0 0.02 1.25
- added link hand_sensor_0_right, mass 0; collision box size=1.0 0.02 1.25; visual box size=1.0 0.02 1.25
- added link hand_sensor_0_start, mass 0; collision box size=0.02 1 1.25; visual box size=0.02 1 1.25
- added link hand_sensor_0_stop, mass 0; collision box size=0.02 1 1.25; visual box size=0.02 1 1.25
- added link hand_sensor_0_top, mass 0; collision box size=1.0 1 0.02; visual box size=1.0 1 0.02
- link arm: geometry collision box size=1.75 0.2 0.2; visual box size=1.75 0.2 0.2
- link arm_sensor_0_bottom: geometry collision box size=1.75 0.2 0.02; visual box size=1.75 0.2 0.02
- link arm_sensor_0_left: geometry collision box size=1.75 0.02 0.2; visual box size=1.75 0.02 0.2
- link arm_sensor_0_right: geometry collision box size=1.75 0.02 0.2; visual box size=1.75 0.02 0.2
- link arm_sensor_0_top: geometry collision box size=1.75 0.2 0.02; visual box size=1.75 0.2 0.02
Joints:
- removed joint arm_wrist_joint
- removed joint hand_part_0_hand_part_0_sensor_0_bottom_joint
- removed joint hand_part_0_hand_part_0_sensor_0_start_joint
- removed joint hand_part_0_hand_part_0_sensor_0_stop_joint
- removed joint hand_part_0_hand_part_0_sensor_0_top_joint
- removed joint hand_part_0_hand_part_11_joint
- removed joint hand_part_0_hand_part_12_joint
- removed joint hand_part_0_hand_part_13_joint
- removed joint hand_part_0_hand_part_14_joint
- removed joint hand_part_0_hand_part_15_joint
- removed joint hand_part_0_hand_part_1_joint
- removed joint hand_part_0_hand_part_2_joint
- removed joint hand_part_0_hand_part_3_joint
- removed joint hand_part_0_hand_part_4_joint
- removed joint hand_part_0_hand_part_5_joint
- removed joint hand_part_11_hand_part_11_sensor_0_bottom_joint
- removed joint hand_part_11_hand_part_11_sensor_0_left_joint
- removed joint hand_part_11_hand_part_11_sensor_0_right_joint
- removed joint hand_part_11_hand_part_11_sensor_0_start_joint
- removed joint hand_part_11_hand_part_11_sensor_0_top_joint
- removed joint hand_part_12_hand_part_12_sensor_0_bottom_joint
- removed joint hand_part_12_hand_part_12_sensor_0_left_joint
- removed joint hand_part_12_hand_part_12_sensor_0_right_joint
- removed joint hand_part_12_hand_part_12_sensor_0_top_joint
- removed joint hand_part_13_hand_part_13_sensor_0_bottom_joint
- removed joint hand_part_13_hand_part_13_sensor_0_left_joint
- removed joint hand_part_13_hand_part_13_sensor_0_right_joint
- removed joint hand_part_13_hand_part_13_sensor_0_top_joint
- removed joint hand_part_14_hand_part_14_sensor_0_bottom_joint
- removed joint hand_part_14_hand_part_14_sensor_0_left_joint
- removed joint hand_part_14_hand_part_14_sensor_0_right_joint
- removed joint hand_part_14_hand_part_14_sensor_0_top_joint
- removed joint hand_part_15_hand_part_15_sensor_0_bottom_joint
- removed joint hand_part_15_hand_part_15_sensor_0_left_joint
- removed joint hand_part_15_hand_part_15_sensor_0_right_joint
- removed joint hand_part_15_hand_part_15_sensor_0_top_joint
- removed joint hand_part_1_hand_part_1_sensor_0_bottom_joint
- removed joint hand_part_1_hand_part_1_sensor_0_left_joint
- removed joint hand_part_1_hand_part_1_sensor_0_right_joint
- removed joint hand_part_1_hand_part_1_sensor_0_top_joint
- removed joint hand_part_2_hand_part_2_sensor_0_bottom_joint
- removed joint hand_part_2_hand_part_2_sensor_0_left_joint
- removed joint hand_part_2_hand_part_2_sensor_0_right_joint
- removed joint hand_part_2_hand_part_2_sensor_0_top_joint
- removed joint hand_part_3_hand_part_3_sensor_0_bottom_joint
- removed joint hand_part_3_hand_part_3_sensor_0_left_joint
- removed joint hand_part_3_hand_part_3_sensor_0_right_joint
- removed joint hand_part_3_hand_part_3_sensor_0_top_joint
- removed joint hand_part_4_hand_part_4_sensor_0_bottom_joint
- removed joint hand_part_4_hand_part_4_sensor_0_left_joint
- removed joint hand_part_4_hand_part_4_sensor_0_right_joint
- removed joint hand_part_4_hand_part_4_sensor_0_top_joint
- removed joint hand_part_5_hand_part_5_sensor_0_bottom_joint
- removed joint hand_part_5_hand_part_5_sensor_0_left_joint
- removed joint hand_part_5_hand_part_5_sensor_0_right_joint
- removed joint hand_part_5_hand_part_5_sensor_0_stop_joint
- removed joint hand_part_5_hand_part_5_sensor_0_top_joint
- removed joint wrist_hand_part_0_joint
- removed joint wrist_wrist_sensor_0_left_joint
- removed joint wrist_wrist_sensor_0_right_joint
- removed joint wrist_wrist_sensor_0_start_joint
- removed joint wrist_wrist_sensor_0_stop_joint
- added joint arm_hand_joint: type fixed, parent arm, child hand, origin xyz=1.375 0 -0.525 rpy=0 0 0, axis 0 1 0
- added joint hand_hand_sensor_0_bottom_joint: type fixed, parent hand, child hand_sensor_0_bottom, origin xyz=0 0 -0.625 rpy=0 0 0, axis 0 1 0
- added joint hand_hand_sensor_0_left_joint: type fixed, parent hand, child hand_sensor_0_left, origin xyz=0 0.5 0 rpy=0 0 0, axis 0 1 0
- added joint hand_hand_sensor_0_right_joint: type fixed, parent hand, child hand_sensor_0_right, origin xyz=0 -0.5 0 rpy=0 0 0, axis 0 1 0
- added joint hand_hand_sensor_0_start_joint: type fixed, parent hand, child hand_sensor_0_start, origin xyz=0.5 0 0 rpy=0 0 0, axis 0 1 0
- added joint hand_hand_sensor_0_stop_joint: type fixed, parent hand, child hand_sensor_0_stop, origin xyz=-0.5 0 0 rpy=0 0 0, axis 0 1 0
- added joint hand_hand_sensor_0_top_joint: type fixed, parent hand, child hand_sensor_0_top, origin xyz=0 0 0.625 rpy=0 0 0, axis 0 1 0
- joint arm_arm_sensor_0_start_joint: origin xyz=1.375 0 0 rpy=0 0 0 -> xyz=0.875 0 0 rpy=0 0 0
- joint joint_2_arm_joint: origin xyz=1.475 0 0 rpy=0 0 0 -> xyz=0.975 0 0 rpy=0 0 0
