Commit message: 2025_03_21. Big test: Working awesomely!

File: pybullet_data/robots/robot_two_head_arm_c.urdf (robot description, URDF)
Before this commit: robot robot, 54 links, 53 joints
Links:
- removed link hand
- removed link hand_sensor_0_left
- removed link hand_sensor_0_right
- removed link hand_sensor_0_start
- removed link hand_sensor_0_stop
- added link hand_part_0, mass 2; collision box size=0.2 0.3901806440322565 1; visual box size=0.2 0.3901806440322565 1
- added link hand_part_0_sensor_0_bottom, mass 0; collision box size=0.2 0.3901806440322565 0.02; visual box size=0.2 0.3901806440322565 0.02
- added link hand_part_0_sensor_0_start, mass 0; collision box size=0.02 0.3901806440322565 1; visual box size=0.02 0.3901806440322565 1
- added link hand_part_0_sensor_0_stop, mass 0; collision box size=0.02 0.3901806440322565 1; visual box size=0.02 0.3901806440322565 1
- added link hand_part_0_sensor_0_top, mass 0; collision box size=0.2 0.3901806440322565 0.02; visual box size=0.2 0.3901806440322565 0.02
- added link hand_part_1, mass 2; collision box size=0.3901806440322565 0.2 1; visual box size=0.3901806440322565 0.2 1
- added link hand_part_11, mass 2; collision box size=0.3901806440322565 0.2 1; visual box size=0.3901806440322565 0.2 1
- added link hand_part_11_sensor_0_bottom, mass 0; collision box size=0.3901806440322565 0.2 0.02; visual box size=0.3901806440322565 0.2 0.02
- added link hand_part_11_sensor_0_left, mass 0; collision box size=0.3901806440322565 0.02 1; visual box size=0.3901806440322565 0.02 1
- added link hand_part_11_sensor_0_right, mass 0; collision box size=0.3901806440322565 0.02 1; visual box size=0.3901806440322565 0.02 1
- added link hand_part_11_sensor_0_start, mass 0; collision box size=0.02 0.2 1; visual box size=0.02 0.2 1
- added link hand_part_11_sensor_0_top, mass 0; collision box size=0.3901806440322565 0.2 0.02; visual box size=0.3901806440322565 0.2 0.02
- added link hand_part_12, mass 2; collision box size=0.3901806440322565 0.2 1; visual box size=0.3901806440322565 0.2 1
- added link hand_part_12_sensor_0_bottom, mass 0; collision box size=0.3901806440322565 0.2 0.02; visual box size=0.3901806440322565 0.2 0.02
- added link hand_part_12_sensor_0_left, mass 0; collision box size=0.3901806440322565 0.02 1; visual box size=0.3901806440322565 0.02 1
- added link hand_part_12_sensor_0_right, mass 0; collision box size=0.3901806440322565 0.02 1; visual box size=0.3901806440322565 0.02 1
- added link hand_part_12_sensor_0_top, mass 0; collision box size=0.3901806440322565 0.2 0.02; visual box size=0.3901806440322565 0.2 0.02
- added link hand_part_13, mass 2; collision box size=0.3901806440322565 0.2 1; visual box size=0.3901806440322565 0.2 1
- added link hand_part_13_sensor_0_bottom, mass 0; collision box size=0.3901806440322565 0.2 0.02; visual box size=0.3901806440322565 0.2 0.02
- added link hand_part_13_sensor_0_left, mass 0; collision box size=0.3901806440322565 0.02 1; visual box size=0.3901806440322565 0.02 1
- added link hand_part_13_sensor_0_right, mass 0; collision box size=0.3901806440322565 0.02 1; visual box size=0.3901806440322565 0.02 1
- added link hand_part_13_sensor_0_top, mass 0; collision box size=0.3901806440322565 0.2 0.02; visual box size=0.3901806440322565 0.2 0.02
- added link hand_part_14, mass 2; collision box size=0.3901806440322565 0.2 1; visual box size=0.3901806440322565 0.2 1
- added link hand_part_14_sensor_0_bottom, mass 0; collision box size=0.3901806440322565 0.2 0.02; visual box size=0.3901806440322565 0.2 0.02
- added link hand_part_14_sensor_0_left, mass 0; collision box size=0.3901806440322565 0.02 1; visual box size=0.3901806440322565 0.02 1
- added link hand_part_14_sensor_0_right, mass 0; collision box size=0.3901806440322565 0.02 1; visual box size=0.3901806440322565 0.02 1
- added link hand_part_14_sensor_0_top, mass 0; collision box size=0.3901806440322565 0.2 0.02; visual box size=0.3901806440322565 0.2 0.02
- added link hand_part_15, mass 2; collision box size=0.3901806440322565 0.2 1; visual box size=0.3901806440322565 0.2 1
- added link hand_part_15_sensor_0_bottom, mass 0; collision box size=0.3901806440322565 0.2 0.02; visual box size=0.3901806440322565 0.2 0.02
- added link hand_part_15_sensor_0_left, mass 0; collision box size=0.3901806440322565 0.02 1; visual box size=0.3901806440322565 0.02 1
- added link hand_part_15_sensor_0_right, mass 0; collision box size=0.3901806440322565 0.02 1; visual box size=0.3901806440322565 0.02 1
- added link hand_part_15_sensor_0_top, mass 0; collision box size=0.3901806440322565 0.2 0.02; visual box size=0.3901806440322565 0.2 0.02
- added link hand_part_1_sensor_0_bottom, mass 0; collision box size=0.3901806440322565 0.2 0.02; visual box size=0.3901806440322565 0.2 0.02
- added link hand_part_1_sensor_0_left, mass 0; collision box size=0.3901806440322565 0.02 1; visual box size=0.3901806440322565 0.02 1
- added link hand_part_1_sensor_0_right, mass 0; collision box size=0.3901806440322565 0.02 1; visual box size=0.3901806440322565 0.02 1
- added link hand_part_1_sensor_0_top, mass 0; collision box size=0.3901806440322565 0.2 0.02; visual box size=0.3901806440322565 0.2 0.02
- added link hand_part_2, mass 2; collision box size=0.3901806440322565 0.2 1; visual box size=0.3901806440322565 0.2 1
- added link hand_part_2_sensor_0_bottom, mass 0; collision box size=0.3901806440322565 0.2 0.02; visual box size=0.3901806440322565 0.2 0.02
- added link hand_part_2_sensor_0_left, mass 0; collision box size=0.3901806440322565 0.02 1; visual box size=0.3901806440322565 0.02 1
- added link hand_part_2_sensor_0_right, mass 0; collision box size=0.3901806440322565 0.02 1; visual box size=0.3901806440322565 0.02 1
- added link hand_part_2_sensor_0_top, mass 0; collision box size=0.3901806440322565 0.2 0.02; visual box size=0.3901806440322565 0.2 0.02
- added link hand_part_3, mass 2; collision box size=0.3901806440322565 0.2 1; visual box size=0.3901806440322565 0.2 1
- added link hand_part_3_sensor_0_bottom, mass 0; collision box size=0.3901806440322565 0.2 0.02; visual box size=0.3901806440322565 0.2 0.02
- added link hand_part_3_sensor_0_left, mass 0; collision box size=0.3901806440322565 0.02 1; visual box size=0.3901806440322565 0.02 1
- added link hand_part_3_sensor_0_right, mass 0; collision box size=0.3901806440322565 0.02 1; visual box size=0.3901806440322565 0.02 1
- added link hand_part_3_sensor_0_top, mass 0; collision box size=0.3901806440322565 0.2 0.02; visual box size=0.3901806440322565 0.2 0.02
- added link hand_part_4, mass 2; collision box size=0.3901806440322565 0.2 1; visual box size=0.3901806440322565 0.2 1
- added link hand_part_4_sensor_0_bottom, mass 0; collision box size=0.3901806440322565 0.2 0.02; visual box size=0.3901806440322565 0.2 0.02
- added link hand_part_4_sensor_0_left, mass 0; collision box size=0.3901806440322565 0.02 1; visual box size=0.3901806440322565 0.02 1
- added link hand_part_4_sensor_0_right, mass 0; collision box size=0.3901806440322565 0.02 1; visual box size=0.3901806440322565 0.02 1
- added link hand_part_4_sensor_0_top, mass 0; collision box size=0.3901806440322565 0.2 0.02; visual box size=0.3901806440322565 0.2 0.02
- added link hand_part_5, mass 2; collision box size=0.3901806440322565 0.2 1; visual box size=0.3901806440322565 0.2 1
- added link hand_part_5_sensor_0_bottom, mass 0; collision box size=0.3901806440322565 0.2 0.02; visual box size=0.3901806440322565 0.2 0.02
- added link hand_part_5_sensor_0_left, mass 0; collision box size=0.3901806440322565 0.02 1; visual box size=0.3901806440322565 0.02 1
- added link hand_part_5_sensor_0_right, mass 0; collision box size=0.3901806440322565 0.02 1; visual box size=0.3901806440322565 0.02 1
- added link hand_part_5_sensor_0_stop, mass 0; collision box size=0.02 0.2 1; visual box size=0.02 0.2 1
- added link hand_part_5_sensor_0_top, mass 0; collision box size=0.3901806440322565 0.2 0.02; visual box size=0.3901806440322565 0.2 0.02
- added link wrist, mass 2; collision box size=0.2 0.2 0.1; visual box size=0.2 0.2 0.1
- added link wrist_sensor_0_left, mass 0; collision box size=0.2 0.02 0.1; visual box size=0.2 0.02 0.1
- added link wrist_sensor_0_right, mass 0; collision box size=0.2 0.02 0.1; visual box size=0.2 0.02 0.1
- added link wrist_sensor_0_start, mass 0; collision box size=0.02 0.2 0.1; visual box size=0.02 0.2 0.1
- added link wrist_sensor_0_stop, mass 0; collision box size=0.02 0.2 0.1; visual box size=0.02 0.2 0.1
Joints:
- removed joint arm_hand_joint
- removed joint hand_hand_sensor_0_left_joint
- removed joint hand_hand_sensor_0_right_joint
- removed joint hand_hand_sensor_0_start_joint
- removed joint hand_hand_sensor_0_stop_joint
- added joint arm_wrist_joint: type fixed, parent arm, child wrist, origin xyz=1.275 0 -0.15000000000000002 rpy=0 0 0, axis 0 1 0
- added joint hand_part_0_hand_part_0_sensor_0_bottom_joint: type fixed, parent hand_part_0, child hand_part_0_sensor_0_bottom, origin xyz=0 0 -0.5 rpy=0 0 0, axis 0 1 0
- added joint hand_part_0_hand_part_0_sensor_0_start_joint: type fixed, parent hand_part_0, child hand_part_0_sensor_0_start, origin xyz=0.1 0 0 rpy=0 0 0, axis 0 1 0
- added joint hand_part_0_hand_part_0_sensor_0_stop_joint: type fixed, parent hand_part_0, child hand_part_0_sensor_0_stop, origin xyz=-0.1 0 0 rpy=0 0 0, axis 0 1 0
- added joint hand_part_0_hand_part_0_sensor_0_top_joint: type fixed, parent hand_part_0, child hand_part_0_sensor_0_top, origin xyz=0 0 0.5 rpy=0 0 0, axis 0 1 0
- added joint hand_part_0_hand_part_11_joint: type fixed, parent hand_part_0, child hand_part_11, origin xyz=-1.356115557921096 -0.9061274463528874 0 rpy=0 0 2.7488935718910685, axis 0 1 0
- added joint hand_part_0_hand_part_12_joint: type fixed, parent hand_part_0, child hand_part_12, origin xyz=-0.9807852804032305 -0.9807852804032303 0 rpy=0 0 3.141592653589793, axis 0 1 0
- added joint hand_part_0_hand_part_13_joint: type fixed, parent hand_part_0, child hand_part_13, origin xyz=-0.6054550028853648 -0.9061274463528876 0 rpy=0 0 3.5342917352885177, axis 0 1 0
- added joint hand_part_0_hand_part_14_joint: type fixed, parent hand_part_0, child hand_part_14, origin xyz=-0.28726535774215683 -0.6935199226610738 0 rpy=0 0 3.9269908169872414, axis 0 1 0
- added joint hand_part_0_hand_part_15_joint: type fixed, parent hand_part_0, child hand_part_15, origin xyz=-0.07465783405034283 -0.3753302775178658 0 rpy=0 0 4.319689898685965, axis 0 1 0
- added joint hand_part_0_hand_part_1_joint: type fixed, parent hand_part_0, child hand_part_1, origin xyz=-0.07465783405034261 0.3753302775178652 0 rpy=0 0 -1.1780972450961724, axis 0 1 0
- added joint hand_part_0_hand_part_2_joint: type fixed, parent hand_part_0, child hand_part_2, origin xyz=-0.2872653577421566 0.6935199226610735 0 rpy=0 0 -0.7853981633974483, axis 0 1 0
- added joint hand_part_0_hand_part_3_joint: type fixed, parent hand_part_0, child hand_part_3, origin xyz=-0.605455002885365 0.9061274463528877 0 rpy=0 0 -0.39269908169872414, axis 0 1 0
- added joint hand_part_0_hand_part_4_joint: type fixed, parent hand_part_0, child hand_part_4, origin xyz=-0.9807852804032302 0.9807852804032303 0 rpy=0 0 0.0, axis 0 1 0
- added joint hand_part_0_hand_part_5_joint: type fixed, parent hand_part_0, child hand_part_5, origin xyz=-1.3561155579210953 0.9061274463528877 0 rpy=0 0 0.39269908169872414, axis 0 1 0
- added joint hand_part_11_hand_part_11_sensor_0_bottom_joint: type fixed, parent hand_part_11, child hand_part_11_sensor_0_bottom, origin xyz=0 0 -0.5 rpy=0 0 0, axis 0 1 0
- added joint hand_part_11_hand_part_11_sensor_0_left_joint: type fixed, parent hand_part_11, child hand_part_11_sensor_0_left, origin xyz=0 0.1 0 rpy=0 0 0, axis 0 1 0
- added joint hand_part_11_hand_part_11_sensor_0_right_joint: type fixed, parent hand_part_11, child hand_part_11_sensor_0_right, origin xyz=0 -0.1 0 rpy=0 0 0, axis 0 1 0
- added joint hand_part_11_hand_part_11_sensor_0_start_joint: type fixed, parent hand_part_11, child hand_part_11_sensor_0_start, origin xyz=0.19509032201612825 0 0 rpy=0 0 0, axis 0 1 0
- added joint hand_part_11_hand_part_11_sensor_0_top_joint: type fixed, parent hand_part_11, child hand_part_11_sensor_0_top, origin xyz=0 0 0.5 rpy=0 0 0, axis 0 1 0
- added joint hand_part_12_hand_part_12_sensor_0_bottom_joint: type fixed, parent hand_part_12, child hand_part_12_sensor_0_bottom, origin xyz=0 0 -0.5 rpy=0 0 0, axis 0 1 0
- added joint hand_part_12_hand_part_12_sensor_0_left_joint: type fixed, parent hand_part_12, child hand_part_12_sensor_0_left, origin xyz=0 0.1 0 rpy=0 0 0, axis 0 1 0
- added joint hand_part_12_hand_part_12_sensor_0_right_joint: type fixed, parent hand_part_12, child hand_part_12_sensor_0_right, origin xyz=0 -0.1 0 rpy=0 0 0, axis 0 1 0
- added joint hand_part_12_hand_part_12_sensor_0_top_joint: type fixed, parent hand_part_12, child hand_part_12_sensor_0_top, origin xyz=0 0 0.5 rpy=0 0 0, axis 0 1 0
- added joint hand_part_13_hand_part_13_sensor_0_bottom_joint: type fixed, parent hand_part_13, child hand_part_13_sensor_0_bottom, origin xyz=0 0 -0.5 rpy=0 0 0, axis 0 1 0
- added joint hand_part_13_hand_part_13_sensor_0_left_joint: type fixed, parent hand_part_13, child hand_part_13_sensor_0_left, origin xyz=0 0.1 0 rpy=0 0 0, axis 0 1 0
- added joint hand_part_13_hand_part_13_sensor_0_right_joint: type fixed, parent hand_part_13, child hand_part_13_sensor_0_right, origin xyz=0 -0.1 0 rpy=0 0 0, axis 0 1 0
- added joint hand_part_13_hand_part_13_sensor_0_top_joint: type fixed, parent hand_part_13, child hand_part_13_sensor_0_top, origin xyz=0 0 0.5 rpy=0 0 0, axis 0 1 0
- added joint hand_part_14_hand_part_14_sensor_0_bottom_joint: type fixed, parent hand_part_14, child hand_part_14_sensor_0_bottom, origin xyz=0 0 -0.5 rpy=0 0 0, axis 0 1 0
- added joint hand_part_14_hand_part_14_sensor_0_left_joint: type fixed, parent hand_part_14, child hand_part_14_sensor_0_left, origin xyz=0 0.1 0 rpy=0 0 0, axis 0 1 0
- added joint hand_part_14_hand_part_14_sensor_0_right_joint: type fixed, parent hand_part_14, child hand_part_14_sensor_0_right, origin xyz=0 -0.1 0 rpy=0 0 0, axis 0 1 0
- added joint hand_part_14_hand_part_14_sensor_0_top_joint: type fixed, parent hand_part_14, child hand_part_14_sensor_0_top, origin xyz=0 0 0.5 rpy=0 0 0, axis 0 1 0
- added joint hand_part_15_hand_part_15_sensor_0_bottom_joint: type fixed, parent hand_part_15, child hand_part_15_sensor_0_bottom, origin xyz=0 0 -0.5 rpy=0 0 0, axis 0 1 0
- added joint hand_part_15_hand_part_15_sensor_0_left_joint: type fixed, parent hand_part_15, child hand_part_15_sensor_0_left, origin xyz=0 0.1 0 rpy=0 0 0, axis 0 1 0
- added joint hand_part_15_hand_part_15_sensor_0_right_joint: type fixed, parent hand_part_15, child hand_part_15_sensor_0_right, origin xyz=0 -0.1 0 rpy=0 0 0, axis 0 1 0
- added joint hand_part_15_hand_part_15_sensor_0_top_joint: type fixed, parent hand_part_15, child hand_part_15_sensor_0_top, origin xyz=0 0 0.5 rpy=0 0 0, axis 0 1 0
- added joint hand_part_1_hand_part_1_sensor_0_bottom_joint: type fixed, parent hand_part_1, child hand_part_1_sensor_0_bottom, origin xyz=0 0 -0.5 rpy=0 0 0, axis 0 1 0
- added joint hand_part_1_hand_part_1_sensor_0_left_joint: type fixed, parent hand_part_1, child hand_part_1_sensor_0_left, origin xyz=0 0.1 0 rpy=0 0 0, axis 0 1 0
- added joint hand_part_1_hand_part_1_sensor_0_right_joint: type fixed, parent hand_part_1, child hand_part_1_sensor_0_right, origin xyz=0 -0.1 0 rpy=0 0 0, axis 0 1 0
- added joint hand_part_1_hand_part_1_sensor_0_top_joint: type fixed, parent hand_part_1, child hand_part_1_sensor_0_top, origin xyz=0 0 0.5 rpy=0 0 0, axis 0 1 0
- added joint hand_part_2_hand_part_2_sensor_0_bottom_joint: type fixed, parent hand_part_2, child hand_part_2_sensor_0_bottom, origin xyz=0 0 -0.5 rpy=0 0 0, axis 0 1 0
- added joint hand_part_2_hand_part_2_sensor_0_left_joint: type fixed, parent hand_part_2, child hand_part_2_sensor_0_left, origin xyz=0 0.1 0 rpy=0 0 0, axis 0 1 0
- added joint hand_part_2_hand_part_2_sensor_0_right_joint: type fixed, parent hand_part_2, child hand_part_2_sensor_0_right, origin xyz=0 -0.1 0 rpy=0 0 0, axis 0 1 0
- added joint hand_part_2_hand_part_2_sensor_0_top_joint: type fixed, parent hand_part_2, child hand_part_2_sensor_0_top, origin xyz=0 0 0.5 rpy=0 0 0, axis 0 1 0
- added joint hand_part_3_hand_part_3_sensor_0_bottom_joint: type fixed, parent hand_part_3, child hand_part_3_sensor_0_bottom, origin xyz=0 0 -0.5 rpy=0 0 0, axis 0 1 0
- added joint hand_part_3_hand_part_3_sensor_0_left_joint: type fixed, parent hand_part_3, child hand_part_3_sensor_0_left, origin xyz=0 0.1 0 rpy=0 0 0, axis 0 1 0
- added joint hand_part_3_hand_part_3_sensor_0_right_joint: type fixed, parent hand_part_3, child hand_part_3_sensor_0_right, origin xyz=0 -0.1 0 rpy=0 0 0, axis 0 1 0
- added joint hand_part_3_hand_part_3_sensor_0_top_joint: type fixed, parent hand_part_3, child hand_part_3_sensor_0_top, origin xyz=0 0 0.5 rpy=0 0 0, axis 0 1 0
- added joint hand_part_4_hand_part_4_sensor_0_bottom_joint: type fixed, parent hand_part_4, child hand_part_4_sensor_0_bottom, origin xyz=0 0 -0.5 rpy=0 0 0, axis 0 1 0
- added joint hand_part_4_hand_part_4_sensor_0_left_joint: type fixed, parent hand_part_4, child hand_part_4_sensor_0_left, origin xyz=0 0.1 0 rpy=0 0 0, axis 0 1 0
- added joint hand_part_4_hand_part_4_sensor_0_right_joint: type fixed, parent hand_part_4, child hand_part_4_sensor_0_right, origin xyz=0 -0.1 0 rpy=0 0 0, axis 0 1 0
- added joint hand_part_4_hand_part_4_sensor_0_top_joint: type fixed, parent hand_part_4, child hand_part_4_sensor_0_top, origin xyz=0 0 0.5 rpy=0 0 0, axis 0 1 0
- added joint hand_part_5_hand_part_5_sensor_0_bottom_joint: type fixed, parent hand_part_5, child hand_part_5_sensor_0_bottom, origin xyz=0 0 -0.5 rpy=0 0 0, axis 0 1 0
- added joint hand_part_5_hand_part_5_sensor_0_left_joint: type fixed, parent hand_part_5, child hand_part_5_sensor_0_left, origin xyz=0 0.1 0 rpy=0 0 0, axis 0 1 0
- added joint hand_part_5_hand_part_5_sensor_0_right_joint: type fixed, parent hand_part_5, child hand_part_5_sensor_0_right, origin xyz=0 -0.1 0 rpy=0 0 0, axis 0 1 0
- added joint hand_part_5_hand_part_5_sensor_0_stop_joint: type fixed, parent hand_part_5, child hand_part_5_sensor_0_stop, origin xyz=-0.19509032201612825 0 0 rpy=0 0 0, axis 0 1 0
- added joint hand_part_5_hand_part_5_sensor_0_top_joint: type fixed, parent hand_part_5, child hand_part_5_sensor_0_top, origin xyz=0 0 0.5 rpy=0 0 0, axis 0 1 0
- added joint wrist_hand_part_0_joint: type fixed, parent wrist, child hand_part_0, origin xyz=0 0 -0.55 rpy=0 0 0, axis 0 1 0
- added joint wrist_wrist_sensor_0_left_joint: type fixed, parent wrist, child wrist_sensor_0_left, origin xyz=0 0.1 0 rpy=0 0 0, axis 0 1 0
- added joint wrist_wrist_sensor_0_right_joint: type fixed, parent wrist, child wrist_sensor_0_right, origin xyz=0 -0.1 0 rpy=0 0 0, axis 0 1 0
- added joint wrist_wrist_sensor_0_start_joint: type fixed, parent wrist, child wrist_sensor_0_start, origin xyz=0.1 0 0 rpy=0 0 0, axis 0 1 0
- added joint wrist_wrist_sensor_0_stop_joint: type fixed, parent wrist, child wrist_sensor_0_stop, origin xyz=-0.1 0 0 rpy=0 0 0, axis 0 1 0

Commit message: 2025_03_24, big test, great results. wide view doesn't seem to help.

File: pybullet_data/robots/robot_two_head_arm_a.urdf (robot description, URDF)
Before this commit: robot robot, 56 links, 55 joints
Links:
- removed link body_face_top_0
- removed link body_face_top_1
- removed link body_face_top_10
- removed link body_face_top_11
- removed link body_face_top_12
- removed link body_face_top_2
- removed link body_face_top_3
- removed link body_face_top_4
- removed link body_face_top_5
- removed link body_face_top_6
- removed link body_face_top_7
- removed link body_face_top_8
- removed link body_face_top_9
Joints:
- removed joint body_body_face_top_0_joint
- removed joint body_body_face_top_10_joint
- removed joint body_body_face_top_11_joint
- removed joint body_body_face_top_12_joint
- removed joint body_body_face_top_1_joint
- removed joint body_body_face_top_2_joint
- removed joint body_body_face_top_3_joint
- removed joint body_body_face_top_4_joint
- removed joint body_body_face_top_5_joint
- removed joint body_body_face_top_6_joint
- removed joint body_body_face_top_7_joint
- removed joint body_body_face_top_8_joint
- removed joint body_body_face_top_9_joint

File: pybullet_data/robots/robot_two_head_arm_b.urdf (robot description, URDF)
Before this commit: robot robot, 56 links, 55 joints
Links:
- removed link body_face_top_0
- removed link body_face_top_1
- removed link body_face_top_10
- removed link body_face_top_11
- removed link body_face_top_12
- removed link body_face_top_2
- removed link body_face_top_3
- removed link body_face_top_4
- removed link body_face_top_5
- removed link body_face_top_6
- removed link body_face_top_7
- removed link body_face_top_8
- removed link body_face_top_9
- link hand: geometry collision box size=1 0.6000000000000001 1.25; visual box size=1 0.6000000000000001 1.25
- link hand_sensor_0_bottom: geometry collision box size=1.0 0.6000000000000001 0.02; visual box size=1.0 0.6000000000000001 0.02
- link hand_sensor_0_start: geometry collision box size=0.02 0.6000000000000001 1.25; visual box size=0.02 0.6000000000000001 1.25
- link hand_sensor_0_stop: geometry collision box size=0.02 0.6000000000000001 1.25; visual box size=0.02 0.6000000000000001 1.25
- link hand_sensor_0_top: geometry collision box size=1.0 0.6000000000000001 0.02; visual box size=1.0 0.6000000000000001 0.02
Joints:
- removed joint body_body_face_top_0_joint
- removed joint body_body_face_top_10_joint
- removed joint body_body_face_top_11_joint
- removed joint body_body_face_top_12_joint
- removed joint body_body_face_top_1_joint
- removed joint body_body_face_top_2_joint
- removed joint body_body_face_top_3_joint
- removed joint body_body_face_top_4_joint
- removed joint body_body_face_top_5_joint
- removed joint body_body_face_top_6_joint
- removed joint body_body_face_top_7_joint
- removed joint body_body_face_top_8_joint
- removed joint body_body_face_top_9_joint
- joint hand_hand_sensor_0_left_joint: origin xyz=0 0.5 0 rpy=0 0 0 -> xyz=0 0.30000000000000004 0 rpy=0 0 0
- joint hand_hand_sensor_0_right_joint: origin xyz=0 -0.5 0 rpy=0 0 0 -> xyz=0 -0.30000000000000004 0 rpy=0 0 0
