Commit message: 2025_04_02. Big test, great results. Still need to fix generalization tests.

File: pybullet_data/robots/robot_two_head_arm_a.urdf (robot description, URDF)
Before this commit: robot robot, 34 links, 33 joints
Links:
- removed link back_left_wheel
- removed link back_right_wheel
- removed link from_left_wheel
- removed link from_right_wheel
- added link left_spoke_1, mass 0; collision box size=0.3 0.03 0.1; visual box size=0.3 0.03 0.1
- added link left_spoke_2, mass 0; collision box size=0.03 0.3 0.1; visual box size=0.03 0.3 0.1
- added link left_wheel, mass 0.1; collision cylinder length=0.1 radius=0.2; visual cylinder length=0.1 radius=0.2
- added link right_spoke_1, mass 0; collision box size=0.3 0.03 0.1; visual box size=0.3 0.03 0.1
- added link right_spoke_2, mass 0; collision box size=0.03 0.3 0.1; visual box size=0.03 0.3 0.1
- added link right_wheel, mass 0.1; collision cylinder length=0.1 radius=0.2; visual cylinder length=0.1 radius=0.2
Joints:
- removed joint body_back_left_wheel_joint
- removed joint body_back_right_wheel_joint
- removed joint body_from_left_wheel_joint
- removed joint body_from_right_wheel_joint
- added joint body_left_wheel_joint: type continuous, parent body, child left_wheel, origin xyz=0 0.5 -0.3 rpy=1.5708 0 0, axis 0 0 1, limit lower=0 upper=0 effort=0 velocity=0
- added joint body_right_wheel_joint: type continuous, parent body, child right_wheel, origin xyz=0 -0.5 -0.3 rpy=1.5708 0 0, axis 0 0 1, limit lower=0 upper=0 effort=0 velocity=0
- added joint left_wheel_left_spoke_1_joint: type fixed, parent left_wheel, child left_spoke_1, origin xyz=0 0 -0.01 rpy=0 0 0, axis 0 0 1
- added joint left_wheel_left_spoke_2_joint: type fixed, parent left_wheel, child left_spoke_2, origin xyz=0 0 -0.01 rpy=0 0 0, axis 0 0 1
- added joint right_wheel_right_spoke_1_joint: type fixed, parent right_wheel, child right_spoke_1, origin xyz=0 0 0.01 rpy=0 0 0, axis 0 0 1
- added joint right_wheel_right_spoke_2_joint: type fixed, parent right_wheel, child right_spoke_2, origin xyz=0 0 0.01 rpy=0 0 0, axis 0 0 1
