Commit message: 2025_04_14. Big test, successful! Better compositionality, better robot.

File: pybullet_data/robots/robot.urdf (robot description, URDF)
Before this commit: robot robot, 48 links, 47 joints
Links:
- added link arm_outline_1, mass 0; collision box size=1.77 0.01 0.01; visual box size=1.77 0.01 0.01
- added link arm_outline_2, mass 0; collision box size=1.77 0.01 0.01; visual box size=1.77 0.01 0.01
- added link arm_outline_3, mass 0; collision box size=1.77 0.01 0.01; visual box size=1.77 0.01 0.01
- added link arm_outline_4, mass 0; collision box size=1.77 0.01 0.01; visual box size=1.77 0.01 0.01
- added link arm_outline_5, mass 0; collision box size=0.01 0.01 0.22; visual box size=0.01 0.01 0.22
- added link arm_outline_6, mass 0; collision box size=0.01 0.01 0.22; visual box size=0.01 0.01 0.22
- added link arm_outline_7, mass 0; collision box size=0.01 0.22 0.01; visual box size=0.01 0.22 0.01
- link left_wheel: mass 0 -> 0.1
- link right_wheel: mass 0 -> 0.1
Joints:
- added joint arm_arm_outline_1_joint: type fixed, parent arm, child arm_outline_1, origin xyz=0 0.1 0.1 rpy=0 0 0, axis 0 1 0
- added joint arm_arm_outline_2_joint: type fixed, parent arm, child arm_outline_2, origin xyz=0 -0.1 0.1 rpy=0 0 0, axis 0 1 0
- added joint arm_arm_outline_3_joint: type fixed, parent arm, child arm_outline_3, origin xyz=0 0.1 -0.1 rpy=0 0 0, axis 0 1 0
- added joint arm_arm_outline_4_joint: type fixed, parent arm, child arm_outline_4, origin xyz=0 -0.1 -0.1 rpy=0 0 0, axis 0 1 0
- added joint arm_arm_outline_5_joint: type fixed, parent arm, child arm_outline_5, origin xyz=0.875 0.1 0 rpy=0 0 0, axis 0 1 0
- added joint arm_arm_outline_6_joint: type fixed, parent arm, child arm_outline_6, origin xyz=0.875 -0.1 0 rpy=0 0 0, axis 0 1 0
- added joint arm_arm_outline_7_joint: type fixed, parent arm, child arm_outline_7, origin xyz=0.875 0 -0.1 rpy=0 0 0, axis 0 1 0

Commit message: 2025_05_13. Big test, kind of good. Trying durations.

File: pybullet_data/robots/robot.urdf (robot description, URDF)
Before this commit: robot robot, 65 links, 64 joints
Links:
- link arm_sensor_0_bottom: geometry collision box size=1.75 0.2 0.03; visual box size=1.75 0.2 0.03
- link arm_sensor_0_left: geometry collision box size=1.75 0.03 0.2; visual box size=1.75 0.03 0.2
- link arm_sensor_0_right: geometry collision box size=1.75 0.03 0.2; visual box size=1.75 0.03 0.2
- link arm_sensor_0_top: geometry collision box size=1.75 0.2 0.03; visual box size=1.75 0.2 0.03
- link body_sensor_0_bottom: geometry collision box size=1.0 1 0.03; visual box size=1.0 1 0.03
- link body_sensor_0_left: geometry collision box size=1.0 0.03 1; visual box size=1.0 0.03 1
- link body_sensor_0_right: geometry collision box size=1.0 0.03 1; visual box size=1.0 0.03 1
- link body_sensor_0_start: geometry collision box size=0.03 1 1; visual box size=0.03 1 1
- link body_sensor_0_stop: geometry collision box size=0.03 1 1; visual box size=0.03 1 1
- link body_sensor_0_top: geometry collision box size=1.0 1 0.03; visual box size=1.0 1 0.03
- link hand_sensor_0_bottom: geometry collision box size=1.0 0.6000000000000001 0.03; visual box size=1.0 0.6000000000000001 0.03
- link hand_sensor_0_left: geometry collision box size=1.0 0.03 1.25; visual box size=1.0 0.03 1.25
- link hand_sensor_0_right: geometry collision box size=1.0 0.03 1.25; visual box size=1.0 0.03 1.25
- link hand_sensor_0_start: geometry collision box size=0.03 0.6000000000000001 1.25; visual box size=0.03 0.6000000000000001 1.25
- link hand_sensor_0_stop: geometry collision box size=0.03 0.6000000000000001 1.25; visual box size=0.03 0.6000000000000001 1.25
- link hand_sensor_0_top: geometry collision box size=1.0 0.6000000000000001 0.03; visual box size=1.0 0.6000000000000001 0.03

Commit message: 2025_07_06. Big test. Awesome physics, but why is left easier than right?

File: pybullet_data/robots/robot.urdf (robot description, URDF)
Before this commit: robot robot, 65 links, 64 joints
Links:
- link arm_sensor_0_bottom: geometry collision box size=1.75 0.2 0.03; visual box size=1.75 0.2 0.03
- link arm_sensor_0_left: geometry collision box size=1.75 0.03 0.2; visual box size=1.75 0.03 0.2
- link arm_sensor_0_right: geometry collision box size=1.75 0.03 0.2; visual box size=1.75 0.03 0.2
- link arm_sensor_0_top: geometry collision box size=1.75 0.2 0.03; visual box size=1.75 0.2 0.03
- link body: mass 100 -> 1000
- link body_sensor_0_bottom: geometry collision box size=1.0 1 0.03; visual box size=1.0 1 0.03
- link body_sensor_0_left: geometry collision box size=1.0 0.03 1; visual box size=1.0 0.03 1
- link body_sensor_0_right: geometry collision box size=1.0 0.03 1; visual box size=1.0 0.03 1
- link body_sensor_0_start: geometry collision box size=0.03 1 1; visual box size=0.03 1 1
- link body_sensor_0_stop: geometry collision box size=0.03 1 1; visual box size=0.03 1 1
- link body_sensor_0_top: geometry collision box size=1.0 1 0.03; visual box size=1.0 1 0.03
- link hand_sensor_0_bottom: geometry collision box size=1.0 0.6000000000000001 0.03; visual box size=1.0 0.6000000000000001 0.03
- link hand_sensor_0_left: geometry collision box size=1.0 0.03 1.25; visual box size=1.0 0.03 1.25
- link hand_sensor_0_right: geometry collision box size=1.0 0.03 1.25; visual box size=1.0 0.03 1.25
- link hand_sensor_0_start: geometry collision box size=0.03 0.6000000000000001 1.25; visual box size=0.03 0.6000000000000001 1.25
- link hand_sensor_0_stop: geometry collision box size=0.03 0.6000000000000001 1.25; visual box size=0.03 0.6000000000000001 1.25
- link hand_sensor_0_top: geometry collision box size=1.0 0.6000000000000001 0.03; visual box size=1.0 0.6000000000000001 0.03

File: pybullet_data/robots/robot_2.urdf (robot description, URDF)
Before this commit: robot robot, 65 links, 64 joints
Links:
- link arm: geometry collision box size=1.3 0.2 0.2; visual box size=1.3 0.2 0.2
- link arm_outline_1: geometry collision box size=1.3 0.005 0.005; visual box size=1.3 0.005 0.005
- link arm_outline_2: geometry collision box size=1.3 0.005 0.005; visual box size=1.3 0.005 0.005
- link arm_outline_3: geometry collision box size=1.3 0.005 0.005; visual box size=1.3 0.005 0.005
- link arm_outline_4: geometry collision box size=1.3 0.005 0.005; visual box size=1.3 0.005 0.005
- link arm_sensor_0_bottom: geometry collision box size=1.3 0.2 0.03; visual box size=1.3 0.2 0.03
- link arm_sensor_0_left: geometry collision box size=1.3 0.03 0.2; visual box size=1.3 0.03 0.2
- link arm_sensor_0_right: geometry collision box size=1.3 0.03 0.2; visual box size=1.3 0.03 0.2
- link arm_sensor_0_top: geometry collision box size=1.3 0.2 0.03; visual box size=1.3 0.2 0.03
- link body: mass 100 -> 1000
Joints:
- joint arm_arm_outline_5_joint: origin xyz=0.8724999999999999 0.10250000000000001 0 rpy=0 0 0 -> xyz=0.6475 0.10250000000000001 0 rpy=0 0 0
- joint arm_arm_outline_6_joint: origin xyz=0.8724999999999999 -0.10250000000000001 0 rpy=0 0 0 -> xyz=0.6475 -0.10250000000000001 0 rpy=0 0 0
- joint arm_arm_outline_7_joint: origin xyz=0.8724999999999999 0 -0.10250000000000001 rpy=0 0 0 -> xyz=0.6475 0 -0.10250000000000001 rpy=0 0 0
- joint arm_hand_joint: origin xyz=1.375 0 -0.525 rpy=0 0 0 -> xyz=1.15 0 -0.525 rpy=0 0 0
- joint joint_2_arm_joint: origin xyz=0.975 0 0 rpy=0 0 0 -> xyz=0.75 0 0 rpy=0 0 0

File: robot_2.urdf (robot description, URDF)
Before this commit: robot robot, 65 links, 64 joints
Links:
- link arm: geometry collision box size=1.3 0.2 0.2; visual box size=1.3 0.2 0.2
- link arm_outline_1: geometry collision box size=1.3 0.005 0.005; visual box size=1.3 0.005 0.005
- link arm_outline_2: geometry collision box size=1.3 0.005 0.005; visual box size=1.3 0.005 0.005
- link arm_outline_3: geometry collision box size=1.3 0.005 0.005; visual box size=1.3 0.005 0.005
- link arm_outline_4: geometry collision box size=1.3 0.005 0.005; visual box size=1.3 0.005 0.005
- link arm_sensor_0_bottom: geometry collision box size=1.3 0.2 0.03; visual box size=1.3 0.2 0.03
- link arm_sensor_0_left: geometry collision box size=1.3 0.03 0.2; visual box size=1.3 0.03 0.2
- link arm_sensor_0_right: geometry collision box size=1.3 0.03 0.2; visual box size=1.3 0.03 0.2
- link arm_sensor_0_top: geometry collision box size=1.3 0.2 0.03; visual box size=1.3 0.2 0.03
Joints:
- joint arm_arm_outline_5_joint: origin xyz=0.8724999999999999 0.10250000000000001 0 rpy=0 0 0 -> xyz=0.6475 0.10250000000000001 0 rpy=0 0 0
- joint arm_arm_outline_6_joint: origin xyz=0.8724999999999999 -0.10250000000000001 0 rpy=0 0 0 -> xyz=0.6475 -0.10250000000000001 0 rpy=0 0 0
- joint arm_arm_outline_7_joint: origin xyz=0.8724999999999999 0 -0.10250000000000001 rpy=0 0 0 -> xyz=0.6475 0 -0.10250000000000001 rpy=0 0 0
- joint arm_hand_joint: origin xyz=1.375 0 -0.525 rpy=0 0 0 -> xyz=1.15 0 -0.525 rpy=0 0 0
- joint joint_2_arm_joint: origin xyz=0.975 0 0 rpy=0 0 0 -> xyz=0.75 0 0 rpy=0 0 0

Commit message: 2025_07_11. AWESOME, fixed the left/right problem.

File: pybullet_data/robots/robot.urdf (robot description, URDF)
Before this commit: robot robot, 65 links, 64 joints
Joints:
- joint body_joint_1_joint: type continuous -> revolute
- joint joint_1_joint_2_joint: type continuous -> revolute

File: pybullet_data/robots/robot_2.urdf (robot description, URDF)
Before this commit: robot robot, 65 links, 64 joints
Joints:
- joint body_joint_1_joint: type continuous -> revolute
- joint joint_1_joint_2_joint: type continuous -> revolute

Commit message: 2025_08_20. Better, but also bad.

File: pybullet_data/robots/robot.urdf (robot description, URDF)
Before this commit: robot robot, 65 links, 64 joints
Links:
- link arm: geometry collision box size=1.5 0.2 0.2; visual box size=1.5 0.2 0.2
- link arm_outline_1: geometry collision box size=1.5 0.005 0.005; visual box size=1.5 0.005 0.005
- link arm_outline_2: geometry collision box size=1.5 0.005 0.005; visual box size=1.5 0.005 0.005
- link arm_outline_3: geometry collision box size=1.5 0.005 0.005; visual box size=1.5 0.005 0.005
- link arm_outline_4: geometry collision box size=1.5 0.005 0.005; visual box size=1.5 0.005 0.005
- link arm_sensor_0_bottom: geometry collision box size=1.5 0.2 0.03; visual box size=1.5 0.2 0.03
- link arm_sensor_0_left: geometry collision box size=1.5 0.03 0.2; visual box size=1.5 0.03 0.2
- link arm_sensor_0_right: geometry collision box size=1.5 0.03 0.2; visual box size=1.5 0.03 0.2
- link arm_sensor_0_top: geometry collision box size=1.5 0.2 0.03; visual box size=1.5 0.2 0.03
Joints:
- joint arm_arm_outline_5_joint: origin xyz=0.8724999999999999 0.10250000000000001 0 rpy=0 0 0 -> xyz=0.7474999999999999 0.10250000000000001 0 rpy=0 0 0
- joint arm_arm_outline_6_joint: origin xyz=0.8724999999999999 -0.10250000000000001 0 rpy=0 0 0 -> xyz=0.7474999999999999 -0.10250000000000001 0 rpy=0 0 0
- joint arm_arm_outline_7_joint: origin xyz=0.8724999999999999 0 -0.10250000000000001 rpy=0 0 0 -> xyz=0.7474999999999999 0 -0.10250000000000001 rpy=0 0 0
- joint arm_hand_joint: origin xyz=1.375 0 -0.525 rpy=0 0 0 -> xyz=1.25 0 -0.525 rpy=0 0 0
- joint joint_2_arm_joint: origin xyz=0.975 0 0 rpy=0 0 0 -> xyz=0.85 0 0 rpy=0 0 0

Commit message: 2025_09_24. Experimenting with longer object distances.

File: pybullet_data/robots/robot.urdf (robot description, URDF)
Before this commit: robot robot, 65 links, 64 joints
Links:
- removed link body_face_front_0
- removed link body_face_front_1
- removed link body_face_front_2
- removed link body_face_front_3
- removed link body_face_front_4
- removed link body_face_front_5
- removed link body_face_front_6
- removed link body_face_front_7
- removed link body_face_front_8
- added link camera_1, mass 0; collision cylinder length=0.05 radius=0.2; visual cylinder length=0.05 radius=0.2
- added link camera_2, mass 0; collision cylinder length=0.05 radius=0.175; visual cylinder length=0.05 radius=0.175
- added link camera_3, mass 0; collision cylinder length=0.05 radius=0.1; visual cylinder length=0.05 radius=0.1
- added link camera_4, mass 0; collision cylinder length=0.05 radius=0.025; visual cylinder length=0.05 radius=0.025
Joints:
- removed joint body_body_face_front_0_joint
- removed joint body_body_face_front_1_joint
- removed joint body_body_face_front_2_joint
- removed joint body_body_face_front_3_joint
- removed joint body_body_face_front_4_joint
- removed joint body_body_face_front_5_joint
- removed joint body_body_face_front_6_joint
- removed joint body_body_face_front_7_joint
- removed joint body_body_face_front_8_joint
- added joint body_camera_1_joint: type fixed, parent body, child camera_1, origin xyz=0.5 0 0 rpy=0 1.5708 0, axis 0 0 1
- added joint body_camera_2_joint: type fixed, parent body, child camera_2, origin xyz=0.501 0 0 rpy=0 1.5708 0, axis 0 0 1
- added joint body_camera_3_joint: type fixed, parent body, child camera_3, origin xyz=0.502 0 0 rpy=0 1.5708 0, axis 0 0 1
- added joint body_camera_4_joint: type fixed, parent body, child camera_4, origin xyz=0.503 0 0 rpy=0 1.5708 0, axis 0 0 1

File: pybullet_data/robots/robot_2.urdf (robot description, URDF)
Before this commit: robot robot, 65 links, 64 joints
Links:
- removed link body_face_front_0
- removed link body_face_front_1
- removed link body_face_front_2
- removed link body_face_front_3
- removed link body_face_front_4
- removed link body_face_front_5
- removed link body_face_front_6
- removed link body_face_front_7
- removed link body_face_front_8
Joints:
- removed joint body_body_face_front_0_joint
- removed joint body_body_face_front_1_joint
- removed joint body_body_face_front_2_joint
- removed joint body_body_face_front_3_joint
- removed joint body_body_face_front_4_joint
- removed joint body_body_face_front_5_joint
- removed joint body_body_face_front_6_joint
- removed joint body_body_face_front_7_joint
- removed joint body_body_face_front_8_joint

File: pybullet_data/robots/robot_3.urdf (robot description, URDF)
Before this commit: robot robot, 65 links, 64 joints
Links:
- removed link body_face_front_0
- removed link body_face_front_1
- removed link body_face_front_2
- removed link body_face_front_3
- removed link body_face_front_4
- removed link body_face_front_5
- removed link body_face_front_6
- removed link body_face_front_7
- removed link body_face_front_8
Joints:
- removed joint body_body_face_front_0_joint
- removed joint body_body_face_front_1_joint
- removed joint body_body_face_front_2_joint
- removed joint body_body_face_front_3_joint
- removed joint body_body_face_front_4_joint
- removed joint body_body_face_front_5_joint
- removed joint body_body_face_front_6_joint
- removed joint body_body_face_front_7_joint
- removed joint body_body_face_front_8_joint

File: robot.urdf (robot description, URDF)
Before this commit: robot robot, 65 links, 64 joints
Links:
- added link camera_1, mass 0; collision cylinder length=0.05 radius=0.2; visual cylinder length=0.05 radius=0.2
- added link camera_2, mass 0; collision cylinder length=0.05 radius=0.175; visual cylinder length=0.05 radius=0.175
- added link camera_3, mass 0; collision cylinder length=0.05 radius=0.1; visual cylinder length=0.05 radius=0.1
- added link camera_4, mass 0; collision cylinder length=0.05 radius=0.025; visual cylinder length=0.05 radius=0.025
Joints:
- added joint body_camera_1_joint: type fixed, parent body, child camera_1, origin xyz=0.5 0 0 rpy=0 1.5708 0, axis 0 0 1
- added joint body_camera_2_joint: type fixed, parent body, child camera_2, origin xyz=0.501 0 0 rpy=0 1.5708 0, axis 0 0 1
- added joint body_camera_3_joint: type fixed, parent body, child camera_3, origin xyz=0.502 0 0 rpy=0 1.5708 0, axis 0 0 1
- added joint body_camera_4_joint: type fixed, parent body, child camera_4, origin xyz=0.503 0 0 rpy=0 1.5708 0, axis 0 0 1
