Commit message: 2025_09_28. Still working, but testing force-to-move stuff.

File: pybullet_data/robots/robot_2.urdf (robot description, URDF)
Before this commit: robot robot, 56 links, 55 joints
Links:
- added link camera_1, mass 0; collision cylinder length=0.05 radius=0.2; visual cylinder length=0.05 radius=0.2
- added link camera_2, mass 0; collision cylinder length=0.05 radius=0.175; visual cylinder length=0.05 radius=0.175
- added link camera_3, mass 0; collision cylinder length=0.05 radius=0.1; visual cylinder length=0.05 radius=0.1
- added link camera_4, mass 0; collision cylinder length=0.05 radius=0.025; visual cylinder length=0.05 radius=0.025
Joints:
- added joint body_camera_1_joint: type fixed, parent body, child camera_1, origin xyz=0.5 0 0 rpy=0 1.5708 0, axis 0 0 1
- added joint body_camera_2_joint: type fixed, parent body, child camera_2, origin xyz=0.501 0 0 rpy=0 1.5708 0, axis 0 0 1
- added joint body_camera_3_joint: type fixed, parent body, child camera_3, origin xyz=0.502 0 0 rpy=0 1.5708 0, axis 0 0 1
- added joint body_camera_4_joint: type fixed, parent body, child camera_4, origin xyz=0.503 0 0 rpy=0 1.5708 0, axis 0 0 1

File: robot_2.urdf (robot description, URDF)
Before this commit: robot robot, 65 links, 64 joints
Links:
- added link camera_1, mass 0; collision cylinder length=0.05 radius=0.2; visual cylinder length=0.05 radius=0.2
- added link camera_2, mass 0; collision cylinder length=0.05 radius=0.175; visual cylinder length=0.05 radius=0.175
- added link camera_3, mass 0; collision cylinder length=0.05 radius=0.1; visual cylinder length=0.05 radius=0.1
- added link camera_4, mass 0; collision cylinder length=0.05 radius=0.025; visual cylinder length=0.05 radius=0.025
Joints:
- added joint body_camera_1_joint: type fixed, parent body, child camera_1, origin xyz=0.5 0 0 rpy=0 1.5708 0, axis 0 0 1
- added joint body_camera_2_joint: type fixed, parent body, child camera_2, origin xyz=0.501 0 0 rpy=0 1.5708 0, axis 0 0 1
- added joint body_camera_3_joint: type fixed, parent body, child camera_3, origin xyz=0.502 0 0 rpy=0 1.5708 0, axis 0 0 1
- added joint body_camera_4_joint: type fixed, parent body, child camera_4, origin xyz=0.503 0 0 rpy=0 1.5708 0, axis 0 0 1
